Commit message: description: cleaned up xacro files and fixed paths

File: up1_description/xacro/base_module/base_module.xacro (robot description, xacro)
@@ -1,6 +1,6 @@
 <?xml version="1.0"?>
 <robot xmlns:xacro="http://www.ros.org/wiki/xacro">
-  <xacro:include filename="$(find up1_description)/urdf/base_module/wheel.xacro" />
-  <xacro:include filename="$(find up1_description)/urdf/base_module/base_module.gazebo.xacro" />
+  <xacro:include filename="$(find up1_description)/xacro/base_module/wheel.xacro" />
+  <xacro:include filename="$(find up1_description)/xacro/base_module/base_module.gazebo.xacro" />
   <!-- ============================   Base Module   ============================ -->
   <xacro:macro name="base_module">
@@ -33,5 +33,5 @@
       <visual>
         <geometry>
-          <mesh filename="package://up1_description/meshes/base.stl" scale="0.001 0.001 0.001" />
+          <mesh filename="package://up1_description/meshes/base/base.stl" scale="0.001 0.001 0.001" />
         </geometry>
         <material name="grey" />
@@ -39,5 +39,5 @@
       <collision>
         <geometry>
-          <mesh filename="package://up1_description/meshes/base.stl" scale="0.001 0.001 0.001" />
+          <mesh filename="package://up1_description/meshes/base/base.stl" scale="0.001 0.001 0.001" />
         </geometry>
       </collision>

File: up1_description/xacro/base_module/wheel.xacro (robot description, xacro)
@@ -15,5 +15,5 @@
       <visual>
         <geometry>
-          <mesh filename="package://up1_description/meshes/wheel.stl" scale="0.001 0.001 0.001" />
+          <mesh filename="package://up1_description/meshes/base/wheel.stl" scale="0.001 0.001 0.001" />
         </geometry>
         <material name="black" />
@@ -21,5 +21,5 @@
       <collision>
         <geometry>
-          <mesh filename="package://up1_description/meshes/wheel.stl" scale="0.001 0.001 0.001" />
+          <mesh filename="package://up1_description/meshes/base/wheel.stl" scale="0.001 0.001 0.001" />
         </geometry>
       </collision>
@@ -42,5 +42,5 @@
       <visual>
         <geometry>
-          <mesh filename="package://up1_description/meshes/wheel.stl" scale="0.001 0.001 0.001" />
+          <mesh filename="package://up1_description/meshes/base/wheel.stl" scale="0.001 0.001 0.001" />
         </geometry>
         <material name="black" />
@@ -48,5 +48,5 @@
       <collision>
         <geometry>
-          <mesh filename="package://up1_description/meshes/wheel.stl" scale="0.001 0.001 0.001" />
+          <mesh filename="package://up1_description/meshes/base/wheel.stl" scale="0.001 0.001 0.001" />
         </geometry>
       </collision>

File: up1_description/xacro/dual_arm_module/arm.xacro (robot description, xacro)
@@ -1,5 +1,5 @@
 <?xml version="1.0"?>
 <robot xmlns:xacro="http://www.ros.org/wiki/xacro">
-  <xacro:include filename="$(find up1_description)/urdf/arm_module/arm.gazebo.xacro" />
+  <xacro:include filename="$(find up1_description)/xacro/dual_arm_module/arm.gazebo.xacro" />
   <!-- ============================   Arm   ============================ -->
   <xacro:macro name="arm" params="prefix reflect">
@@ -17,5 +17,5 @@
       <visual>
         <geometry>
-          <mesh filename="package://up1_description/meshes/armlink1.stl" scale="0.001 0.001 0.001" />
+          <mesh filename="package://up1_description/meshes/dual_arm/armlink1.stl" scale="0.001 0.001 0.001" />
         </geometry>
         <material name="white" />
@@ -23,5 +23,5 @@
       <collision>
         <geometry>
-          <mesh filename="package://up1_description/meshes/armlink1.stl" scale="0.001 0.001 0.001" />
+          <mesh filename="package://up1_description/meshes/dual_arm/armlink1.stl" scale="0.001 0.001 0.001" />
         </geometry>
       </collision>
@@ -45,5 +45,5 @@
       <visual>
         <geometry>
-          <mesh filename="package://up1_description/meshes/armlink2.stl" scale="0.001 0.001 0.001" />
+          <mesh filename="package://up1_description/meshes/dual_arm/armlink2.stl" scale="0.001 0.001 0.001" />
         </geometry>
         <material name="white" />
@@ -51,5 +51,5 @@
       <collision>
         <geometry>
-          <mesh filename="package://up1_description/meshes/armlink2.stl" scale="0.001 0.001 0.001" />
+          <mesh filename="package://up1_description/meshes/dual_arm/armlink2.stl" scale="0.001 0.001 0.001" />
         </geometry>
       </collision>
@@ -73,5 +73,5 @@
       <visual>
         <geometry>
-          <mesh filename="package://up1_description/meshes/armlink3.stl" scale="0.001 0.001 0.001" />
+          <mesh filename="package://up1_description/meshes/dual_arm/armlink3.stl" scale="0.001 0.001 0.001" />
         </geometry>
         <material name="white" />
@@ -79,5 +79,5 @@
       <collision>
         <geometry>
-          <mesh filename="package://up1_description/meshes/armlink3.stl" scale="0.001 0.001 0.001" />
+          <mesh filename="package://up1_description/meshes/dual_arm/armlink3.stl" scale="0.001 0.001 0.001" />
         </geometry>
       </collision>
@@ -101,5 +101,5 @@
       <visual>
         <geometry>
-          <mesh filename="package://up1_description/meshes/armlink4.stl" scale="0.001 0.001 0.001" />
+          <mesh filename="package://up1_description/meshes/dual_arm/armlink4.stl" scale="0.001 0.001 0.001" />
         </geometry>
         <material name="white" />
@@ -107,5 +107,5 @@
       <collision>
         <geometry>
-          <mesh filename="package://up1_description/meshes/armlink4.stl" scale="0.001 0.001 0.001" />
+          <mesh filename="package://up1_description/meshes/dual_arm/armlink4.stl" scale="0.001 0.001 0.001" />
         </geometry>
       </collision>
@@ -129,5 +129,5 @@
       <visual>
         <geometry>
-          <mesh filename="package://up1_description/meshes/armlink5.stl" scale="0.001 0.001 0.001" />
+          <mesh filename="package://up1_description/meshes/dual_arm/armlink5.stl" scale="0.001 0.001 0.001" />
         </geometry>
         <material name="white" />
@@ -135,5 +135,5 @@
       <collision>
         <geometry>
-          <mesh filename="package://up1_description/meshes/armlink5.stl" scale="0.001 0.001 0.001" />
+          <mesh filename="package://up1_description/meshes/dual_arm/armlink5.stl" scale="0.001 0.001 0.001" />
         </geometry>
       </collision>

File: up1_description/xacro/dual_arm_module/gripper.xacro (robot description, xacro)
@@ -1,5 +1,5 @@
 <?xml version="1.0"?>
 <robot xmlns:xacro="http://www.ros.org/wiki/xacro">
-  <xacro:include filename="$(find up1_description)/urdf/arm_module/gripper.gazebo.xacro" />
+  <xacro:include filename="$(find up1_description)/xacro/dual_arm_module/gripper.gazebo.xacro" />
   <!-- ============================   Gripper   ============================ -->
   <xacro:macro name="gripper" params="prefix reflect">
@@ -17,5 +17,5 @@
       <visual>
         <geometry>
-          <mesh filename="package://up1_description/meshes/finger.stl" scale="0.001 0.001 0.001" />
+          <mesh filename="package://up1_description/meshes/dual_arm/finger.stl" scale="0.001 0.001 0.001" />
         </geometry>
         <material name="grey" />
@@ -23,5 +23,5 @@
       <collision>
         <geometry>
-          <mesh filename="package://up1_description/meshes/finger.stl" scale="0.001 0.001 0.001" />
+          <mesh filename="package://up1_description/meshes/dual_arm/finger.stl" scale="0.001 0.001 0.001" />
         </geometry>
       </collision>
@@ -46,5 +46,5 @@
       <visual>
         <geometry>
-          <mesh filename="package://up1_description/meshes/finger.stl" scale="0.001 0.001 0.001" />
+          <mesh filename="package://up1_description/meshes/dual_arm/finger.stl" scale="0.001 0.001 0.001" />
         </geometry>
         <material name="grey" />
@@ -52,5 +52,5 @@
       <collision>
         <geometry>
-          <mesh filename="package://up1_description/meshes/finger.stl" scale="0.001 0.001 0.001" />
+          <mesh filename="package://up1_description/meshes/dual_arm/finger.stl" scale="0.001 0.001 0.001" />
         </geometry>
       </collision>

File: up1_description/xacro/dual_arm_module/left_arm_module.xacro (robot description, xacro)
@@ -1,7 +1,7 @@
 <?xml version="1.0"?>
 <robot xmlns:xacro="http://www.ros.org/wiki/xacro">
-  <xacro:include filename="$(find up1_description)/urdf/arm_module/arm.xacro" />
-  <xacro:include filename="$(find up1_description)/urdf/arm_module/gripper.xacro" />
-  <xacro:include filename="$(find up1_description)/urdf/arm_module/arm_module.gazebo.xacro" />
+  <xacro:include filename="$(find up1_description)/xacro/dual_arm_module/arm.xacro" />
+  <xacro:include filename="$(find up1_description)/xacro/dual_arm_module/gripper.xacro" />
+  <xacro:include filename="$(find up1_description)/xacro/dual_arm_module/arm_module.gazebo.xacro" />
   <!-- ============================   Arm Module   ============================ -->
   <xacro:macro name="left_arm_module">
@@ -16,5 +16,5 @@
       <visual>
         <geometry>
-          <mesh filename="package://up1_description/meshes/armroot.stl" scale="0.001 0.001 0.001" />
+          <mesh filename="package://up1_description/meshes/dual_arm/armroot.stl" scale="0.001 0.001 0.001" />
         </geometry>
         <material name="grey" />
@@ -22,5 +22,5 @@
       <collision>
         <geometry>
-          <mesh filename="package://up1_description/meshes/armroot.stl" scale="0.001 0.001 0.001" />
+          <mesh filename="package://up1_description/meshes/dual_arm/armroot.stl" scale="0.001 0.001 0.001" />
         </geometry>
       </collision>

File: up1_description/xacro/dual_arm_module/right_arm_module.xacro (robot description, xacro)
@@ -1,7 +1,7 @@
 <?xml version="1.0"?>
 <robot xmlns:xacro="http://www.ros.org/wiki/xacro">
-  <xacro:include filename="$(find up1_description)/urdf/arm_module/arm.xacro" />
-  <xacro:include filename="$(find up1_description)/urdf/arm_module/gripper.xacro" />
-  <xacro:include filename="$(find up1_description)/urdf/arm_module/arm_module.gazebo.xacro" />
+  <xacro:include filename="$(find up1_description)/xacro/dual_arm_module/arm.xacro" />
+  <xacro:include filename="$(find up1_description)/xacro/dual_arm_module/gripper.xacro" />
+  <xacro:include filename="$(find up1_description)/xacro/dual_arm_module/arm_module.gazebo.xacro" />
   <!-- ============================   Arm Module   ============================ -->
   <xacro:macro name="right_arm_module">
@@ -16,5 +16,5 @@
       <visual>
         <geometry>
-          <mesh filename="package://up1_description/meshes/armroot.stl" scale="0.001 0.001 0.001" />
+          <mesh filename="package://up1_description/meshes/dual_arm/armroot.stl" scale="0.001 0.001 0.001" />
         </geometry>
         <material name="grey" />
@@ -22,5 +22,5 @@
       <collision>
         <geometry>
-          <mesh filename="package://up1_description/meshes/armroot.stl" scale="0.001 0.001 0.001" />
+          <mesh filename="package://up1_description/meshes/dual_arm/armroot.stl" scale="0.001 0.001 0.001" />
         </geometry>
       </collision>

File: up1_description/xacro/dual_arm_module/two_arm_module.xacro (robot description, xacro)
@@ -1,7 +1,7 @@
 <?xml version="1.0"?>
 <robot xmlns:xacro="http://www.ros.org/wiki/xacro">
-  <xacro:include filename="$(find up1_description)/urdf/dual_arm_module/arm.xacro" />
-  <xacro:include filename="$(find up1_description)/urdf/dual_arm_module/gripper.xacro" />
-  <xacro:include filename="$(find up1_description)/urdf/dual_arm_module/arm_module.gazebo.xacro" />
+  <xacro:include filename="$(find up1_description)/xacro/dual_arm_module/arm.xacro" />
+  <xacro:include filename="$(find up1_description)/xacro/dual_arm_module/gripper.xacro" />
+  <xacro:include filename="$(find up1_description)/xacro/dual_arm_module/arm_module.gazebo.xacro" />
   <!-- ============================   Arm Module   ============================ -->
   <xacro:macro name="two_arm_module">
@@ -16,5 +16,5 @@
       <visual>
         <geometry>
-          <mesh filename="package://up1_description/meshes/armroot.stl" scale="0.001 0.001 0.001" />
+          <mesh filename="package://up1_description/meshes/dual_arm/armroot.stl" scale="0.001 0.001 0.001" />
         </geometry>
         <material name="grey" />
@@ -22,5 +22,5 @@
       <collision>
         <geometry>
-          <mesh filename="package://up1_description/meshes/armroot.stl" scale="0.001 0.001 0.001" />
+          <mesh filename="package://up1_description/meshes/dual_arm/armroot.stl" scale="0.001 0.001 0.001" />
         </geometry>
       </collision>

File: up1_description/xacro/io_module/camera.xacro (robot description, xacro)
@@ -13,5 +13,5 @@
       <visual>
         <geometry>
-          <mesh filename="package://up1_description/meshes/camera.stl" scale="0.001 0.001 0.001" />
+          <mesh filename="package://up1_description/meshes/io/camera.stl" scale="0.001 0.001 0.001" />
         </geometry>
         <material name="black" />
@@ -19,5 +19,5 @@
       <collision>
         <geometry>
-          <mesh filename="package://up1_description/meshes/camera.stl" scale="0.001 0.001 0.001" />
+          <mesh filename="package://up1_description/meshes/io/camera.stl" scale="0.001 0.001 0.001" />
         </geometry>
       </collision>

File: up1_description/xacro/io_module/io_module.xacro (robot description, xacro)
@@ -1,6 +1,6 @@
 <?xml version="1.0"?>
 <robot xmlns:xacro="http://www.ros.org/wiki/xacro">
-  <xacro:include filename="$(find up1_description)/urdf/io_module/camera.xacro" />
-  <xacro:include filename="$(find up1_description)/urdf/io_module/io_module.gazebo.xacro" />
+  <xacro:include filename="$(find up1_description)/xacro/io_module/camera.xacro" />
+  <xacro:include filename="$(find up1_description)/xacro/io_module/io_module.gazebo.xacro" />
   <!-- ============================   IO Module   ============================ -->
   <xacro:macro name="io_module">
@@ -15,5 +15,5 @@
       <visual>
         <geometry>
-          <mesh filename="package://up1_description/meshes/io.stl" scale="0.001 0.001 0.001" />
+          <mesh filename="package://up1_description/meshes/io/io.stl" scale="0.001 0.001 0.001" />
         </geometry>
         <material name="grey" />
@@ -21,5 +21,5 @@
       <collision>
         <geometry>
-          <mesh filename="package://up1_description/meshes/io.stl" scale="0.001 0.001 0.001" />
+          <mesh filename="package://up1_description/meshes/io/io.stl" scale="0.001 0.001 0.001" />
         </geometry>
       </collision>

File: up1_description/xacro/mono_arm_module/arm.xacro (robot description, xacro)
@@ -1,5 +1,5 @@
 <?xml version="1.0"?>
 <robot xmlns:xacro="http://www.ros.org/wiki/xacro">
-  <xacro:include filename="$(find up1_description)/urdf/arm_module/arm.gazebo.xacro" />
+  <xacro:include filename="$(find up1_description)/xacro/mono_arm_module/arm.gazebo.xacro" />
   <!-- ============================   Arm   ============================ -->
   <xacro:macro name="arm" params="prefix reflect">
@@ -17,5 +17,5 @@
       <visual>
         <geometry>
-          <mesh filename="package://up1_description/meshes/armlink1.stl" scale="0.001 0.001 0.001" />
+          <mesh filename="package://up1_description/meshes/mono_arm/armlink1.stl" scale="0.001 0.001 0.001" />
         </geometry>
         <material name="white" />
@@ -23,5 +23,5 @@
       <collision>
         <geometry>
-          <mesh filename="package://up1_description/meshes/armlink1.stl" scale="0.001 0.001 0.001" />
+          <mesh filename="package://up1_description/meshes/mono_arm/armlink1.stl" scale="0.001 0.001 0.001" />
         </geometry>
       </collision>
@@ -45,5 +45,5 @@
       <visual>
         <geometry>
-          <mesh filename="package://up1_description/meshes/armlink2.stl" scale="0.001 0.001 0.001" />
+          <mesh filename="package://up1_description/meshes/mono_arm/armlink2.stl" scale="0.001 0.001 0.001" />
         </geometry>
         <material name="white" />
@@ -51,5 +51,5 @@
       <collision>
         <geometry>
-          <mesh filename="package://up1_description/meshes/armlink2.stl" scale="0.001 0.001 0.001" />
+          <mesh filename="package://up1_description/meshes/mono_arm/armlink2.stl" scale="0.001 0.001 0.001" />
         </geometry>
       </collision>
@@ -73,5 +73,5 @@
       <visual>
         <geometry>
-          <mesh filename="package://up1_description/meshes/armlink3.stl" scale="0.001 0.001 0.001" />
+          <mesh filename="package://up1_description/meshes/mono_arm/armlink3.stl" scale="0.001 0.001 0.001" />
         </geometry>
         <material name="white" />
@@ -79,5 +79,5 @@
       <collision>
         <geometry>
-          <mesh filename="package://up1_description/meshes/armlink3.stl" scale="0.001 0.001 0.001" />
+          <mesh filename="package://up1_description/meshes/mono_arm/armlink3.stl" scale="0.001 0.001 0.001" />
         </geometry>
       </collision>
@@ -101,5 +101,5 @@
       <visual>
         <geometry>
-          <mesh filename="package://up1_description/meshes/armlink4.stl" scale="0.001 0.001 0.001" />
+          <mesh filename="package://up1_description/meshes/mono_arm/armlink4.stl" scale="0.001 0.001 0.001" />
         </geometry>
         <material name="white" />
@@ -107,5 +107,5 @@
       <collision>
         <geometry>
-          <mesh filename="package://up1_description/meshes/armlink4.stl" scale="0.001 0.001 0.001" />
+          <mesh filename="package://up1_description/meshes/mono_arm/armlink4.stl" scale="0.001 0.001 0.001" />
         </geometry>
       </collision>
@@ -129,5 +129,5 @@
       <visual>
         <geometry>
-          <mesh filename="package://up1_description/meshes/armlink5.stl" scale="0.001 0.001 0.001" />
+          <mesh filename="package://up1_description/meshes/mono_arm/armlink5.stl" scale="0.001 0.001 0.001" />
         </geometry>
         <material name="white" />
@@ -135,5 +135,5 @@
       <collision>
         <geometry>
-          <mesh filename="package://up1_description/meshes/armlink5.stl" scale="0.001 0.001 0.001" />
+          <mesh filename="package://up1_description/meshes/mono_arm/armlink5.stl" scale="0.001 0.001 0.001" />
         </geometry>
       </collision>

File: up1_description/xacro/mono_arm_module/gripper.xacro (robot description, xacro)
@@ -1,5 +1,5 @@
 <?xml version="1.0"?>
 <robot xmlns:xacro="http://www.ros.org/wiki/xacro">
-  <xacro:include filename="$(find up1_description)/urdf/arm_module/gripper.gazebo.xacro" />
+  <xacro:include filename="$(find up1_description)/xacro/mono_arm_module/gripper.gazebo.xacro" />
   <!-- ============================   Gripper   ============================ -->
   <xacro:macro name="gripper" params="prefix reflect">
@@ -17,5 +17,5 @@
       <visual>
         <geometry>
-          <mesh filename="package://up1_description/meshes/finger.stl" scale="0.001 0.001 0.001" />
+          <mesh filename="package://up1_description/meshes/mono_arm/finger.stl" scale="0.001 0.001 0.001" />
         </geometry>
         <material name="grey" />
@@ -23,5 +23,5 @@
       <collision>
         <geometry>
-          <mesh filename="package://up1_description/meshes/finger.stl" scale="0.001 0.001 0.001" />
+          <mesh filename="package://up1_description/meshes/mono_arm/finger.stl" scale="0.001 0.001 0.001" />
         </geometry>
       </collision>
@@ -46,5 +46,5 @@
       <visual>
         <geometry>
-          <mesh filename="package://up1_description/meshes/finger.stl" scale="0.001 0.001 0.001" />
+          <mesh filename="package://up1_description/meshes/mono_arm/finger.stl" scale="0.001 0.001 0.001" />
         </geometry>
         <material name="grey" />
@@ -52,5 +52,5 @@
       <collision>
         <geometry>
-          <mesh filename="package://up1_description/meshes/finger.stl" scale="0.001 0.001 0.001" />
+          <mesh filename="package://up1_description/meshes/mono_arm/finger.stl" scale="0.001 0.001 0.001" />
         </geometry>
       </collision>

File: up1_description/xacro/mono_arm_module/left_arm_module.xacro (robot description, xacro)
@@ -1,7 +1,7 @@
 <?xml version="1.0"?>
 <robot xmlns:xacro="http://www.ros.org/wiki/xacro">
-  <xacro:include filename="$(find up1_description)/urdf/arm_module/arm.xacro" />
-  <xacro:include filename="$(find up1_description)/urdf/arm_module/gripper.xacro" />
-  <xacro:include filename="$(find up1_description)/urdf/arm_module/arm_module.gazebo.xacro" />
+  <xacro:include filename="$(find up1_description)/xacro/mono_arm_module/arm.xacro" />
+  <xacro:include filename="$(find up1_description)/xacro/mono_arm_module/gripper.xacro" />
+  <xacro:include filename="$(find up1_description)/xacro/mono_arm_module/arm_module.gazebo.xacro" />
   <!-- ============================   Arm Module   ============================ -->
   <xacro:macro name="left_arm_module">
@@ -16,5 +16,5 @@
       <visual>
         <geometry>
-          <mesh filename="package://up1_description/meshes/armroot.stl" scale="0.001 0.001 0.001" />
+          <mesh filename="package://up1_description/meshes/mono_arm/armroot.stl" scale="0.001 0.001 0.001" />
         </geometry>
         <material name="grey" />
@@ -22,5 +22,5 @@
       <collision>
         <geometry>
-          <mesh filename="package://up1_description/meshes/armroot.stl" scale="0.001 0.001 0.001" />
+          <mesh filename="package://up1_description/meshes/mono_arm/armroot.stl" scale="0.001 0.001 0.001" />
         </geometry>
       </collision>

File: up1_description/xacro/mono_arm_module/right_arm_module.xacro (robot description, xacro)
@@ -1,7 +1,7 @@
 <?xml version="1.0"?>
 <robot xmlns:xacro="http://www.ros.org/wiki/xacro">
-  <xacro:include filename="$(find up1_description)/urdf/arm_module/arm.xacro" />
-  <xacro:include filename="$(find up1_description)/urdf/arm_module/gripper.xacro" />
-  <xacro:include filename="$(find up1_description)/urdf/arm_module/arm_module.gazebo.xacro" />
+  <xacro:include filename="$(find up1_description)/xacro/mono_arm_module/arm.xacro" />
+  <xacro:include filename="$(find up1_description)/xacro/mono_arm_module/gripper.xacro" />
+  <xacro:include filename="$(find up1_description)/xacro/mono_arm_module/arm_module.gazebo.xacro" />
   <!-- ============================   Arm Module   ============================ -->
   <xacro:macro name="right_arm_module">
@@ -16,5 +16,5 @@
       <visual>
         <geometry>
-          <mesh filename="package://up1_description/meshes/armroot.stl" scale="0.001 0.001 0.001" />
+          <mesh filename="package://up1_description/meshes/mono_arm/armroot.stl" scale="0.001 0.001 0.001" />
         </geometry>
         <material name="grey" />
@@ -22,5 +22,5 @@
       <collision>
         <geometry>
-          <mesh filename="package://up1_description/meshes/armroot.stl" scale="0.001 0.001 0.001" />
+          <mesh filename="package://up1_description/meshes/mono_arm/armroot.stl" scale="0.001 0.001 0.001" />
         </geometry>
       </collision>
