Commit message: description: cleaned up xacro files and fixed paths

File: up1_description/xacro/mono_arm_module/two_arm_module.xacro (robot description, xacro)
@@ -1,7 +1,7 @@
 <?xml version="1.0"?>
 <robot xmlns:xacro="http://www.ros.org/wiki/xacro">
-  <xacro:include filename="$(find up1_description)/urdf/arm_module/arm.xacro" />
-  <xacro:include filename="$(find up1_description)/urdf/arm_module/gripper.xacro" />
-  <xacro:include filename="$(find up1_description)/urdf/arm_module/arm_module.gazebo.xacro" />
+  <xacro:include filename="$(find up1_description)/xacro/mono_arm_module/arm.xacro" />
+  <xacro:include filename="$(find up1_description)/xacro/mono_arm_module/gripper.xacro" />
+  <xacro:include filename="$(find up1_description)/xacro/mono_arm_module/arm_module.gazebo.xacro" />
   <!-- ============================   Arm Module   ============================ -->
   <xacro:macro name="two_arm_module">
@@ -16,5 +16,5 @@
       <visual>
         <geometry>
-          <mesh filename="package://up1_description/meshes/armroot.stl" scale="0.001 0.001 0.001" />
+          <mesh filename="package://up1_description/meshes/mono_arm/armroot.stl" scale="0.001 0.001 0.001" />
         </geometry>
         <material name="grey" />
@@ -22,5 +22,5 @@
       <collision>
         <geometry>
-          <mesh filename="package://up1_description/meshes/armroot.stl" scale="0.001 0.001 0.001" />
+          <mesh filename="package://up1_description/meshes/mono_arm/armroot.stl" scale="0.001 0.001 0.001" />
         </geometry>
       </collision>
