Commit message: description: rebuilt urdf and generated display files

File: up1_description/urdf/up1.urdf (robot description, URDF)
Before this commit: robot up1, 26 links, 25 joints
Links:
- link armroot_link: geometry collision mesh filename=package://up1_description/meshes/dual_arm/armroot.stl scale=0.001 0.001 0.001; visual mesh filename=package://up1_description/meshes/dual_arm/armroot.stl scale=0.001 0.001 0.001
- link base_link: geometry collision mesh filename=package://up1_description/meshes/base/base.stl scale=0.001 0.001 0.001; visual mesh filename=package://up1_description/meshes/base/base.stl scale=0.001 0.001 0.001
- link io_link: geometry collision mesh filename=package://up1_description/meshes/io/io.stl scale=0.001 0.001 0.001; visual mesh filename=package://up1_description/meshes/io/io.stl scale=0.001 0.001 0.001
- link left_armlink1: geometry collision mesh filename=package://up1_description/meshes/dual_arm/armlink1.stl scale=0.001 0.001 0.001; visual mesh filename=package://up1_description/meshes/dual_arm/armlink1.stl scale=0.001 0.001 0.001
- link left_armlink2: geometry collision mesh filename=package://up1_description/meshes/dual_arm/armlink2.stl scale=0.001 0.001 0.001; visual mesh filename=package://up1_description/meshes/dual_arm/armlink2.stl scale=0.001 0.001 0.001
- link left_armlink3: geometry collision mesh filename=package://up1_description/meshes/dual_arm/armlink3.stl scale=0.001 0.001 0.001; visual mesh filename=package://up1_description/meshes/dual_arm/armlink3.stl scale=0.001 0.001 0.001
- link left_armlink4: geometry collision mesh filename=package://up1_description/meshes/dual_arm/armlink4.stl scale=0.001 0.001 0.001; visual mesh filename=package://up1_description/meshes/dual_arm/armlink4.stl scale=0.001 0.001 0.001
- link left_armlink5: geometry collision mesh filename=package://up1_description/meshes/dual_arm/armlink5.stl scale=0.001 0.001 0.001; visual mesh filename=package://up1_description/meshes/dual_arm/armlink5.stl scale=0.001 0.001 0.001
- link left_back_wheel: geometry collision mesh filename=package://up1_description/meshes/base/wheel.stl scale=0.001 0.001 0.001; visual mesh filename=package://up1_description/meshes/base/wheel.stl scale=0.001 0.001 0.001
- link left_camera: geometry collision mesh filename=package://up1_description/meshes/io/camera.stl scale=0.001 0.001 0.001; visual mesh filename=package://up1_description/meshes/io/camera.stl scale=0.001 0.001 0.001
- link left_finger1: geometry collision mesh filename=package://up1_description/meshes/dual_arm/finger.stl scale=0.001 0.001 0.001; visual mesh filename=package://up1_description/meshes/dual_arm/finger.stl scale=0.001 0.001 0.001
- link left_finger2: geometry collision mesh filename=package://up1_description/meshes/dual_arm/finger.stl scale=0.001 0.001 0.001; visual mesh filename=package://up1_description/meshes/dual_arm/finger.stl scale=0.001 0.001 0.001
- link left_front_wheel: geometry collision mesh filename=package://up1_description/meshes/base/wheel.stl scale=0.001 0.001 0.001; visual mesh filename=package://up1_description/meshes/base/wheel.stl scale=0.001 0.001 0.001
- link right_armlink1: geometry collision mesh filename=package://up1_description/meshes/dual_arm/armlink1.stl scale=0.001 0.001 0.001; visual mesh filename=package://up1_description/meshes/dual_arm/armlink1.stl scale=0.001 0.001 0.001
- link right_armlink2: geometry collision mesh filename=package://up1_description/meshes/dual_arm/armlink2.stl scale=0.001 0.001 0.001; visual mesh filename=package://up1_description/meshes/dual_arm/armlink2.stl scale=0.001 0.001 0.001
- link right_armlink3: geometry collision mesh filename=package://up1_description/meshes/dual_arm/armlink3.stl scale=0.001 0.001 0.001; visual mesh filename=package://up1_description/meshes/dual_arm/armlink3.stl scale=0.001 0.001 0.001
- link right_armlink4: geometry collision mesh filename=package://up1_description/meshes/dual_arm/armlink4.stl scale=0.001 0.001 0.001; visual mesh filename=package://up1_description/meshes/dual_arm/armlink4.stl scale=0.001 0.001 0.001
- link right_armlink5: geometry collision mesh filename=package://up1_description/meshes/dual_arm/armlink5.stl scale=0.001 0.001 0.001; visual mesh filename=package://up1_description/meshes/dual_arm/armlink5.stl scale=0.001 0.001 0.001
- link right_back_wheel: geometry collision mesh filename=package://up1_description/meshes/base/wheel.stl scale=0.001 0.001 0.001; visual mesh filename=package://up1_description/meshes/base/wheel.stl scale=0.001 0.001 0.001
- link right_camera: geometry collision mesh filename=package://up1_description/meshes/io/camera.stl scale=0.001 0.001 0.001; visual mesh filename=package://up1_description/meshes/io/camera.stl scale=0.001 0.001 0.001
- link right_finger1: geometry collision mesh filename=package://up1_description/meshes/dual_arm/finger.stl scale=0.001 0.001 0.001; visual mesh filename=package://up1_description/meshes/dual_arm/finger.stl scale=0.001 0.001 0.001
- link right_finger2: geometry collision mesh filename=package://up1_description/meshes/dual_arm/finger.stl scale=0.001 0.001 0.001; visual mesh filename=package://up1_description/meshes/dual_arm/finger.stl scale=0.001 0.001 0.001
- link right_front_wheel: geometry collision mesh filename=package://up1_description/meshes/base/wheel.stl scale=0.001 0.001 0.001; visual mesh filename=package://up1_description/meshes/base/wheel.stl scale=0.001 0.001 0.001

File: up1_description/urdf/up1_left_arm.urdf (robot description, URDF)
Before this commit: robot up1, 18 links, 17 joints
Links:
- link armroot_link: geometry collision mesh filename=package://up1_description/meshes/dual_arm/armroot.stl scale=0.001 0.001 0.001; visual mesh filename=package://up1_description/meshes/dual_arm/armroot.stl scale=0.001 0.001 0.001
- link base_link: geometry collision mesh filename=package://up1_description/meshes/base/base.stl scale=0.001 0.001 0.001; visual mesh filename=package://up1_description/meshes/base/base.stl scale=0.001 0.001 0.001
- link io_link: geometry collision mesh filename=package://up1_description/meshes/io/io.stl scale=0.001 0.001 0.001; visual mesh filename=package://up1_description/meshes/io/io.stl scale=0.001 0.001 0.001
- link left_armlink1: geometry collision mesh filename=package://up1_description/meshes/dual_arm/armlink1.stl scale=0.001 0.001 0.001; visual mesh filename=package://up1_description/meshes/dual_arm/armlink1.stl scale=0.001 0.001 0.001
- link left_armlink2: geometry collision mesh filename=package://up1_description/meshes/dual_arm/armlink2.stl scale=0.001 0.001 0.001; visual mesh filename=package://up1_description/meshes/dual_arm/armlink2.stl scale=0.001 0.001 0.001
- link left_armlink3: geometry collision mesh filename=package://up1_description/meshes/dual_arm/armlink3.stl scale=0.001 0.001 0.001; visual mesh filename=package://up1_description/meshes/dual_arm/armlink3.stl scale=0.001 0.001 0.001
- link left_armlink4: geometry collision mesh filename=package://up1_description/meshes/dual_arm/armlink4.stl scale=0.001 0.001 0.001; visual mesh filename=package://up1_description/meshes/dual_arm/armlink4.stl scale=0.001 0.001 0.001
- link left_armlink5: geometry collision mesh filename=package://up1_description/meshes/dual_arm/armlink5.stl scale=0.001 0.001 0.001; visual mesh filename=package://up1_description/meshes/dual_arm/armlink5.stl scale=0.001 0.001 0.001
- link left_back_wheel: geometry collision mesh filename=package://up1_description/meshes/base/wheel.stl scale=0.001 0.001 0.001; visual mesh filename=package://up1_description/meshes/base/wheel.stl scale=0.001 0.001 0.001
- link left_camera: geometry collision mesh filename=package://up1_description/meshes/io/camera.stl scale=0.001 0.001 0.001; visual mesh filename=package://up1_description/meshes/io/camera.stl scale=0.001 0.001 0.001
- link left_finger1: geometry collision mesh filename=package://up1_description/meshes/dual_arm/finger.stl scale=0.001 0.001 0.001; visual mesh filename=package://up1_description/meshes/dual_arm/finger.stl scale=0.001 0.001 0.001
- link left_finger2: geometry collision mesh filename=package://up1_description/meshes/dual_arm/finger.stl scale=0.001 0.001 0.001; visual mesh filename=package://up1_description/meshes/dual_arm/finger.stl scale=0.001 0.001 0.001
- link left_front_wheel: geometry collision mesh filename=package://up1_description/meshes/base/wheel.stl scale=0.001 0.001 0.001; visual mesh filename=package://up1_description/meshes/base/wheel.stl scale=0.001 0.001 0.001
- link right_back_wheel: geometry collision mesh filename=package://up1_description/meshes/base/wheel.stl scale=0.001 0.001 0.001; visual mesh filename=package://up1_description/meshes/base/wheel.stl scale=0.001 0.001 0.001
- link right_camera: geometry collision mesh filename=package://up1_description/meshes/io/camera.stl scale=0.001 0.001 0.001; visual mesh filename=package://up1_description/meshes/io/camera.stl scale=0.001 0.001 0.001
- link right_front_wheel: geometry collision mesh filename=package://up1_description/meshes/base/wheel.stl scale=0.001 0.001 0.001; visual mesh filename=package://up1_description/meshes/base/wheel.stl scale=0.001 0.001 0.001

File: up1_description/urdf/up1_right_arm.urdf (robot description, URDF)
Before this commit: robot up1, 18 links, 17 joints
Links:
- link armroot_link: geometry collision mesh filename=package://up1_description/meshes/dual_arm/armroot.stl scale=0.001 0.001 0.001; visual mesh filename=package://up1_description/meshes/dual_arm/armroot.stl scale=0.001 0.001 0.001
- link base_link: geometry collision mesh filename=package://up1_description/meshes/base/base.stl scale=0.001 0.001 0.001; visual mesh filename=package://up1_description/meshes/base/base.stl scale=0.001 0.001 0.001
- link io_link: geometry collision mesh filename=package://up1_description/meshes/io/io.stl scale=0.001 0.001 0.001; visual mesh filename=package://up1_description/meshes/io/io.stl scale=0.001 0.001 0.001
- link left_back_wheel: geometry collision mesh filename=package://up1_description/meshes/base/wheel.stl scale=0.001 0.001 0.001; visual mesh filename=package://up1_description/meshes/base/wheel.stl scale=0.001 0.001 0.001
- link left_camera: geometry collision mesh filename=package://up1_description/meshes/io/camera.stl scale=0.001 0.001 0.001; visual mesh filename=package://up1_description/meshes/io/camera.stl scale=0.001 0.001 0.001
- link left_front_wheel: geometry collision mesh filename=package://up1_description/meshes/base/wheel.stl scale=0.001 0.001 0.001; visual mesh filename=package://up1_description/meshes/base/wheel.stl scale=0.001 0.001 0.001
- link right_armlink1: geometry collision mesh filename=package://up1_description/meshes/dual_arm/armlink1.stl scale=0.001 0.001 0.001; visual mesh filename=package://up1_description/meshes/dual_arm/armlink1.stl scale=0.001 0.001 0.001
- link right_armlink2: geometry collision mesh filename=package://up1_description/meshes/dual_arm/armlink2.stl scale=0.001 0.001 0.001; visual mesh filename=package://up1_description/meshes/dual_arm/armlink2.stl scale=0.001 0.001 0.001
- link right_armlink3: geometry collision mesh filename=package://up1_description/meshes/dual_arm/armlink3.stl scale=0.001 0.001 0.001; visual mesh filename=package://up1_description/meshes/dual_arm/armlink3.stl scale=0.001 0.001 0.001
- link right_armlink4: geometry collision mesh filename=package://up1_description/meshes/dual_arm/armlink4.stl scale=0.001 0.001 0.001; visual mesh filename=package://up1_description/meshes/dual_arm/armlink4.stl scale=0.001 0.001 0.001
- link right_armlink5: geometry collision mesh filename=package://up1_description/meshes/dual_arm/armlink5.stl scale=0.001 0.001 0.001; visual mesh filename=package://up1_description/meshes/dual_arm/armlink5.stl scale=0.001 0.001 0.001
- link right_back_wheel: geometry collision mesh filename=package://up1_description/meshes/base/wheel.stl scale=0.001 0.001 0.001; visual mesh filename=package://up1_description/meshes/base/wheel.stl scale=0.001 0.001 0.001
- link right_camera: geometry collision mesh filename=package://up1_description/meshes/io/camera.stl scale=0.001 0.001 0.001; visual mesh filename=package://up1_description/meshes/io/camera.stl scale=0.001 0.001 0.001
- link right_finger1: geometry collision mesh filename=package://up1_description/meshes/dual_arm/finger.stl scale=0.001 0.001 0.001; visual mesh filename=package://up1_description/meshes/dual_arm/finger.stl scale=0.001 0.001 0.001
- link right_finger2: geometry collision mesh filename=package://up1_description/meshes/dual_arm/finger.stl scale=0.001 0.001 0.001; visual mesh filename=package://up1_description/meshes/dual_arm/finger.stl scale=0.001 0.001 0.001
- link right_front_wheel: geometry collision mesh filename=package://up1_description/meshes/base/wheel.stl scale=0.001 0.001 0.001; visual mesh filename=package://up1_description/meshes/base/wheel.stl scale=0.001 0.001 0.001
