Commit message: description: fixed more renames for armlink5 to gripper and gripper to finger

File: up1_description/urdf/common.xacro (robot description, xacro)
@@ -30,9 +30,6 @@
   <xacro:property name="armlink4_offset_y" value="0" />
   <xacro:property name="armlink4_offset_z" value="0.05588" />
-  <xacro:property name="armlink5_offset_x" value="0" />
-  <xacro:property name="armlink5_offset_y" value="0.07641" />
-  <xacro:property name="armlink5_offset_z" value="0" />
   <xacro:property name="gripper_offset_x" value="0" />
-  <xacro:property name="gripper_offset_y" value="0.138" />
+  <xacro:property name="gripper_offset_y" value="0.07641" />
   <xacro:property name="gripper_offset_z" value="0" />
   <xacro:property name="finger_offset_x" value="0.01800" />
@@ -47,6 +44,6 @@
   <xacro:property name="armlink4_limit_lower" value="${-pi/2}" />
   <xacro:property name="armlink4_limit_upper" value="${pi/2}" />
-  <xacro:property name="armlink5_limit_lower" value="${-pi/2}" />
-  <xacro:property name="armlink5_limit_upper" value="${pi/2}" />
+  <xacro:property name="gripper_limit_lower" value="${-pi/2}" />
+  <xacro:property name="gripper_limit_upper" value="${pi/2}" />
   <xacro:property name="finger_limit_upper" value="0.018" />
   <xacro:property name="armlink1_velocity" value="1" />
@@ -54,5 +51,5 @@
   <xacro:property name="armlink3_velocity" value="1" />
   <xacro:property name="armlink4_velocity" value="1" />
-  <xacro:property name="armlink5_velocity" value="1" />
+  <xacro:property name="gripper_velocity" value="1" />
   <xacro:property name="finger1_velocity" value="1" />
   <xacro:property name="finger2_velocity" value="1" />
@@ -61,5 +58,5 @@
   <xacro:property name="armlink3_effort" value="6.0" />
   <xacro:property name="armlink4_effort" value="6.0" />
-  <xacro:property name="armlink5_effort" value="6.0" />
+  <xacro:property name="gripper_effort" value="6.0" />
   <xacro:property name="finger1_effort" value="6.0" />
   <xacro:property name="finger2_effort" value="6.0" />

File: up1_description/urdf/manipulator_module/dual_arm_module/arm.gazebo.xacro (robot description, xacro)
@@ -15,5 +15,5 @@
       <turnGravityOff>true</turnGravityOff>
     </gazebo>
-    <gazebo reference="${prefix}_armlink5">
+    <gazebo reference="${prefix}_gripper">
       <turnGravityOff>true</turnGravityOff>
     </gazebo>

File: up1_description/urdf/manipulator_module/dual_arm_module/arm.transmission.xacro (robot description, xacro)
@@ -39,10 +39,10 @@
       </actuator>
     </transmission>
-    <transmission name="${prefix}_armlink4_to_armlink5_trans">
+    <transmission name="${prefix}_armlink4_to_gripper_trans">
       <type>transmission_interface/SimpleTransmission</type>
-      <joint name="${prefix}_armlink4_to_armlink5">
+      <joint name="${prefix}_armlink4_to_gripper">
         <hardwareInterface>PositionJointInterface</hardwareInterface>
       </joint>
-      <actuator name="${prefix}_armlink4_to_armlink5_motor">
+      <actuator name="${prefix}_armlink4_to_gripper_motor">
         <mechanicalReduction>1</mechanicalReduction>
       </actuator>

File: up1_description/urdf/manipulator_module/dual_arm_module/arm.xacro (robot description, xacro)
@@ -122,7 +122,7 @@
       <child link="${prefix}_gripper" />
       <origin rpy="0 ${pi/2} 0"
-        xyz="${armlink5_offset_x} ${armlink5_offset_y} ${armlink5_offset_z}" />
+        xyz="${gripper_offset_x} ${gripper_offset_y} ${gripper_offset_z}" />
       <axis xyz="0 0 ${-reflect*1}" />
-      <limit lower="${armlink5_limit_lower}" upper="${armlink5_limit_upper}" velocity="${armlink5_velocity}" effort="${armlink5_effort}" />
+      <limit lower="${gripper_limit_lower}" upper="${gripper_limit_upper}" velocity="${gripper_velocity}" effort="${gripper_effort}" />
     </joint>
     <!-- Gripper Link -->

File: up1_description/urdf/manipulator_module/dual_arm_module/gripper.transmission.xacro (robot description, xacro)
@@ -5,5 +5,5 @@
     <transmission name="${prefix}_gripper_trans">
       <type>transmission_interface/SimpleTransmission</type>
-      <joint name="${prefix}_gripper_joint">
+      <joint name="${prefix}_finger_joint">
         <hardwareInterface>PositionJointInterface</hardwareInterface>
       </joint>
@@ -14,5 +14,5 @@
     <transmission name="${prefix}_gripper_trans">
       <type>transmission_interface/SimpleTransmission</type>
-      <joint name="${prefix}_gripper_joint_fake">
+      <joint name="${prefix}_finger_joint_fake">
         <hardwareInterface>PositionJointInterface</hardwareInterface>
       </joint>

Commit message: description: moved dual arm properties out of common

File: up1_description/urdf/common.xacro (robot description, xacro)
@@ -15,50 +15,4 @@
   <xacro:property name="camera_offset_y" value="0.04027" />
   <xacro:property name="camera_offset_z" value="0.00023" />
-  <xacro:property name="armroot_offset_x" value="-0.01247" />
-  <xacro:property name="armroot_offset_y" value="0" />
-  <xacro:property name="armroot_offset_z" value="0.05187" />
-  <xacro:property name="armlink1_offset_x" value="0.01777" />
-  <xacro:property name="armlink1_offset_y" value="0.07385" />
-  <xacro:property name="armlink1_offset_z" value="0.01853" />
-  <xacro:property name="armlink2_offset_x" value="0" />
-  <xacro:property name="armlink2_offset_y" value="0" />
-  <xacro:property name="armlink2_offset_z" value="-0.07038" />
-  <xacro:property name="armlink3_offset_x" value="0" />
-  <xacro:property name="armlink3_offset_y" value="0.09602" />
-  <xacro:property name="armlink3_offset_z" value="0" />
-  <xacro:property name="armlink4_offset_x" value="0" />
-  <xacro:property name="armlink4_offset_y" value="0" />
-  <xacro:property name="armlink4_offset_z" value="0.05588" />
-  <xacro:property name="gripper_offset_x" value="0" />
-  <xacro:property name="gripper_offset_y" value="0.07641" />
-  <xacro:property name="gripper_offset_z" value="0" />
-  <xacro:property name="finger_offset_x" value="0.01800" />
-  <xacro:property name="finger_offset_y" value="0.08121" />
-  <xacro:property name="finger_offset_z" value="0" />
-  <xacro:property name="armlink1_limit_lower" value="${-pi/2}" />
-  <xacro:property name="armlink1_limit_upper" value="${pi/2}" />
-  <xacro:property name="armlink2_limit_lower" value="${-pi/2}" />
-  <xacro:property name="armlink2_limit_upper" value="${pi/2}" />
-  <xacro:property name="armlink3_limit_lower" value="${-pi/2}" />
-  <xacro:property name="armlink3_limit_upper" value="${pi/2}" />
-  <xacro:property name="armlink4_limit_lower" value="${-pi/2}" />
-  <xacro:property name="armlink4_limit_upper" value="${pi/2}" />
-  <xacro:property name="gripper_limit_lower" value="${-pi/2}" />
-  <xacro:property name="gripper_limit_upper" value="${pi/2}" />
-  <xacro:property name="finger_limit_upper" value="0.018" />
-  <xacro:property name="armlink1_velocity" value="1" />
-  <xacro:property name="armlink2_velocity" value="1" />
-  <xacro:property name="armlink3_velocity" value="1" />
-  <xacro:property name="armlink4_velocity" value="1" />
-  <xacro:property name="gripper_velocity" value="1" />
-  <xacro:property name="finger1_velocity" value="1" />
-  <xacro:property name="finger2_velocity" value="1" />
-  <xacro:property name="armlink1_effort" value="6.0" />
-  <xacro:property name="armlink2_effort" value="6.0" />
-  <xacro:property name="armlink3_effort" value="6.0" />
-  <xacro:property name="armlink4_effort" value="6.0" />
-  <xacro:property name="gripper_effort" value="6.0" />
-  <xacro:property name="finger1_effort" value="6.0" />
-  <xacro:property name="finger2_effort" value="6.0" />
   <material name="black">
     <color rgba="0 0 0 1" />

File: up1_description/urdf/manipulator_module/dual_arm_module/arm.xacro (robot description, xacro)
@@ -3,4 +3,44 @@
   <xacro:include filename="$(find up1_description)/urdf/manipulator_module/dual_arm_module/arm.gazebo.xacro" />
   <xacro:include filename="$(find up1_description)/urdf/manipulator_module/dual_arm_module/arm.transmission.xacro" />
+  <xacro:property name="armlink1_offset_x" value="0.01777" />
+  <xacro:property name="armlink1_offset_y" value="0.07385" />
+  <xacro:property name="armlink1_offset_z" value="0.01853" />
+  <xacro:property name="armlink2_offset_x" value="0" />
+  <xacro:property name="armlink2_offset_y" value="0" />
+  <xacro:property name="armlink2_offset_z" value="-0.07038" />
+  <xacro:property name="armlink3_offset_x" value="0" />
+  <xacro:property name="armlink3_offset_y" value="0.09602" />
+  <xacro:property name="armlink3_offset_z" value="0" />
+  <xacro:property name="armlink4_offset_x" value="0" />
+  <xacro:property name="armlink4_offset_y" value="0" />
+  <xacro:property name="armlink4_offset_z" value="0.05588" />
+  <xacro:property name="gripper_offset_x" value="0" />
+  <xacro:property name="gripper_offset_y" value="0.07641" />
+  <xacro:property name="gripper_offset_z" value="0" />
+  <xacro:property name="armlink1_limit_lower" value="${-pi/2}" />
+  <xacro:property name="armlink1_limit_upper" value="${pi/2}" />
+  <xacro:property name="armlink2_limit_lower" value="${-pi/2}" />
+  <xacro:property name="armlink2_limit_upper" value="${pi/2}" />
+  <xacro:property name="armlink3_limit_lower" value="${-pi/2}" />
+  <xacro:property name="armlink3_limit_upper" value="${pi/2}" />
+  <xacro:property name="armlink4_limit_lower" value="${-pi/2}" />
+  <xacro:property name="armlink4_limit_upper" value="${pi/2}" />
+  <xacro:property name="gripper_limit_lower" value="${-pi/2}" />
+  <xacro:property name="gripper_limit_upper" value="${pi/2}" />
+  <xacro:property name="finger_limit_upper" value="0.018" />
+  <xacro:property name="armlink1_velocity" value="1" />
+  <xacro:property name="armlink2_velocity" value="1" />
+  <xacro:property name="armlink3_velocity" value="1" />
+  <xacro:property name="armlink4_velocity" value="1" />
+  <xacro:property name="gripper_velocity" value="1" />
+  <xacro:property name="finger1_velocity" value="1" />
+  <xacro:property name="finger2_velocity" value="1" />
+  <xacro:property name="armlink1_effort" value="6.0" />
+  <xacro:property name="armlink2_effort" value="6.0" />
+  <xacro:property name="armlink3_effort" value="6.0" />
+  <xacro:property name="armlink4_effort" value="6.0" />
+  <xacro:property name="gripper_effort" value="6.0" />
+  <xacro:property name="finger1_effort" value="6.0" />
+  <xacro:property name="finger2_effort" value="6.0" />
   <xacro:macro name="arm" params="prefix reflect">
     <!-- ============================   Arm   ============================ -->

File: up1_description/urdf/manipulator_module/dual_arm_module/arm_root_link.xacro (robot description, xacro)
@@ -1,4 +1,7 @@
 <?xml version="1.0"?>
 <robot xmlns:xacro="http://www.ros.org/wiki/xacro" name="up1">
+  <xacro:property name="armroot_offset_x" value="-0.01247" />
+  <xacro:property name="armroot_offset_y" value="0" />
+  <xacro:property name="armroot_offset_z" value="0.05187" />
   <xacro:macro name="arm_root_link">
     <!-- ============================   Arm Root Link   ============================ -->

File: up1_description/urdf/manipulator_module/dual_arm_module/gripper.xacro (robot description, xacro)
@@ -3,4 +3,7 @@
   <xacro:include filename="$(find up1_description)/urdf/manipulator_module/dual_arm_module/gripper.gazebo.xacro" />
   <xacro:include filename="$(find up1_description)/urdf/manipulator_module/dual_arm_module/gripper.transmission.xacro" />
+  <xacro:property name="finger_offset_x" value="0.01800" />
+  <xacro:property name="finger_offset_y" value="0.08121" />
+  <xacro:property name="finger_offset_z" value="0" />
   <xacro:macro name="gripper" params="prefix reflect">
     <!-- ============================   Gripper   ============================ -->
