Commit message: description: updated urdf

File: up1_description/urdf/up1_mono.urdf (robot description, URDF)
Before this commit: robot up1, 17 links, 16 joints
Links:
- link left_camera: geometry collision mesh filename=package://up1_description/meshes/io/camera.dae scale=0.001 0.001 0.001; visual mesh filename=package://up1_description/meshes/io/camera.dae scale=0.001 0.001 0.001
- link right_camera: geometry collision mesh filename=package://up1_description/meshes/io/camera.dae scale=0.001 0.001 0.001; visual mesh filename=package://up1_description/meshes/io/camera.dae scale=0.001 0.001 0.001
