Commit message: description: initial tests for mono arm

File: up1_description/xacro/mono_arm_module/arm.xacro (robot description, xacro)
@@ -8,6 +8,5 @@
       <parent link="armroot_link" />
       <child link="${prefix}_armlink1" />
-      <origin rpy="${-reflect*pi/6} ${pi} 0"
-        xyz="${armlink1_offset_x} ${-reflect*armlink1_offset_y} ${armlink1_offset_z}" />
+      <origin rpy="0 0 0" xyz="0 0 0" />
       <axis xyz="0 0 1" />
       <limit lower="${armlink1_limit_lower}" upper="${armlink1_limit_upper}" velocity="${armlink1_velocity}" effort="${armlink1_effort}" />
@@ -27,5 +26,6 @@
       </collision>
       <inertial>
-        <mass value="0.06985"/>
+        <mass value="0.17905"/>
+        <!-- inertia is wrong, get update from Daniel -->
         <inertia ixx="0.00023448766" ixy="0.0000000027" ixz="0.00000001913"
                  iyy="0.00024004726" iyz="-0.0000015393" izz="0.00007431363"/>
@@ -36,6 +36,5 @@
       <parent link="${prefix}_armlink1" />
       <child link="${prefix}_armlink2" />
-      <origin rpy="${pi/2} ${pi} 0"
-        xyz="${armlink2_offset_x} ${armlink2_offset_y} ${armlink2_offset_z}" />
+      <origin rpy="0 0 0" xyz="0 0 0" />
       <axis xyz="0 0 ${reflect*1}" />
       <limit lower="${armlink2_limit_lower}" upper="${armlink2_limit_upper}" velocity="${armlink2_velocity}" effort="${armlink2_effort}" />
@@ -55,5 +54,6 @@
       </collision>
       <inertial>
-        <mass value="0.07067"/>
+        <mass value="0.49779"/>
+        <!-- inertia is wrong, get update from Daniel -->
         <inertia ixx="0.00029708797" ixy="-0.00000000444" ixz="0.00000000068"
                  iyy="0.0000799845" iyz="-0.00000174097" izz="0.00026073683"/>
@@ -64,6 +64,5 @@
       <parent link="${prefix}_armlink2" />
       <child link="${prefix}_armlink3" />
-      <origin rpy="${-pi/2} ${pi} 0"
-        xyz="${armlink3_offset_x} ${armlink3_offset_y} ${armlink3_offset_z}" />
+      <origin rpy="0 0 0" xyz="0 0 0" />
       <axis xyz="0 0 -1" />
       <limit lower="${armlink3_limit_lower}" upper="${armlink3_limit_upper}" velocity="${armlink3_velocity}" effort="${armlink3_effort}" />
@@ -92,6 +91,5 @@
       <parent link="${prefix}_armlink3" />
       <child link="${prefix}_armlink4" />
-      <origin rpy="${pi/2} 0 0"
-        xyz="${armlink4_offset_x} ${armlink4_offset_y} ${armlink4_offset_z}" />
+      <origin rpy="0 0 0" xyz="0 0 0" />
       <axis xyz="0 0 ${reflect*1}" />
       <limit lower="${armlink4_limit_lower}" upper="${armlink4_limit_upper}" velocity="${armlink4_velocity}" effort="${armlink4_effort}" />
@@ -120,6 +118,5 @@
       <parent link="${prefix}_armlink4" />
       <child link="${prefix}_armlink5" />
-      <origin rpy="0 ${pi/2} 0"
-        xyz="${armlink5_offset_x} ${armlink5_offset_y} ${armlink5_offset_z}" />
+      <origin rpy="0 0 0" xyz="0 0 0" />
       <axis xyz="0 0 ${-reflect*1}" />
       <limit lower="${armlink5_limit_lower}" upper="${armlink5_limit_upper}" velocity="${armlink5_velocity}" effort="${armlink5_effort}" />
@@ -148,6 +145,5 @@
       <parent link="${prefix}_armlink5" />
       <child link="${prefix}_gripper" />
-      <origin rpy="0 0 0"
-        xyz="${gripper_offset_x} ${gripper_offset_y} ${gripper_offset_z}" />
+      <origin rpy="0 0 0" xyz="0 0 0" />
     </joint>
     <!-- Gripper -->

File: up1_description/xacro/mono_arm_module/mono_arm_module.xacro (robot description, xacro)
@@ -5,10 +5,10 @@
   <xacro:include filename="$(find up1_description)/xacro/mono_arm_module/arm_module.gazebo.xacro" />
   <!-- ============================   Arm Module   ============================ -->
-  <xacro:macro name="left_arm_module">
+  <xacro:macro name="mono_arm_module">
     <!-- Armroot Joint -->
     <joint name="base_to_armroot" type="fixed">
       <parent link="base_link" />
       <child link="armroot_link" />
-      <origin xyz="${armroot_offset_x} ${armroot_offset_y} ${armroot_offset_z}" />
+      <origin xyz="0.003804 -0.008022 0.001964" />
     </joint>
     <!-- Armroot Link -->
@@ -26,5 +26,6 @@
       </collision>
       <inertial>
-        <mass value="0.20657"/>
+        <mass value="0.17621"/>
+        <!-- inertia is wrong, get update from Daniel -->
         <inertia ixx="0.00096240277" ixy="-0.00000350376" ixz="0.00002354169"
                  iyy="0.00057897825" iyz="0.00000127419" izz="0.00134814249"/>
@@ -32,6 +33,6 @@
     </link>
     <xacro:arm_module_gazebo />
-    <xacro:arm prefix="left" reflect="-1" />
-    <xacro:gripper prefix="left" reflect="-1" />
+    <xacro:arm prefix="mono" reflect="1" />
+    <xacro:gripper prefix="mono" reflect="1" />
   </xacro:macro>
 </robot>
