Commit message: control: added fake gripper controllers

File: up1_description/xacro/dual_arm_module/gripper.transmission.xacro (robot description, xacro)
@@ -12,4 +12,13 @@
       </actuator>
     </transmission>
+    <transmission name="${prefix}_gripper_trans">
+      <type>transmission_interface/SimpleTransmission</type>
+      <joint name="${prefix}_gripper_joint_fake">
+        <hardwareInterface>PositionJointInterface</hardwareInterface>
+      </joint>
+      <actuator name="${prefix}_gripper_motor">
+        <mechanicalReduction>1</mechanicalReduction>
+      </actuator>
+    </transmission>
   </xacro:macro>
 </robot>
