Commit message: description: replaced macro names with generic ones

File: up1_description/xacro/manipulator_module/dual_arm_module/two_arm_module.xacro (robot description, xacro)
@@ -7,5 +7,5 @@
   <xacro:include filename="$(find up1_description)/xacro/dual_arm_module/arm_module.gazebo.xacro" />
   <!-- ============================   Arm Module   ============================ -->
-  <xacro:macro name="two_arm_module">
+  <xacro:macro name="manipulator_module">
     <!-- Armroot Joint -->
     <joint name="base_to_armroot" type="fixed">

File: up1_description/xacro/manipulator_module/mono_arm_module/mono_arm_module.xacro (robot description, xacro)
@@ -5,5 +5,5 @@
   <xacro:include filename="$(find up1_description)/xacro/mono_arm_module/arm_module.gazebo.xacro" />
   <!-- ============================   Arm Module   ============================ -->
-  <xacro:macro name="mono_arm_module">
+  <xacro:macro name="manipulator_module">
     <!-- Armroot Joint -->
     <joint name="base_to_armroot" type="fixed">
