Commit message: description: fixed confusing comments in xacro files

File: up1_description/urdf/base_module/base_module.gazebo.xacro (robot description, xacro)
@@ -1,6 +1,6 @@
 <?xml version="1.0"?>
-<robot xmlns:xacro="http://www.ros.org/wiki/xacro">
-  <!-- ============================   Base Module   ============================ -->
+<robot xmlns:xacro="http://www.ros.org/wiki/xacro" name="up1">
   <xacro:macro name="base_module_gazebo">
+    <!-- ============================   Base Module Gazebo   ============================ -->
     <gazebo>
       <plugin name="skid_steer_drive_controller" filename="libgazebo_ros_skid_steer_drive.so">

File: up1_description/urdf/base_module/base_module.xacro (robot description, xacro)
@@ -1,8 +1,8 @@
 <?xml version="1.0"?>
-<robot xmlns:xacro="http://www.ros.org/wiki/xacro">
+<robot xmlns:xacro="http://www.ros.org/wiki/xacro" name="up1">
   <xacro:include filename="$(find up1_description)/urdf/base_module/wheel.xacro" />
   <xacro:include filename="$(find up1_description)/urdf/base_module/base_module.gazebo.xacro" />
-  <!-- ============================   Base Module   ============================ -->
   <xacro:macro name="base_module">
+    <!-- ============================   Base Module   ============================ -->
     <!-- base_footprint is a fictitious link(frame) that is on the ground right below base_link origin,
          navigation stack dedpends on this frame -->

File: up1_description/urdf/base_module/wheel.xacro (robot description, xacro)
@@ -1,6 +1,6 @@
 <?xml version="1.0"?>
-<robot xmlns:xacro="http://www.ros.org/wiki/xacro">
-  <!-- ============================   Wheel   ============================ -->
+<robot xmlns:xacro="http://www.ros.org/wiki/xacro" name="up1">
   <xacro:macro name="wheel" params="prefix reflect">
+    <!-- ============================   Wheel   ============================ -->
     <!-- Front Wheel Joint -->
     <joint name="base_to_${prefix}_front_wheel" type="continuous">

File: up1_description/urdf/io_module/camera.xacro (robot description, xacro)
@@ -1,6 +1,6 @@
 <?xml version="1.0"?>
-<robot xmlns:xacro="http://www.ros.org/wiki/xacro">
-  <!-- ============================   Camera   ============================ -->
+<robot xmlns:xacro="http://www.ros.org/wiki/xacro" name="up1">
   <xacro:macro name="camera" params="prefix reflect">
+    <!-- ============================   Camera   ============================ -->
     <!-- Camera Joint -->
     <joint name="io_to_${prefix}_camera" type="fixed">

File: up1_description/urdf/io_module/io_module.gazebo.xacro (robot description, xacro)
@@ -1,5 +1,6 @@
 <?xml version="1.0"?>
-<robot xmlns:xacro="http://www.ros.org/wiki/xacro">
+<robot xmlns:xacro="http://www.ros.org/wiki/xacro" name="up1">
   <xacro:macro name="io_module_gazebo">
+    <!-- ============================   IO Module Gazebo   ============================ -->
     <gazebo>
     </gazebo>

File: up1_description/urdf/io_module/io_module.xacro (robot description, xacro)
@@ -1,8 +1,8 @@
 <?xml version="1.0"?>
-<robot xmlns:xacro="http://www.ros.org/wiki/xacro">
+<robot xmlns:xacro="http://www.ros.org/wiki/xacro" name="up1">
   <xacro:include filename="$(find up1_description)/urdf/io_module/camera.xacro" />
   <xacro:include filename="$(find up1_description)/urdf/io_module/io_module.gazebo.xacro" />
-  <!-- ============================   IO Module   ============================ -->
   <xacro:macro name="io_module">
+    <!-- ============================   IO Module   ============================ -->
     <!-- IO Joint -->
     <joint name="base_to_io" type="fixed">

File: up1_description/urdf/manipulator_module/dual_arm_module/arm.gazebo.xacro (robot description, xacro)
@@ -1,6 +1,6 @@
 <?xml version="1.0"?>
-<robot xmlns:xacro="http://www.ros.org/wiki/xacro">
-  <!-- ============================   Arm   ============================ -->
+<robot xmlns:xacro="http://www.ros.org/wiki/xacro" name="up1">
   <xacro:macro name="arm_gazebo" params="prefix">
+    <!-- ============================   Arm Gazebo  ============================ -->
     <gazebo reference="${prefix}_armlink1">
       <turnGravityOff>true</turnGravityOff>

File: up1_description/urdf/manipulator_module/dual_arm_module/arm.transmission.xacro (robot description, xacro)
@@ -1,6 +1,6 @@
 <?xml version="1.0"?>
-<robot xmlns:xacro="http://www.ros.org/wiki/xacro">
-  <!-- ============================   Arm   ============================ -->
+<robot xmlns:xacro="http://www.ros.org/wiki/xacro" name="up1">
   <xacro:macro name="arm_transmission" params="prefix">
+    <!-- ============================   Arm Transmission  ============================ -->
     <transmission name="${prefix}_armroot_to_armlink1_trans">
       <type>transmission_interface/SimpleTransmission</type>

File: up1_description/urdf/manipulator_module/dual_arm_module/arm.xacro (robot description, xacro)
@@ -1,7 +1,7 @@
 <?xml version="1.0"?>
-<robot xmlns:xacro="http://www.ros.org/wiki/xacro">
+<robot xmlns:xacro="http://www.ros.org/wiki/xacro" name="up1">
   <xacro:include filename="$(find up1_description)/urdf/manipulator_module/dual_arm_module/arm.gazebo.xacro" />
-  <!-- ============================   Arm   ============================ -->
   <xacro:macro name="arm" params="prefix reflect">
+    <!-- ============================   Arm   ============================ -->
     <!-- Arm Joint 1 -->
     <joint name="${prefix}_armroot_to_armlink1" type="revolute">

File: up1_description/urdf/manipulator_module/dual_arm_module/arm_module.gazebo.xacro (robot description, xacro)
@@ -1,5 +1,6 @@
 <?xml version="1.0"?>
-<robot xmlns:xacro="http://www.ros.org/wiki/xacro">
+<robot xmlns:xacro="http://www.ros.org/wiki/xacro" name="up1">
   <xacro:macro name="arm_module_gazebo">
+    <!-- ============================   Arm Module Gazebo  ============================ -->
   </xacro:macro>
 </robot>

File: up1_description/urdf/manipulator_module/dual_arm_module/dual_arm_module.xacro (robot description, xacro)
@@ -1,4 +1,4 @@
 <?xml version="1.0"?>
-<robot xmlns:xacro="http://www.ros.org/wiki/xacro">
+<robot xmlns:xacro="http://www.ros.org/wiki/xacro" name="up1">
   <xacro:include filename="$(find up1_description)/urdf/manipulator_module/dual_arm_module/arm.xacro" />
   <xacro:include filename="$(find up1_description)/urdf/manipulator_module/dual_arm_module/arm.transmission.xacro" />
@@ -6,6 +6,6 @@
   <xacro:include filename="$(find up1_description)/urdf/manipulator_module/dual_arm_module/gripper.transmission.xacro" />
   <xacro:include filename="$(find up1_description)/urdf/manipulator_module/dual_arm_module/arm_module.gazebo.xacro" />
-  <!-- ============================   Arm Module   ============================ -->
   <xacro:macro name="manipulator_module">
+    <!-- ============================   Dual Arm Module   ============================ -->
     <!-- Armroot Joint -->
     <joint name="base_to_armroot" type="fixed">

File: up1_description/urdf/manipulator_module/dual_arm_module/gripper.gazebo.xacro (robot description, xacro)
@@ -1,6 +1,6 @@
 <?xml version="1.0"?>
-<robot xmlns:xacro="http://www.ros.org/wiki/xacro">
-  <!-- ============================   Gripper   ============================ -->
+<robot xmlns:xacro="http://www.ros.org/wiki/xacro" name="up1">
   <xacro:macro name="gripper_gazebo" params="prefix">
+    <!-- ============================   Gripper Gazebo   ============================ -->
     <gazebo reference="${prefix}_finger1">
       <turnGravityOff>true</turnGravityOff>

File: up1_description/urdf/manipulator_module/dual_arm_module/gripper.transmission.xacro (robot description, xacro)
@@ -1,6 +1,6 @@
 <?xml version="1.0"?>
-<robot xmlns:xacro="http://www.ros.org/wiki/xacro">
-  <!-- ============================   Gripper   ============================ -->
+<robot xmlns:xacro="http://www.ros.org/wiki/xacro" name="up1">
   <xacro:macro name="gripper_transmission" params="prefix">
+    <!-- ============================   Gripper Transmission   ============================ -->
     <transmission name="${prefix}_gripper_trans">
       <type>transmission_interface/SimpleTransmission</type>

File: up1_description/urdf/manipulator_module/dual_arm_module/gripper.xacro (robot description, xacro)
@@ -1,7 +1,7 @@
 <?xml version="1.0"?>
-<robot xmlns:xacro="http://www.ros.org/wiki/xacro">
+<robot xmlns:xacro="http://www.ros.org/wiki/xacro" name="up1">
   <xacro:include filename="$(find up1_description)/urdf/manipulator_module/dual_arm_module/gripper.gazebo.xacro" />
-  <!-- ============================   Gripper   ============================ -->
   <xacro:macro name="gripper" params="prefix reflect">
+    <!-- ============================   Gripper   ============================ -->
     <!-- Finger Joint 1 -->
     <joint name="${prefix}_gripper_joint" type="prismatic">

File: up1_description/urdf/manipulator_module/dual_arm_module/left_arm_module.xacro (robot description, xacro)
@@ -1,4 +1,4 @@
 <?xml version="1.0"?>
-<robot xmlns:xacro="http://www.ros.org/wiki/xacro">
+<robot xmlns:xacro="http://www.ros.org/wiki/xacro" name="up1">
   <xacro:include filename="$(find up1_description)/urdf/manipulator_module/dual_arm_module/arm.xacro" />
   <xacro:include filename="$(find up1_description)/urdf/manipulator_module/dual_arm_module/arm.transmission.xacro" />
@@ -6,6 +6,6 @@
   <xacro:include filename="$(find up1_description)/urdf/manipulator_module/dual_arm_module/gripper.transmission.xacro" />
   <xacro:include filename="$(find up1_description)/urdf/manipulator_module/dual_arm_module/arm_module.gazebo.xacro" />
-  <!-- ============================   Arm Module   ============================ -->
-  <xacro:macro name="left_arm_module">
+  <xacro:macro name="manipulator_module">
+    <!-- ============================   Left Arm Module   ============================ -->
     <!-- Armroot Joint -->
     <joint name="base_to_armroot" type="fixed">

File: up1_description/urdf/manipulator_module/dual_arm_module/right_arm_module.xacro (robot description, xacro)
@@ -1,4 +1,4 @@
 <?xml version="1.0"?>
-<robot xmlns:xacro="http://www.ros.org/wiki/xacro">
+<robot xmlns:xacro="http://www.ros.org/wiki/xacro" name="up1">
   <xacro:include filename="$(find up1_description)/urdf/manipulator_module/dual_arm_module/arm.xacro" />
   <xacro:include filename="$(find up1_description)/urdf/manipulator_module/dual_arm_module/arm.transmission.xacro" />
@@ -7,5 +7,5 @@
   <xacro:include filename="$(find up1_description)/urdf/manipulator_module/dual_arm_module/arm_module.gazebo.xacro" />
   <!-- ============================   Arm Module   ============================ -->
-  <xacro:macro name="right_arm_module">
+  <xacro:macro name="manipulator_module">
     <!-- Armroot Joint -->
     <joint name="base_to_armroot" type="fixed">

File: up1_description/urdf/manipulator_module/mono_arm_module/arm.gazebo.xacro (robot description, xacro)
@@ -1,4 +1,4 @@
 <?xml version="1.0"?>
-<robot xmlns:xacro="http://www.ros.org/wiki/xacro">
+<robot xmlns:xacro="http://www.ros.org/wiki/xacro" name="up1">
   <!-- ============================   Arm   ============================ -->
   <xacro:macro name="arm_gazebo" params="prefix">

File: up1_description/urdf/manipulator_module/mono_arm_module/arm.xacro (robot description, xacro)
@@ -1,4 +1,4 @@
 <?xml version="1.0"?>
-<robot xmlns:xacro="http://www.ros.org/wiki/xacro">
+<robot xmlns:xacro="http://www.ros.org/wiki/xacro" name="up1">
   <xacro:include filename="$(find up1_description)/urdf/mono_arm_module/arm.gazebo.xacro" />
   <!-- ============================   Arm   ============================ -->

File: up1_description/urdf/manipulator_module/mono_arm_module/arm_module.gazebo.xacro (robot description, xacro)
@@ -1,4 +1,4 @@
 <?xml version="1.0"?>
-<robot xmlns:xacro="http://www.ros.org/wiki/xacro">
+<robot xmlns:xacro="http://www.ros.org/wiki/xacro" name="up1">
   <xacro:macro name="arm_module_gazebo">
   </xacro:macro>

File: up1_description/urdf/manipulator_module/mono_arm_module/gripper.gazebo.xacro (robot description, xacro)
@@ -1,4 +1,4 @@
 <?xml version="1.0"?>
-<robot xmlns:xacro="http://www.ros.org/wiki/xacro">
+<robot xmlns:xacro="http://www.ros.org/wiki/xacro" name="up1">
   <!-- ============================   Gripper   ============================ -->
   <xacro:macro name="gripper_gazebo" params="prefix">
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