Commit message: description: renamed xacro dir to urdf dir as that is the more common convention

File: up1_description/urdf/base_module/base_module.xacro (robot description, xacro)
@@ -1,6 +1,6 @@
 <?xml version="1.0"?>
 <robot xmlns:xacro="http://www.ros.org/wiki/xacro">
-  <xacro:include filename="$(find up1_description)/xacro/base_module/wheel.xacro" />
-  <xacro:include filename="$(find up1_description)/xacro/base_module/base_module.gazebo.xacro" />
+  <xacro:include filename="$(find up1_description)/urdf/base_module/wheel.xacro" />
+  <xacro:include filename="$(find up1_description)/urdf/base_module/base_module.gazebo.xacro" />
   <!-- ============================   Base Module   ============================ -->
   <xacro:macro name="base_module">

File: up1_description/urdf/common.xacro (robot description, xacro)
@@ -1,5 +1,5 @@
 <?xml version="1.0"?>
 <robot xmlns:xacro="http://www.ros.org/wiki/xacro">
-  <xacro:include filename="$(find up1_description)/xacro/common.gazebo.xacro" />
+  <xacro:include filename="$(find up1_description)/urdf/common.gazebo.xacro" />
   <xacro:property name="pi" value="3.14159" />
   <xacro:property name="front_wheel_offset_x" value="0.05569" />

File: up1_description/urdf/io_module/io_module.xacro (robot description, xacro)
@@ -1,6 +1,6 @@
 <?xml version="1.0"?>
 <robot xmlns:xacro="http://www.ros.org/wiki/xacro">
-  <xacro:include filename="$(find up1_description)/xacro/io_module/camera.xacro" />
-  <xacro:include filename="$(find up1_description)/xacro/io_module/io_module.gazebo.xacro" />
+  <xacro:include filename="$(find up1_description)/urdf/io_module/camera.xacro" />
+  <xacro:include filename="$(find up1_description)/urdf/io_module/io_module.gazebo.xacro" />
   <!-- ============================   IO Module   ============================ -->
   <xacro:macro name="io_module">

File: up1_description/urdf/manipulator_module/dual_arm_module/arm.xacro (robot description, xacro)
@@ -1,5 +1,5 @@
 <?xml version="1.0"?>
 <robot xmlns:xacro="http://www.ros.org/wiki/xacro">
-  <xacro:include filename="$(find up1_description)/xacro/mono_arm_module/arm.gazebo.xacro" />
+  <xacro:include filename="$(find up1_description)/urdf/manipulator_module/dual_arm_module/arm.gazebo.xacro" />
   <!-- ============================   Arm   ============================ -->
   <xacro:macro name="arm" params="prefix reflect">
@@ -8,5 +8,6 @@
       <parent link="armroot_link" />
       <child link="${prefix}_armlink1" />
-      <origin rpy="0 0 0" xyz="0 0 0" />
+      <origin rpy="${-reflect*pi/6} ${pi} 0"
+        xyz="${armlink1_offset_x} ${-reflect*armlink1_offset_y} ${armlink1_offset_z}" />
       <axis xyz="0 0 1" />
       <limit lower="${armlink1_limit_lower}" upper="${armlink1_limit_upper}" velocity="${armlink1_velocity}" effort="${armlink1_effort}" />
@@ -16,5 +17,5 @@
       <visual>
         <geometry>
-          <mesh filename="package://up1_description/meshes/mono_arm/armlink1.stl" scale="0.001 0.001 0.001" />
+          <mesh filename="package://up1_description/meshes/dual_arm/armlink1.stl" scale="0.001 0.001 0.001" />
         </geometry>
         <material name="white" />
@@ -22,10 +23,9 @@
       <collision>
         <geometry>
-          <mesh filename="package://up1_description/meshes/mono_arm/armlink1.stl" scale="0.001 0.001 0.001" />
+          <mesh filename="package://up1_description/meshes/dual_arm/armlink1.stl" scale="0.001 0.001 0.001" />
         </geometry>
       </collision>
       <inertial>
-        <mass value="0.17905"/>
-        <!-- inertia is wrong, get update from Daniel -->
+        <mass value="0.06985"/>
         <inertia ixx="0.00023448766" ixy="0.0000000027" ixz="0.00000001913"
                  iyy="0.00024004726" iyz="-0.0000015393" izz="0.00007431363"/>
@@ -36,5 +36,6 @@
       <parent link="${prefix}_armlink1" />
       <child link="${prefix}_armlink2" />
-      <origin rpy="0 0 0" xyz="0 0 0" />
+      <origin rpy="${pi/2} ${pi} 0"
+        xyz="${armlink2_offset_x} ${armlink2_offset_y} ${armlink2_offset_z}" />
       <axis xyz="0 0 ${reflect*1}" />
       <limit lower="${armlink2_limit_lower}" upper="${armlink2_limit_upper}" velocity="${armlink2_velocity}" effort="${armlink2_effort}" />
@@ -44,5 +45,5 @@
       <visual>
         <geometry>
-          <mesh filename="package://up1_description/meshes/mono_arm/armlink2.stl" scale="0.001 0.001 0.001" />
+          <mesh filename="package://up1_description/meshes/dual_arm/armlink2.stl" scale="0.001 0.001 0.001" />
         </geometry>
         <material name="white" />
@@ -50,10 +51,9 @@
       <collision>
         <geometry>
-          <mesh filename="package://up1_description/meshes/mono_arm/armlink2.stl" scale="0.001 0.001 0.001" />
+          <mesh filename="package://up1_description/meshes/dual_arm/armlink2.stl" scale="0.001 0.001 0.001" />
         </geometry>
       </collision>
       <inertial>
-        <mass value="0.49779"/>
-        <!-- inertia is wrong, get update from Daniel -->
+        <mass value="0.07067"/>
         <inertia ixx="0.00029708797" ixy="-0.00000000444" ixz="0.00000000068"
                  iyy="0.0000799845" iyz="-0.00000174097" izz="0.00026073683"/>
@@ -64,5 +64,6 @@
       <parent link="${prefix}_armlink2" />
       <child link="${prefix}_armlink3" />
-      <origin rpy="0 0 0" xyz="0 0 0" />
+      <origin rpy="${-pi/2} ${pi} 0"
+        xyz="${armlink3_offset_x} ${armlink3_offset_y} ${armlink3_offset_z}" />
       <axis xyz="0 0 -1" />
       <limit lower="${armlink3_limit_lower}" upper="${armlink3_limit_upper}" velocity="${armlink3_velocity}" effort="${armlink3_effort}" />
@@ -72,5 +73,5 @@
       <visual>
         <geometry>
-          <mesh filename="package://up1_description/meshes/mono_arm/armlink3.stl" scale="0.001 0.001 0.001" />
+          <mesh filename="package://up1_description/meshes/dual_arm/armlink3.stl" scale="0.001 0.001 0.001" />
         </geometry>
         <material name="white" />
@@ -78,5 +79,5 @@
       <collision>
         <geometry>
-          <mesh filename="package://up1_description/meshes/mono_arm/armlink3.stl" scale="0.001 0.001 0.001" />
+          <mesh filename="package://up1_description/meshes/dual_arm/armlink3.stl" scale="0.001 0.001 0.001" />
         </geometry>
       </collision>
@@ -91,5 +92,6 @@
       <parent link="${prefix}_armlink3" />
       <child link="${prefix}_armlink4" />
-      <origin rpy="0 0 0" xyz="0 0 0" />
+      <origin rpy="${pi/2} 0 0"
+        xyz="${armlink4_offset_x} ${armlink4_offset_y} ${armlink4_offset_z}" />
       <axis xyz="0 0 ${reflect*1}" />
       <limit lower="${armlink4_limit_lower}" upper="${armlink4_limit_upper}" velocity="${armlink4_velocity}" effort="${armlink4_effort}" />
@@ -99,5 +101,5 @@
       <visual>
         <geometry>
-          <mesh filename="package://up1_description/meshes/mono_arm/armlink4.stl" scale="0.001 0.001 0.001" />
+          <mesh filename="package://up1_description/meshes/dual_arm/armlink4.stl" scale="0.001 0.001 0.001" />
         </geometry>
         <material name="white" />
@@ -105,5 +107,5 @@
       <collision>
         <geometry>
-          <mesh filename="package://up1_description/meshes/mono_arm/armlink4.stl" scale="0.001 0.001 0.001" />
+          <mesh filename="package://up1_description/meshes/dual_arm/armlink4.stl" scale="0.001 0.001 0.001" />
         </geometry>
       </collision>
@@ -118,5 +120,6 @@
       <parent link="${prefix}_armlink4" />
       <child link="${prefix}_armlink5" />
-      <origin rpy="0 0 0" xyz="0 0 0" />
+      <origin rpy="0 ${pi/2} 0"
+        xyz="${armlink5_offset_x} ${armlink5_offset_y} ${armlink5_offset_z}" />
       <axis xyz="0 0 ${-reflect*1}" />
       <limit lower="${armlink5_limit_lower}" upper="${armlink5_limit_upper}" velocity="${armlink5_velocity}" effort="${armlink5_effort}" />
@@ -126,5 +129,5 @@
       <visual>
         <geometry>
-          <mesh filename="package://up1_description/meshes/mono_arm/armlink5.stl" scale="0.001 0.001 0.001" />
+          <mesh filename="package://up1_description/meshes/dual_arm/armlink5.stl" scale="0.001 0.001 0.001" />
         </geometry>
         <material name="white" />
@@ -132,5 +135,5 @@
       <collision>
         <geometry>
-          <mesh filename="package://up1_description/meshes/mono_arm/armlink5.stl" scale="0.001 0.001 0.001" />
+          <mesh filename="package://up1_description/meshes/dual_arm/armlink5.stl" scale="0.001 0.001 0.001" />
         </geometry>
       </collision>
@@ -145,9 +148,11 @@
       <parent link="${prefix}_armlink5" />
       <child link="${prefix}_gripper" />
-      <origin rpy="0 0 0" xyz="0 0 0" />
+      <origin rpy="0 0 0"
+        xyz="${gripper_offset_x} ${gripper_offset_y} ${gripper_offset_z}" />
     </joint>
     <!-- Gripper -->
     <link name="${prefix}_gripper" />
     <xacro:arm_gazebo prefix="${prefix}" />
+    <xacro:arm_transmission prefix="${prefix}" />
   </xacro:macro>
 </robot>

File: up1_description/urdf/manipulator_module/dual_arm_module/dual_arm_module.xacro (robot description, xacro)
@@ -1,11 +1,11 @@
 <?xml version="1.0"?>
 <robot xmlns:xacro="http://www.ros.org/wiki/xacro">
-  <xacro:include filename="$(find up1_description)/xacro/manipulator_module/dual_arm_module/arm.xacro" />
-  <xacro:include filename="$(find up1_description)/xacro/manipulator_module/dual_arm_module/arm.transmission.xacro" />
-  <xacro:include filename="$(find up1_description)/xacro/manipulator_module/dual_arm_module/gripper.xacro" />
-  <xacro:include filename="$(find up1_description)/xacro/manipulator_module/dual_arm_module/gripper.transmission.xacro" />
-  <xacro:include filename="$(find up1_description)/xacro/manipulator_module/dual_arm_module/arm_module.gazebo.xacro" />
+  <xacro:include filename="$(find up1_description)/urdf/manipulator_module/dual_arm_module/arm.xacro" />
+  <xacro:include filename="$(find up1_description)/urdf/manipulator_module/dual_arm_module/arm.transmission.xacro" />
+  <xacro:include filename="$(find up1_description)/urdf/manipulator_module/dual_arm_module/gripper.xacro" />
+  <xacro:include filename="$(find up1_description)/urdf/manipulator_module/dual_arm_module/gripper.transmission.xacro" />
+  <xacro:include filename="$(find up1_description)/urdf/manipulator_module/dual_arm_module/arm_module.gazebo.xacro" />
   <!-- ============================   Arm Module   ============================ -->
-  <xacro:macro name="left_arm_module">
+  <xacro:macro name="manipulator_module">
     <!-- Armroot Joint -->
     <joint name="base_to_armroot" type="fixed">
@@ -34,5 +34,7 @@
     </link>
     <xacro:arm_module_gazebo />
+    <xacro:arm prefix="right" reflect="1" />
     <xacro:arm prefix="left" reflect="-1" />
+    <xacro:gripper prefix="right" reflect="1" />
     <xacro:gripper prefix="left" reflect="-1" />
   </xacro:macro>

File: up1_description/urdf/manipulator_module/dual_arm_module/gripper.xacro (robot description, xacro)
@@ -1,5 +1,5 @@
 <?xml version="1.0"?>
 <robot xmlns:xacro="http://www.ros.org/wiki/xacro">
-  <xacro:include filename="$(find up1_description)/xacro/manipulator_module/dual_arm_module/gripper.gazebo.xacro" />
+  <xacro:include filename="$(find up1_description)/urdf/manipulator_module/dual_arm_module/gripper.gazebo.xacro" />
   <!-- ============================   Gripper   ============================ -->
   <xacro:macro name="gripper" params="prefix reflect">

File: up1_description/urdf/manipulator_module/dual_arm_module/left_arm_module.xacro (robot description, xacro)
@@ -1,11 +1,11 @@
 <?xml version="1.0"?>
 <robot xmlns:xacro="http://www.ros.org/wiki/xacro">
-  <xacro:include filename="$(find up1_description)/xacro/manipulator_module/dual_arm_module/arm.xacro" />
-  <xacro:include filename="$(find up1_description)/xacro/manipulator_module/dual_arm_module/arm.transmission.xacro" />
-  <xacro:include filename="$(find up1_description)/xacro/manipulator_module/dual_arm_module/gripper.xacro" />
-  <xacro:include filename="$(find up1_description)/xacro/manipulator_module/dual_arm_module/gripper.transmission.xacro" />
-  <xacro:include filename="$(find up1_description)/xacro/manipulator_module/dual_arm_module/arm_module.gazebo.xacro" />
+  <xacro:include filename="$(find up1_description)/urdf/manipulator_module/dual_arm_module/arm.xacro" />
+  <xacro:include filename="$(find up1_description)/urdf/manipulator_module/dual_arm_module/arm.transmission.xacro" />
+  <xacro:include filename="$(find up1_description)/urdf/manipulator_module/dual_arm_module/gripper.xacro" />
+  <xacro:include filename="$(find up1_description)/urdf/manipulator_module/dual_arm_module/gripper.transmission.xacro" />
+  <xacro:include filename="$(find up1_description)/urdf/manipulator_module/dual_arm_module/arm_module.gazebo.xacro" />
   <!-- ============================   Arm Module   ============================ -->
-  <xacro:macro name="manipulator_module">
+  <xacro:macro name="left_arm_module">
     <!-- Armroot Joint -->
     <joint name="base_to_armroot" type="fixed">
@@ -34,7 +34,5 @@
     </link>
     <xacro:arm_module_gazebo />
-    <xacro:arm prefix="right" reflect="1" />
     <xacro:arm prefix="left" reflect="-1" />
-    <xacro:gripper prefix="right" reflect="1" />
     <xacro:gripper prefix="left" reflect="-1" />
   </xacro:macro>

File: up1_description/urdf/manipulator_module/dual_arm_module/right_arm_module.xacro (robot description, xacro)
@@ -1,9 +1,9 @@
 <?xml version="1.0"?>
 <robot xmlns:xacro="http://www.ros.org/wiki/xacro">
-  <xacro:include filename="$(find up1_description)/xacro/manipulator_module/dual_arm_module/arm.xacro" />
-  <xacro:include filename="$(find up1_description)/xacro/manipulator_module/dual_arm_module/arm.transmission.xacro" />
-  <xacro:include filename="$(find up1_description)/xacro/manipulator_module/dual_arm_module/gripper.xacro" />
-  <xacro:include filename="$(find up1_description)/xacro/manipulator_module/dual_arm_module/gripper.transmission.xacro" />
-  <xacro:include filename="$(find up1_description)/xacro/manipulator_module/dual_arm_module/arm_module.gazebo.xacro" />
+  <xacro:include filename="$(find up1_description)/urdf/manipulator_module/dual_arm_module/arm.xacro" />
+  <xacro:include filename="$(find up1_description)/urdf/manipulator_module/dual_arm_module/arm.transmission.xacro" />
+  <xacro:include filename="$(find up1_description)/urdf/manipulator_module/dual_arm_module/gripper.xacro" />
+  <xacro:include filename="$(find up1_description)/urdf/manipulator_module/dual_arm_module/gripper.transmission.xacro" />
+  <xacro:include filename="$(find up1_description)/urdf/manipulator_module/dual_arm_module/arm_module.gazebo.xacro" />
   <!-- ============================   Arm Module   ============================ -->
   <xacro:macro name="right_arm_module">

File: up1_description/urdf/manipulator_module/mono_arm_module/arm.xacro (robot description, xacro)
@@ -1,5 +1,5 @@
 <?xml version="1.0"?>
 <robot xmlns:xacro="http://www.ros.org/wiki/xacro">
-  <xacro:include filename="$(find up1_description)/xacro/manipulator_module/dual_arm_module/arm.gazebo.xacro" />
+  <xacro:include filename="$(find up1_description)/urdf/mono_arm_module/arm.gazebo.xacro" />
   <!-- ============================   Arm   ============================ -->
   <xacro:macro name="arm" params="prefix reflect">
@@ -8,6 +8,5 @@
       <parent link="armroot_link" />
       <child link="${prefix}_armlink1" />
-      <origin rpy="${-reflect*pi/6} ${pi} 0"
-        xyz="${armlink1_offset_x} ${-reflect*armlink1_offset_y} ${armlink1_offset_z}" />
+      <origin rpy="0 0 0" xyz="0 0 0" />
       <axis xyz="0 0 1" />
       <limit lower="${armlink1_limit_lower}" upper="${armlink1_limit_upper}" velocity="${armlink1_velocity}" effort="${armlink1_effort}" />
@@ -17,5 +16,5 @@
       <visual>
         <geometry>
-          <mesh filename="package://up1_description/meshes/dual_arm/armlink1.stl" scale="0.001 0.001 0.001" />
+          <mesh filename="package://up1_description/meshes/mono_arm/armlink1.stl" scale="0.001 0.001 0.001" />
         </geometry>
         <material name="white" />
@@ -23,9 +22,10 @@
       <collision>
         <geometry>
-          <mesh filename="package://up1_description/meshes/dual_arm/armlink1.stl" scale="0.001 0.001 0.001" />
+          <mesh filename="package://up1_description/meshes/mono_arm/armlink1.stl" scale="0.001 0.001 0.001" />
         </geometry>
       </collision>
       <inertial>
-        <mass value="0.06985"/>
+        <mass value="0.17905"/>
+        <!-- inertia is wrong, get update from Daniel -->
         <inertia ixx="0.00023448766" ixy="0.0000000027" ixz="0.00000001913"
                  iyy="0.00024004726" iyz="-0.0000015393" izz="0.00007431363"/>
@@ -36,6 +36,5 @@
       <parent link="${prefix}_armlink1" />
       <child link="${prefix}_armlink2" />
-      <origin rpy="${pi/2} ${pi} 0"
-        xyz="${armlink2_offset_x} ${armlink2_offset_y} ${armlink2_offset_z}" />
+      <origin rpy="0 0 0" xyz="0 0 0" />
       <axis xyz="0 0 ${reflect*1}" />
       <limit lower="${armlink2_limit_lower}" upper="${armlink2_limit_upper}" velocity="${armlink2_velocity}" effort="${armlink2_effort}" />
@@ -45,5 +44,5 @@
       <visual>
         <geometry>
-          <mesh filename="package://up1_description/meshes/dual_arm/armlink2.stl" scale="0.001 0.001 0.001" />
+          <mesh filename="package://up1_description/meshes/mono_arm/armlink2.stl" scale="0.001 0.001 0.001" />
         </geometry>
         <material name="white" />
@@ -51,9 +50,10 @@
       <collision>
         <geometry>
-          <mesh filename="package://up1_description/meshes/dual_arm/armlink2.stl" scale="0.001 0.001 0.001" />
+          <mesh filename="package://up1_description/meshes/mono_arm/armlink2.stl" scale="0.001 0.001 0.001" />
         </geometry>
       </collision>
       <inertial>
-        <mass value="0.07067"/>
+        <mass value="0.49779"/>
+        <!-- inertia is wrong, get update from Daniel -->
         <inertia ixx="0.00029708797" ixy="-0.00000000444" ixz="0.00000000068"
                  iyy="0.0000799845" iyz="-0.00000174097" izz="0.00026073683"/>
@@ -64,6 +64,5 @@
       <parent link="${prefix}_armlink2" />
       <child link="${prefix}_armlink3" />
-      <origin rpy="${-pi/2} ${pi} 0"
-        xyz="${armlink3_offset_x} ${armlink3_offset_y} ${armlink3_offset_z}" />
+      <origin rpy="0 0 0" xyz="0 0 0" />
       <axis xyz="0 0 -1" />
       <limit lower="${armlink3_limit_lower}" upper="${armlink3_limit_upper}" velocity="${armlink3_velocity}" effort="${armlink3_effort}" />
@@ -73,5 +72,5 @@
       <visual>
         <geometry>
-          <mesh filename="package://up1_description/meshes/dual_arm/armlink3.stl" scale="0.001 0.001 0.001" />
+          <mesh filename="package://up1_description/meshes/mono_arm/armlink3.stl" scale="0.001 0.001 0.001" />
         </geometry>
         <material name="white" />
@@ -79,5 +78,5 @@
       <collision>
         <geometry>
-          <mesh filename="package://up1_description/meshes/dual_arm/armlink3.stl" scale="0.001 0.001 0.001" />
+          <mesh filename="package://up1_description/meshes/mono_arm/armlink3.stl" scale="0.001 0.001 0.001" />
         </geometry>
       </collision>
@@ -92,6 +91,5 @@
       <parent link="${prefix}_armlink3" />
       <child link="${prefix}_armlink4" />
-      <origin rpy="${pi/2} 0 0"
-        xyz="${armlink4_offset_x} ${armlink4_offset_y} ${armlink4_offset_z}" />
+      <origin rpy="0 0 0" xyz="0 0 0" />
       <axis xyz="0 0 ${reflect*1}" />
       <limit lower="${armlink4_limit_lower}" upper="${armlink4_limit_upper}" velocity="${armlink4_velocity}" effort="${armlink4_effort}" />
@@ -101,5 +99,5 @@
       <visual>
         <geometry>
-          <mesh filename="package://up1_description/meshes/dual_arm/armlink4.stl" scale="0.001 0.001 0.001" />
+          <mesh filename="package://up1_description/meshes/mono_arm/armlink4.stl" scale="0.001 0.001 0.001" />
         </geometry>
         <material name="white" />
@@ -107,5 +105,5 @@
       <collision>
         <geometry>
-          <mesh filename="package://up1_description/meshes/dual_arm/armlink4.stl" scale="0.001 0.001 0.001" />
+          <mesh filename="package://up1_description/meshes/mono_arm/armlink4.stl" scale="0.001 0.001 0.001" />
         </geometry>
       </collision>
@@ -120,6 +118,5 @@
       <parent link="${prefix}_armlink4" />
       <child link="${prefix}_armlink5" />
-      <origin rpy="0 ${pi/2} 0"
-        xyz="${armlink5_offset_x} ${armlink5_offset_y} ${armlink5_offset_z}" />
+      <origin rpy="0 0 0" xyz="0 0 0" />
       <axis xyz="0 0 ${-reflect*1}" />
       <limit lower="${armlink5_limit_lower}" upper="${armlink5_limit_upper}" velocity="${armlink5_velocity}" effort="${armlink5_effort}" />
@@ -129,5 +126,5 @@
       <visual>
         <geometry>
-          <mesh filename="package://up1_description/meshes/dual_arm/armlink5.stl" scale="0.001 0.001 0.001" />
+          <mesh filename="package://up1_description/meshes/mono_arm/armlink5.stl" scale="0.001 0.001 0.001" />
         </geometry>
         <material name="white" />
@@ -135,5 +132,5 @@
       <collision>
         <geometry>
-          <mesh filename="package://up1_description/meshes/dual_arm/armlink5.stl" scale="0.001 0.001 0.001" />
+          <mesh filename="package://up1_description/meshes/mono_arm/armlink5.stl" scale="0.001 0.001 0.001" />
         </geometry>
       </collision>
@@ -148,11 +145,9 @@
       <parent link="${prefix}_armlink5" />
       <child link="${prefix}_gripper" />
-      <origin rpy="0 0 0"
-        xyz="${gripper_offset_x} ${gripper_offset_y} ${gripper_offset_z}" />
+      <origin rpy="0 0 0" xyz="0 0 0" />
     </joint>
     <!-- Gripper -->
     <link name="${prefix}_gripper" />
     <xacro:arm_gazebo prefix="${prefix}" />
-    <xacro:arm_transmission prefix="${prefix}" />
   </xacro:macro>
 </robot>

File: up1_description/urdf/manipulator_module/mono_arm_module/gripper.xacro (robot description, xacro)
@@ -1,5 +1,5 @@
 <?xml version="1.0"?>
 <robot xmlns:xacro="http://www.ros.org/wiki/xacro">
-  <xacro:include filename="$(find up1_description)/xacro/mono_arm_module/gripper.gazebo.xacro" />
+  <xacro:include filename="$(find up1_description)/urdf/mono_arm_module/gripper.gazebo.xacro" />
   <!-- ============================   Gripper   ============================ -->
   <xacro:macro name="gripper" params="prefix reflect">
