Commit message: description: renamed xacro dir to urdf dir as that is the more common convention

File: up1_description/urdf/manipulator_module/mono_arm_module/mono_arm_module.xacro (robot description, xacro)
@@ -1,7 +1,7 @@
 <?xml version="1.0"?>
 <robot xmlns:xacro="http://www.ros.org/wiki/xacro">
-  <xacro:include filename="$(find up1_description)/xacro/mono_arm_module/arm.xacro" />
-  <xacro:include filename="$(find up1_description)/xacro/mono_arm_module/gripper.xacro" />
-  <xacro:include filename="$(find up1_description)/xacro/mono_arm_module/arm_module.gazebo.xacro" />
+  <xacro:include filename="$(find up1_description)/urdf/mono_arm_module/arm.xacro" />
+  <xacro:include filename="$(find up1_description)/urdf/mono_arm_module/gripper.xacro" />
+  <xacro:include filename="$(find up1_description)/urdf/mono_arm_module/arm_module.gazebo.xacro" />
   <!-- ============================   Arm Module   ============================ -->
   <xacro:macro name="manipulator_module">

File: up1_description/urdf/up1.xacro (robot description, xacro)
@@ -5,9 +5,9 @@
   <xacro:arg name="base_module" default="base" />
   <xacro:arg name="io_module" default="io" /> -->
-  <xacro:include filename="$(find up1_description)/xacro/common.xacro" />
-  <xacro:include filename="$(find up1_description)/xacro/manipulator_module/$(arg manipulator_module)_module/$(arg manipulator_module)_module.xacro" />
+  <xacro:include filename="$(find up1_description)/urdf/common.xacro" />
+  <xacro:include filename="$(find up1_description)/urdf/manipulator_module/$(arg manipulator_module)_module/$(arg manipulator_module)_module.xacro" />
   <!-- TODO: the other modules will eventually need to be modularized based on config -->
-  <xacro:include filename="$(find up1_description)/xacro/base_module/$(arg base_module)_module.xacro" />
-  <xacro:include filename="$(find up1_description)/xacro/io_module/$(arg io_module)_module.xacro" />
+  <xacro:include filename="$(find up1_description)/urdf/base_module/$(arg base_module)_module.xacro" />
+  <xacro:include filename="$(find up1_description)/urdf/io_module/$(arg io_module)_module.xacro" />
   <xacro:manipulator_module />
   <xacro:base_module />

Commit message: description: switched over from stl format to collada

File: up1_description/urdf/base_module/base_module.xacro (robot description, xacro)
@@ -33,5 +33,5 @@
       <visual>
         <geometry>
-          <mesh filename="package://up1_description/meshes/base/base.stl" scale="0.001 0.001 0.001" />
+          <mesh filename="package://up1_description/meshes/base/base.dae" scale="0.001 0.001 0.001" />
         </geometry>
         <material name="grey" />
@@ -39,5 +39,5 @@
       <collision>
         <geometry>
-          <mesh filename="package://up1_description/meshes/base/base.stl" scale="0.001 0.001 0.001" />
+          <mesh filename="package://up1_description/meshes/base/base.dae" scale="0.001 0.001 0.001" />
         </geometry>
       </collision>

File: up1_description/urdf/base_module/wheel.xacro (robot description, xacro)
@@ -15,5 +15,5 @@
       <visual>
         <geometry>
-          <mesh filename="package://up1_description/meshes/base/wheel.stl" scale="0.001 0.001 0.001" />
+          <mesh filename="package://up1_description/meshes/base/wheel.dae" scale="0.001 0.001 0.001" />
         </geometry>
         <material name="black" />
@@ -21,5 +21,5 @@
       <collision>
         <geometry>
-          <mesh filename="package://up1_description/meshes/base/wheel.stl" scale="0.001 0.001 0.001" />
+          <mesh filename="package://up1_description/meshes/base/wheel.dae" scale="0.001 0.001 0.001" />
         </geometry>
       </collision>
@@ -42,5 +42,5 @@
       <visual>
         <geometry>
-          <mesh filename="package://up1_description/meshes/base/wheel.stl" scale="0.001 0.001 0.001" />
+          <mesh filename="package://up1_description/meshes/base/wheel.dae" scale="0.001 0.001 0.001" />
         </geometry>
         <material name="black" />
@@ -48,5 +48,5 @@
       <collision>
         <geometry>
-          <mesh filename="package://up1_description/meshes/base/wheel.stl" scale="0.001 0.001 0.001" />
+          <mesh filename="package://up1_description/meshes/base/wheel.dae" scale="0.001 0.001 0.001" />
         </geometry>
       </collision>

File: up1_description/urdf/io_module/io_module.xacro (robot description, xacro)
@@ -15,5 +15,5 @@
       <visual>
         <geometry>
-          <mesh filename="package://up1_description/meshes/io/io.stl" scale="0.001 0.001 0.001" />
+          <mesh filename="package://up1_description/meshes/io/io.dae" scale="0.001 0.001 0.001" />
         </geometry>
         <material name="grey" />
@@ -21,5 +21,5 @@
       <collision>
         <geometry>
-          <mesh filename="package://up1_description/meshes/io/io.stl" scale="0.001 0.001 0.001" />
+          <mesh filename="package://up1_description/meshes/io/io.dae" scale="0.001 0.001 0.001" />
         </geometry>
       </collision>

File: up1_description/urdf/manipulator_module/mono_arm_module/arm.xacro (robot description, xacro)
@@ -58,5 +58,5 @@
       <visual>
         <geometry>
-          <mesh filename="package://up1_description/meshes/mono_arm/armlink1.stl" scale="0.001 0.001 0.001" />
+          <mesh filename="package://up1_description/meshes/mono_arm/armlink1.dae" scale="0.001 0.001 0.001" />
         </geometry>
         <material name="white" />
@@ -64,5 +64,5 @@
       <collision>
         <geometry>
-          <mesh filename="package://up1_description/meshes/mono_arm/armlink1.stl" scale="0.001 0.001 0.001" />
+          <mesh filename="package://up1_description/meshes/mono_arm/armlink1.dae" scale="0.001 0.001 0.001" />
         </geometry>
       </collision>
@@ -86,5 +86,5 @@
       <visual>
         <geometry>
-          <mesh filename="package://up1_description/meshes/mono_arm/armlink2.stl" scale="0.001 0.001 0.001" />
+          <mesh filename="package://up1_description/meshes/mono_arm/armlink2.dae" scale="0.001 0.001 0.001" />
         </geometry>
         <material name="white" />
@@ -92,5 +92,5 @@
       <collision>
         <geometry>
-          <mesh filename="package://up1_description/meshes/mono_arm/armlink2.stl" scale="0.001 0.001 0.001" />
+          <mesh filename="package://up1_description/meshes/mono_arm/armlink2.dae" scale="0.001 0.001 0.001" />
         </geometry>
       </collision>
@@ -114,5 +114,5 @@
       <visual>
         <geometry>
-          <mesh filename="package://up1_description/meshes/mono_arm/armlink3.stl" scale="0.001 0.001 0.001" />
+          <mesh filename="package://up1_description/meshes/mono_arm/armlink3.dae" scale="0.001 0.001 0.001" />
         </geometry>
         <material name="white" />
@@ -120,5 +120,5 @@
       <collision>
         <geometry>
-          <mesh filename="package://up1_description/meshes/mono_arm/armlink3.stl" scale="0.001 0.001 0.001" />
+          <mesh filename="package://up1_description/meshes/mono_arm/armlink3.dae" scale="0.001 0.001 0.001" />
         </geometry>
       </collision>
@@ -142,5 +142,5 @@
       <visual>
         <geometry>
-          <mesh filename="package://up1_description/meshes/mono_arm/armlink4.stl" scale="0.001 0.001 0.001" />
+          <mesh filename="package://up1_description/meshes/mono_arm/armlink4.dae" scale="0.001 0.001 0.001" />
         </geometry>
         <material name="white" />
@@ -148,5 +148,5 @@
       <collision>
         <geometry>
-          <mesh filename="package://up1_description/meshes/mono_arm/armlink4.stl" scale="0.001 0.001 0.001" />
+          <mesh filename="package://up1_description/meshes/mono_arm/armlink4.dae" scale="0.001 0.001 0.001" />
         </geometry>
       </collision>
@@ -170,5 +170,5 @@
       <visual>
         <geometry>
-          <mesh filename="package://up1_description/meshes/mono_arm/armlink5.stl" scale="0.001 0.001 0.001" />
+          <mesh filename="package://up1_description/meshes/mono_arm/armlink5.dae" scale="0.001 0.001 0.001" />
         </geometry>
         <material name="white" />
@@ -176,5 +176,5 @@
       <collision>
         <geometry>
-          <mesh filename="package://up1_description/meshes/mono_arm/armlink5.stl" scale="0.001 0.001 0.001" />
+          <mesh filename="package://up1_description/meshes/mono_arm/armlink5.dae" scale="0.001 0.001 0.001" />
         </geometry>
       </collision>

File: up1_description/urdf/manipulator_module/mono_arm_module/arm_root_link.xacro (robot description, xacro)
@@ -10,5 +10,5 @@
       <visual>
         <geometry>
-          <mesh filename="package://up1_description/meshes/mono_arm/armroot.stl" scale="0.001 0.001 0.001" />
+          <mesh filename="package://up1_description/meshes/mono_arm/armroot.dae" scale="0.001 0.001 0.001" />
         </geometry>
         <material name="grey" />
@@ -16,5 +16,5 @@
       <collision>
         <geometry>
-          <mesh filename="package://up1_description/meshes/mono_arm/armroot.stl" scale="0.001 0.001 0.001" />
+          <mesh filename="package://up1_description/meshes/mono_arm/armroot.dae" scale="0.001 0.001 0.001" />
         </geometry>
       </collision>

File: up1_description/urdf/manipulator_module/mono_arm_module/gripper.xacro (robot description, xacro)
@@ -21,5 +21,5 @@
       <visual>
         <geometry>
-          <mesh filename="package://up1_description/meshes/mono_arm/finger.stl" scale="0.001 0.001 0.001" />
+          <mesh filename="package://up1_description/meshes/mono_arm/finger.dae" scale="0.001 0.001 0.001" />
         </geometry>
         <material name="grey" />
@@ -27,5 +27,5 @@
       <collision>
         <geometry>
-          <mesh filename="package://up1_description/meshes/mono_arm/finger.stl" scale="0.001 0.001 0.001" />
+          <mesh filename="package://up1_description/meshes/mono_arm/finger.dae" scale="0.001 0.001 0.001" />
         </geometry>
       </collision>
@@ -50,5 +50,5 @@
       <visual>
         <geometry>
-          <mesh filename="package://up1_description/meshes/mono_arm/finger.stl" scale="0.001 0.001 0.001" />
+          <mesh filename="package://up1_description/meshes/mono_arm/finger.dae" scale="0.001 0.001 0.001" />
         </geometry>
         <material name="grey" />
@@ -56,5 +56,5 @@
       <collision>
         <geometry>
-          <mesh filename="package://up1_description/meshes/mono_arm/finger.stl" scale="0.001 0.001 0.001" />
+          <mesh filename="package://up1_description/meshes/mono_arm/finger.dae" scale="0.001 0.001 0.001" />
         </geometry>
       </collision>

File: up1_description/urdf/up1_mono.urdf (robot description, URDF)
Before this commit: robot up1, 17 links, 16 joints
Links:
- link armroot_link: geometry collision mesh filename=package://up1_description/meshes/mono_arm/armroot.dae scale=0.001 0.001 0.001; visual mesh filename=package://up1_description/meshes/mono_arm/armroot.dae scale=0.001 0.001 0.001
- link base_link: geometry collision mesh filename=package://up1_description/meshes/base/base.dae scale=0.001 0.001 0.001; visual mesh filename=package://up1_description/meshes/base/base.dae scale=0.001 0.001 0.001
- link io_link: geometry collision mesh filename=package://up1_description/meshes/io/io.dae scale=0.001 0.001 0.001; visual mesh filename=package://up1_description/meshes/io/io.dae scale=0.001 0.001 0.001
- link left_back_wheel: geometry collision mesh filename=package://up1_description/meshes/base/wheel.dae scale=0.001 0.001 0.001; visual mesh filename=package://up1_description/meshes/base/wheel.dae scale=0.001 0.001 0.001
- link left_front_wheel: geometry collision mesh filename=package://up1_description/meshes/base/wheel.dae scale=0.001 0.001 0.001; visual mesh filename=package://up1_description/meshes/base/wheel.dae scale=0.001 0.001 0.001
- link right_armlink1: geometry collision mesh filename=package://up1_description/meshes/mono_arm/armlink1.dae scale=0.001 0.001 0.001; visual mesh filename=package://up1_description/meshes/mono_arm/armlink1.dae scale=0.001 0.001 0.001
- link right_armlink2: geometry collision mesh filename=package://up1_description/meshes/mono_arm/armlink2.dae scale=0.001 0.001 0.001; visual mesh filename=package://up1_description/meshes/mono_arm/armlink2.dae scale=0.001 0.001 0.001
- link right_armlink3: geometry collision mesh filename=package://up1_description/meshes/mono_arm/armlink3.dae scale=0.001 0.001 0.001; visual mesh filename=package://up1_description/meshes/mono_arm/armlink3.dae scale=0.001 0.001 0.001
- link right_armlink4: geometry collision mesh filename=package://up1_description/meshes/mono_arm/armlink4.dae scale=0.001 0.001 0.001; visual mesh filename=package://up1_description/meshes/mono_arm/armlink4.dae scale=0.001 0.001 0.001
- link right_back_wheel: geometry collision mesh filename=package://up1_description/meshes/base/wheel.dae scale=0.001 0.001 0.001; visual mesh filename=package://up1_description/meshes/base/wheel.dae scale=0.001 0.001 0.001
- link right_finger1: geometry collision mesh filename=package://up1_description/meshes/mono_arm/finger.dae scale=0.001 0.001 0.001; visual mesh filename=package://up1_description/meshes/mono_arm/finger.dae scale=0.001 0.001 0.001
- link right_finger2: geometry collision mesh filename=package://up1_description/meshes/mono_arm/finger.dae scale=0.001 0.001 0.001; visual mesh filename=package://up1_description/meshes/mono_arm/finger.dae scale=0.001 0.001 0.001
- link right_front_wheel: geometry collision mesh filename=package://up1_description/meshes/base/wheel.dae scale=0.001 0.001 0.001; visual mesh filename=package://up1_description/meshes/base/wheel.dae scale=0.001 0.001 0.001
- link right_gripper: geometry collision mesh filename=package://up1_description/meshes/mono_arm/armlink5.dae scale=0.001 0.001 0.001; visual mesh filename=package://up1_description/meshes/mono_arm/armlink5.dae scale=0.001 0.001 0.001
Joints:
- joint right_armlink1_to_armlink2: limit lower=-1.570795 upper=1.570795 effort=6.0 velocity=1 -> lower=-1.570795 upper=1.570795 effort=6.0 velocity=4.553
- joint right_armlink2_to_armlink3: limit lower=-1.570795 upper=1.570795 effort=6.0 velocity=1 -> lower=-1.570795 upper=1.570795 effort=6.0 velocity=5.236
- joint right_armlink3_to_armlink4: limit lower=-1.570795 upper=1.570795 effort=6.0 velocity=1 -> lower=-1.570795 upper=1.570795 effort=6.0 velocity=5.236
- joint right_armlink4_to_gripper: limit lower=-1.570795 upper=1.570795 effort=6.0 velocity=1 -> lower=-1.570795 upper=1.570795 effort=6.0 velocity=5.236
- joint right_armroot_to_armlink1: limit lower=-1.570795 upper=1.570795 effort=6.0 velocity=1 -> lower=-1.570795 upper=1.570795 effort=6.0 velocity=5.236
