Commit message: description: updated meshes and urdf

File: up1_description/urdf/base_module/base_module.xacro (robot description, xacro)
@@ -16,7 +16,5 @@
       </visual>
       <collision>
-        <!-- represent base collision with a simple rectangular model, positioned by base_size_z s.t. top
-             surface of the collision box matches the top surface of the PR2 base -->
-        <origin xyz="0 0 ${0.051+0.04/2}" rpy="0 0 0" />
+        <origin xyz="0 0 0" rpy="0 0 0" />
         <geometry>
           <box size="0.001 0.001 0.001" />
@@ -25,5 +23,5 @@
     </link>
     <joint name="up1_footprint_joint" type="fixed">
-      <origin xyz="0 0 0.051" rpy="0 0 0" />
+      <origin xyz="0 0 0.06016" rpy="0 0 0" />
       <child link="base_link" />
       <parent link="up1_footprint"/>
@@ -33,5 +31,5 @@
       <visual>
         <geometry>
-          <mesh filename="package://up1_description/meshes/base/base.dae" scale="0.001 0.001 0.001" />
+          <mesh filename="package://up1_description/meshes/base/base_viz.dae" scale="0.001 0.001 0.001" />
         </geometry>
         <material name="grey" />

File: up1_description/urdf/base_module/wheel.xacro (robot description, xacro)
@@ -15,5 +15,5 @@
       <visual>
         <geometry>
-          <mesh filename="package://up1_description/meshes/base/wheel.dae" scale="0.001 0.001 0.001" />
+          <mesh filename="package://up1_description/meshes/base/wheel_viz.dae" scale="0.001 0.001 0.001" />
         </geometry>
         <material name="black" />
@@ -42,5 +42,5 @@
       <visual>
         <geometry>
-          <mesh filename="package://up1_description/meshes/base/wheel.dae" scale="0.001 0.001 0.001" />
+          <mesh filename="package://up1_description/meshes/base/wheel_viz.dae" scale="0.001 0.001 0.001" />
         </geometry>
         <material name="black" />

File: up1_description/urdf/common.xacro (robot description, xacro)
@@ -12,7 +12,7 @@
   <xacro:property name="io_offset_y" value="0" />
   <xacro:property name="io_offset_z" value="0.03356" />
-  <xacro:property name="camera_offset_x" value="-0.01219" />
-  <xacro:property name="camera_offset_y" value="0.04027" />
-  <xacro:property name="camera_offset_z" value="0.00023" />
+  <xacro:property name="camera_offset_x" value="-0.00619" />
+  <xacro:property name="camera_offset_y" value="0.02127" />
+  <xacro:property name="camera_offset_z" value="0.00451" />
   <material name="black">
     <color rgba="0 0 0 1" />

File: up1_description/urdf/io_module/camera.xacro (robot description, xacro)
@@ -7,5 +7,5 @@
       <parent link="io_link" />
       <child link="${prefix}_camera" />
-      <origin xyz="${camera_offset_x} ${-reflect*camera_offset_y} ${camera_offset_z}" />
+      <origin xyz="${camera_offset_x} ${-reflect*camera_offset_y} ${camera_offset_z}" rpy="0 ${pi/15} 0"/>
     </joint>
     <!-- Camera Link -->
@@ -13,5 +13,5 @@
       <visual>
         <geometry>
-          <mesh filename="package://up1_description/meshes/io/camera.dae" scale="0.001 0.001 0.001" />
+          <mesh filename="package://up1_description/meshes/io/camera_viz.dae" scale="0.001 0.001 0.001" />
         </geometry>
         <material name="black" />

File: up1_description/urdf/io_module/io_module.xacro (robot description, xacro)
@@ -15,5 +15,5 @@
       <visual>
         <geometry>
-          <mesh filename="package://up1_description/meshes/io/io.dae" scale="0.001 0.001 0.001" />
+          <mesh filename="package://up1_description/meshes/io/io_viz.dae" scale="0.001 0.001 0.001" />
         </geometry>
         <material name="grey" />

File: up1_description/urdf/manipulator_module/mono_arm_module/arm.xacro (robot description, xacro)
@@ -58,5 +58,5 @@
       <visual>
         <geometry>
-          <mesh filename="package://up1_description/meshes/mono_arm/armlink1.dae" scale="0.001 0.001 0.001" />
+          <mesh filename="package://up1_description/meshes/mono_arm/armlink1_viz.dae" scale="0.001 0.001 0.001" />
         </geometry>
         <material name="white" />
@@ -86,5 +86,5 @@
       <visual>
         <geometry>
-          <mesh filename="package://up1_description/meshes/mono_arm/armlink2.dae" scale="0.001 0.001 0.001" />
+          <mesh filename="package://up1_description/meshes/mono_arm/armlink2_viz.dae" scale="0.001 0.001 0.001" />
         </geometry>
         <material name="white" />
@@ -114,5 +114,5 @@
       <visual>
         <geometry>
-          <mesh filename="package://up1_description/meshes/mono_arm/armlink3.dae" scale="0.001 0.001 0.001" />
+          <mesh filename="package://up1_description/meshes/mono_arm/armlink3_viz.dae" scale="0.001 0.001 0.001" />
         </geometry>
         <material name="white" />
@@ -142,5 +142,5 @@
       <visual>
         <geometry>
-          <mesh filename="package://up1_description/meshes/mono_arm/armlink4.dae" scale="0.001 0.001 0.001" />
+          <mesh filename="package://up1_description/meshes/mono_arm/armlink4_viz.dae" scale="0.001 0.001 0.001" />
         </geometry>
         <material name="white" />
@@ -170,5 +170,5 @@
       <visual>
         <geometry>
-          <mesh filename="package://up1_description/meshes/mono_arm/armlink5.dae" scale="0.001 0.001 0.001" />
+          <mesh filename="package://up1_description/meshes/mono_arm/armlink5_viz.dae" scale="0.001 0.001 0.001" />
         </geometry>
         <material name="white" />

File: up1_description/urdf/manipulator_module/mono_arm_module/arm_root_link.xacro (robot description, xacro)
@@ -10,5 +10,5 @@
       <visual>
         <geometry>
-          <mesh filename="package://up1_description/meshes/mono_arm/armroot.dae" scale="0.001 0.001 0.001" />
+          <mesh filename="package://up1_description/meshes/mono_arm/armroot_viz.dae" scale="0.001 0.001 0.001" />
         </geometry>
         <material name="grey" />

File: up1_description/urdf/manipulator_module/mono_arm_module/gripper.xacro (robot description, xacro)
@@ -21,5 +21,5 @@
       <visual>
         <geometry>
-          <mesh filename="package://up1_description/meshes/mono_arm/finger.dae" scale="0.001 0.001 0.001" />
+          <mesh filename="package://up1_description/meshes/mono_arm/finger_viz.dae" scale="0.001 0.001 0.001" />
         </geometry>
         <material name="grey" />
@@ -50,5 +50,5 @@
       <visual>
         <geometry>
-          <mesh filename="package://up1_description/meshes/mono_arm/finger.dae" scale="0.001 0.001 0.001" />
+          <mesh filename="package://up1_description/meshes/mono_arm/finger_viz.dae" scale="0.001 0.001 0.001" />
         </geometry>
         <material name="grey" />

File: up1_description/urdf/up1_mono.urdf (robot description, URDF)
Before this commit: robot up1, 17 links, 16 joints
Links:
- link armroot_link: geometry collision mesh filename=package://up1_description/meshes/mono_arm/armroot.dae scale=0.001 0.001 0.001; visual mesh filename=package://up1_description/meshes/mono_arm/armroot_viz.dae scale=0.001 0.001 0.001
- link base_link: geometry collision mesh filename=package://up1_description/meshes/base/base.dae scale=0.001 0.001 0.001; visual mesh filename=package://up1_description/meshes/base/base_viz.dae scale=0.001 0.001 0.001
- link io_link: geometry collision mesh filename=package://up1_description/meshes/io/io.dae scale=0.001 0.001 0.001; visual mesh filename=package://up1_description/meshes/io/io_viz.dae scale=0.001 0.001 0.001
- link left_back_wheel: geometry collision mesh filename=package://up1_description/meshes/base/wheel.dae scale=0.001 0.001 0.001; visual mesh filename=package://up1_description/meshes/base/wheel_viz.dae scale=0.001 0.001 0.001
- link left_camera: geometry collision mesh filename=package://up1_description/meshes/io/camera.dae scale=0.001 0.001 0.001; visual mesh filename=package://up1_description/meshes/io/camera_viz.dae scale=0.001 0.001 0.001
- link left_front_wheel: geometry collision mesh filename=package://up1_description/meshes/base/wheel.dae scale=0.001 0.001 0.001; visual mesh filename=package://up1_description/meshes/base/wheel_viz.dae scale=0.001 0.001 0.001
- link right_armlink1: geometry collision mesh filename=package://up1_description/meshes/mono_arm/armlink1.dae scale=0.001 0.001 0.001; visual mesh filename=package://up1_description/meshes/mono_arm/armlink1_viz.dae scale=0.001 0.001 0.001
- link right_armlink2: geometry collision mesh filename=package://up1_description/meshes/mono_arm/armlink2.dae scale=0.001 0.001 0.001; visual mesh filename=package://up1_description/meshes/mono_arm/armlink2_viz.dae scale=0.001 0.001 0.001
- link right_armlink3: geometry collision mesh filename=package://up1_description/meshes/mono_arm/armlink3.dae scale=0.001 0.001 0.001; visual mesh filename=package://up1_description/meshes/mono_arm/armlink3_viz.dae scale=0.001 0.001 0.001
- link right_armlink4: geometry collision mesh filename=package://up1_description/meshes/mono_arm/armlink4.dae scale=0.001 0.001 0.001; visual mesh filename=package://up1_description/meshes/mono_arm/armlink4_viz.dae scale=0.001 0.001 0.001
- link right_back_wheel: geometry collision mesh filename=package://up1_description/meshes/base/wheel.dae scale=0.001 0.001 0.001; visual mesh filename=package://up1_description/meshes/base/wheel_viz.dae scale=0.001 0.001 0.001
- link right_camera: geometry collision mesh filename=package://up1_description/meshes/io/camera.dae scale=0.001 0.001 0.001; visual mesh filename=package://up1_description/meshes/io/camera_viz.dae scale=0.001 0.001 0.001
- link right_finger1: geometry collision mesh filename=package://up1_description/meshes/mono_arm/finger.dae scale=0.001 0.001 0.001; visual mesh filename=package://up1_description/meshes/mono_arm/finger_viz.dae scale=0.001 0.001 0.001
- link right_finger2: geometry collision mesh filename=package://up1_description/meshes/mono_arm/finger.dae scale=0.001 0.001 0.001; visual mesh filename=package://up1_description/meshes/mono_arm/finger_viz.dae scale=0.001 0.001 0.001
- link right_front_wheel: geometry collision mesh filename=package://up1_description/meshes/base/wheel.dae scale=0.001 0.001 0.001; visual mesh filename=package://up1_description/meshes/base/wheel_viz.dae scale=0.001 0.001 0.001
- link right_gripper: geometry collision mesh filename=package://up1_description/meshes/mono_arm/armlink5.dae scale=0.001 0.001 0.001; visual mesh filename=package://up1_description/meshes/mono_arm/armlink5_viz.dae scale=0.001 0.001 0.001
Joints:
- joint io_to_left_camera: origin xyz=-0.01219 0.04027 0.00023 -> xyz=-0.00619 0.02127 0.00451 rpy=0 0.209439333333 0
- joint io_to_right_camera: origin xyz=-0.01219 -0.04027 0.00023 -> xyz=-0.00619 -0.02127 0.00451 rpy=0 0.209439333333 0
- joint up1_footprint_joint: origin xyz=0 0 0.051 rpy=0 0 0 -> xyz=0 0 0.06016 rpy=0 0 0

Commit message: description: tweaks to xacro files

File: up1_description/urdf/base_module/base_module.xacro (robot description, xacro)
@@ -33,5 +33,4 @@
           <mesh filename="package://up1_description/meshes/base/base_viz.dae" scale="0.001 0.001 0.001" />
         </geometry>
-        <material name="grey" />
       </visual>
       <collision>

File: up1_description/urdf/base_module/wheel.xacro (robot description, xacro)
@@ -17,5 +17,4 @@
           <mesh filename="package://up1_description/meshes/base/wheel_viz.dae" scale="0.001 0.001 0.001" />
         </geometry>
-        <material name="black" />
       </visual>
       <collision>

File: up1_description/urdf/common.xacro (robot description, xacro)
@@ -12,5 +12,5 @@
   <xacro:property name="io_offset_y" value="0" />
   <xacro:property name="io_offset_z" value="0.03356" />
-  <xacro:property name="camera_offset_x" value="-0.00619" />
+  <xacro:property name="camera_offset_x" value="-0.00519" />
   <xacro:property name="camera_offset_y" value="0.02127" />
   <xacro:property name="camera_offset_z" value="0.00451" />

File: up1_description/urdf/io_module/camera.xacro (robot description, xacro)
@@ -15,5 +15,4 @@
           <mesh filename="package://up1_description/meshes/io/camera_viz.dae" scale="0.001 0.001 0.001" />
         </geometry>
-        <material name="black" />
       </visual>
       <collision>

File: up1_description/urdf/manipulator_module/mono_arm_module/arm.xacro (robot description, xacro)
@@ -10,5 +10,5 @@
   <xacro:property name="armlink2_offset_z" value="-0.0553" />
   <xacro:property name="armlink3_offset_x" value="0" />
-  <xacro:property name="armlink3_offset_y" value="0.09602" />
+  <xacro:property name="armlink3_offset_y" value="0.10602" />
   <xacro:property name="armlink3_offset_z" value="0" />
   <xacro:property name="armlink4_offset_x" value="0" />

File: up1_description/urdf/up1_mono.urdf (robot description, URDF)
Before this commit: robot up1, 17 links, 16 joints
Joints:
- joint io_to_left_camera: origin xyz=-0.00619 0.02127 0.00451 rpy=0 0.209439333333 0 -> xyz=-0.00519 0.02127 0.00451 rpy=0 0.209439333333 0
- joint io_to_right_camera: origin xyz=-0.00619 -0.02127 0.00451 rpy=0 0.209439333333 0 -> xyz=-0.00519 -0.02127 0.00451 rpy=0 0.209439333333 0
- joint right_armlink2_to_armlink3: origin xyz=0 0.09602 0 rpy=-1.570795 3.14159 0 -> xyz=0 0.10602 0 rpy=-1.570795 3.14159 0
