Commit message: description: progress save

File: up1_description/urdf/base_module/base_module.xacro (robot description, xacro)
@@ -36,5 +36,5 @@
       <collision>
         <geometry>
-          <mesh filename="package://up1_description/meshes/base/base.dae" scale="0.001 0.001 0.001" />
+          <mesh filename="package://up1_description/meshes/base/base.stl" scale="0.001 0.001 0.001" />
         </geometry>
       </collision>

File: up1_description/urdf/base_module/wheel.xacro (robot description, xacro)
@@ -7,7 +7,7 @@
       <parent link="base_link" />
       <child link="${prefix}_front_wheel" />
-      <origin rpy="${reflect*pi/2} 0 0"
-          xyz="${front_wheel_offset_x} ${-reflect*front_wheel_offset_y} ${front_wheel_offset_z}" />
-      <axis xyz="0 0 ${-reflect*1}" />
+      <origin rpy="0 0 0"
+          xyz="${front_wheel_offset_x} ${reflect*front_wheel_offset_y} ${front_wheel_offset_z}" />
+      <axis xyz="0 1 0" />
     </joint>
     <!-- Front Wheel Link -->
@@ -20,5 +20,5 @@
       <collision>
         <geometry>
-          <mesh filename="package://up1_description/meshes/base/wheel.dae" scale="0.001 0.001 0.001" />
+          <mesh filename="package://up1_description/meshes/base/wheel_left.stl" scale="0.001 0.001 0.001" />
         </geometry>
       </collision>
@@ -33,7 +33,7 @@
       <parent link="base_link" />
       <child link="${prefix}_back_wheel" />
-      <origin rpy="${reflect*pi/2} 0 0"
-          xyz="${back_wheel_offset_x} ${-reflect*back_wheel_offset_y} ${back_wheel_offset_z}" />
-      <axis xyz="0 0 ${-reflect*1}" />
+      <origin rpy="0 0 0"
+          xyz="${back_wheel_offset_x} ${reflect*back_wheel_offset_y} ${back_wheel_offset_z}" />
+      <axis xyz="0 1 0" />
     </joint>
     <!-- Back Wheel Link -->
@@ -47,5 +47,5 @@
       <collision>
         <geometry>
-          <mesh filename="package://up1_description/meshes/base/wheel.dae" scale="0.001 0.001 0.001" />
+          <mesh filename="package://up1_description/meshes/base/wheel_left.stl" scale="0.001 0.001 0.001" />
         </geometry>
       </collision>

File: up1_description/urdf/common.xacro (robot description, xacro)
@@ -3,16 +3,16 @@
   <xacro:include filename="$(find up1_description)/urdf/common.gazebo.xacro" />
   <xacro:property name="pi" value="3.14159" />
-  <xacro:property name="front_wheel_offset_x" value="0.05569" />
-  <xacro:property name="front_wheel_offset_y" value="0.12922" />
-  <xacro:property name="front_wheel_offset_z" value="-0.02110" />
-  <xacro:property name="back_wheel_offset_x" value="-0.05883" />
-  <xacro:property name="back_wheel_offset_y" value="0.12922" />
-  <xacro:property name="back_wheel_offset_z" value="-0.02110" />
-  <xacro:property name="io_offset_x" value="0.09136" />
-  <xacro:property name="io_offset_y" value="0" />
-  <xacro:property name="io_offset_z" value="0.03356" />
-  <xacro:property name="camera_offset_x" value="-0.00519" />
-  <xacro:property name="camera_offset_y" value="0.02127" />
-  <xacro:property name="camera_offset_z" value="0.00451" />
+  <xacro:property name="front_wheel_offset_x" value="0.05605" />
+  <xacro:property name="front_wheel_offset_y" value="0.12005" />
+  <xacro:property name="front_wheel_offset_z" value="-0.02016" />
+  <xacro:property name="back_wheel_offset_x" value="-0.05848" />
+  <xacro:property name="back_wheel_offset_y" value="0.12005" />
+  <xacro:property name="back_wheel_offset_z" value="-0.02016" />
+  <xacro:property name="io_offset_x" value="0.09184" />
+  <xacro:property name="io_offset_y" value="0.0" />
+  <xacro:property name="io_offset_z" value="0.03465" />
+  <xacro:property name="camera_offset_y" value="0.02150" />
+  <xacro:property name="camera_offset_z" value="0.00476" />
+  <xacro:property name="camera_offset_x" value="-0.00751" />
   <material name="black">
     <color rgba="0 0 0 1" />

File: up1_description/urdf/io_module/camera.xacro (robot description, xacro)
@@ -7,5 +7,5 @@
       <parent link="io_link" />
       <child link="${prefix}_camera" />
-      <origin xyz="${camera_offset_x} ${-reflect*camera_offset_y} ${camera_offset_z}" rpy="0 ${pi/15} 0"/>
+      <origin xyz="${camera_offset_x} ${reflect*camera_offset_y} ${camera_offset_z}" rpy="0 ${pi/15} 0"/>
     </joint>
     <!-- Camera Link -->
@@ -18,5 +18,5 @@
       <collision>
         <geometry>
-          <mesh filename="package://up1_description/meshes/io/camera.dae" scale="0.001 0.001 0.001" />
+          <mesh filename="package://up1_description/meshes/io/camera.stl" scale="0.001 0.001 0.001" />
         </geometry>
       </collision>

File: up1_description/urdf/io_module/io_module.xacro (robot description, xacro)
@@ -21,5 +21,5 @@
       <collision>
         <geometry>
-          <mesh filename="package://up1_description/meshes/io/io.dae" scale="0.001 0.001 0.001" />
+          <mesh filename="package://up1_description/meshes/io/io.stl" scale="0.001 0.001 0.001" />
         </geometry>
       </collision>

File: up1_description/urdf/manipulator_module/mono_arm_module/arm.xacro (robot description, xacro)
@@ -3,19 +3,19 @@
   <xacro:include filename="$(find up1_description)/urdf/manipulator_module/mono_arm_module/arm.gazebo.xacro" />
   <xacro:include filename="$(find up1_description)/urdf/manipulator_module/mono_arm_module/arm.transmission.xacro" />
-  <xacro:property name="armlink1_offset_x" value="0.01398" />
-  <xacro:property name="armlink1_offset_y" value="0" />
-  <xacro:property name="armlink1_offset_z" value="0.0402" />
-  <xacro:property name="armlink2_offset_x" value="0" />
-  <xacro:property name="armlink2_offset_y" value="0" />
-  <xacro:property name="armlink2_offset_z" value="-0.0553" />
-  <xacro:property name="armlink3_offset_x" value="0" />
-  <xacro:property name="armlink3_offset_y" value="0.10602" />
-  <xacro:property name="armlink3_offset_z" value="0" />
-  <xacro:property name="armlink4_offset_x" value="0" />
-  <xacro:property name="armlink4_offset_y" value="0" />
+  <xacro:property name="armlink1_offset_x" value="0.0" />
+  <xacro:property name="armlink1_offset_y" value="0.0" />
+  <xacro:property name="armlink1_offset_z" value="0.03099" />
+  <xacro:property name="armlink2_offset_x" value="0.0" />
+  <xacro:property name="armlink2_offset_y" value="0.0" />
+  <xacro:property name="armlink2_offset_z" value="0.05527" />
+  <xacro:property name="armlink3_offset_x" value="0.0" />
+  <xacro:property name="armlink3_offset_y" value="0.0" />
+  <xacro:property name="armlink3_offset_z" value="0.10602" />
+  <xacro:property name="armlink4_offset_x" value="0.0" />
+  <xacro:property name="armlink4_offset_y" value="0.0" />
   <xacro:property name="armlink4_offset_z" value="0.05588" />
-  <xacro:property name="gripper_offset_x" value="0" />
-  <xacro:property name="gripper_offset_y" value="0.07641" />
-  <xacro:property name="gripper_offset_z" value="0" />
+  <xacro:property name="gripper_offset_x" value="0.0" />
+  <xacro:property name="gripper_offset_y" value="0.0" />
+  <xacro:property name="gripper_offset_z" value="0.08471" />
   <xacro:property name="armlink1_limit_lower" value="${-pi/2}" />
   <xacro:property name="armlink1_limit_upper" value="${pi/2}" />
@@ -49,6 +49,6 @@
       <parent link="armroot_link" />
       <child link="${prefix}_armlink1" />
-      <origin rpy="0 ${pi} 0"
-        xyz="${armlink1_offset_x} ${-reflect*armlink1_offset_y} ${armlink1_offset_z}" />
+      <origin rpy="0 0 0"
+        xyz="${armlink1_offset_x} ${armlink1_offset_y} ${armlink1_offset_z}" />
       <axis xyz="0 0 1" />
       <limit lower="${armlink1_limit_lower}" upper="${armlink1_limit_upper}" velocity="${armlink1_velocity}" effort="${armlink1_effort}" />
@@ -64,5 +64,5 @@
       <collision>
         <geometry>
-          <mesh filename="package://up1_description/meshes/mono_arm/armlink1.dae" scale="0.001 0.001 0.001" />
+          <mesh filename="package://up1_description/meshes/mono_arm/armlink1.stl" scale="0.001 0.001 0.001" />
         </geometry>
       </collision>
@@ -77,7 +77,7 @@
       <parent link="${prefix}_armlink1" />
       <child link="${prefix}_armlink2" />
-      <origin rpy="${pi/2} ${pi} 0"
+      <origin rpy="0 0 0"
         xyz="${armlink2_offset_x} ${armlink2_offset_y} ${armlink2_offset_z}" />
-      <axis xyz="0 0 ${reflect*1}" />
+      <axis xyz="0 1 0" />
       <limit lower="${armlink2_limit_lower}" upper="${armlink2_limit_upper}" velocity="${armlink2_velocity}" effort="${armlink2_effort}" />
     </joint>
@@ -92,5 +92,5 @@
       <collision>
         <geometry>
-          <mesh filename="package://up1_description/meshes/mono_arm/armlink2.dae" scale="0.001 0.001 0.001" />
+          <mesh filename="package://up1_description/meshes/mono_arm/armlink2.stl" scale="0.001 0.001 0.001" />
         </geometry>
       </collision>
@@ -105,7 +105,7 @@
       <parent link="${prefix}_armlink2" />
       <child link="${prefix}_armlink3" />
-      <origin rpy="${-pi/2} ${pi} 0"
+      <origin rpy="0 0 0"
         xyz="${armlink3_offset_x} ${armlink3_offset_y} ${armlink3_offset_z}" />
-      <axis xyz="0 0 -1" />
+      <axis xyz="0 0 1" />
       <limit lower="${armlink3_limit_lower}" upper="${armlink3_limit_upper}" velocity="${armlink3_velocity}" effort="${armlink3_effort}" />
     </joint>
@@ -120,5 +120,5 @@
       <collision>
         <geometry>
-          <mesh filename="package://up1_description/meshes/mono_arm/armlink3.dae" scale="0.001 0.001 0.001" />
+          <mesh filename="package://up1_description/meshes/mono_arm/armlink3.stl" scale="0.001 0.001 0.001" />
         </geometry>
       </collision>
@@ -133,7 +133,7 @@
       <parent link="${prefix}_armlink3" />
       <child link="${prefix}_armlink4" />
-      <origin rpy="${pi/2} 0 0"
+      <origin rpy="0 0 0"
         xyz="${armlink4_offset_x} ${armlink4_offset_y} ${armlink4_offset_z}" />
-      <axis xyz="0 0 ${reflect*1}" />
+      <axis xyz="0 1 0" />
       <limit lower="${armlink4_limit_lower}" upper="${armlink4_limit_upper}" velocity="${armlink4_velocity}" effort="${armlink4_effort}" />
     </joint>
@@ -148,5 +148,5 @@
       <collision>
         <geometry>
-          <mesh filename="package://up1_description/meshes/mono_arm/armlink4.dae" scale="0.001 0.001 0.001" />
+          <mesh filename="package://up1_description/meshes/mono_arm/armlink4.stl" scale="0.001 0.001 0.001" />
         </geometry>
       </collision>
@@ -161,7 +161,7 @@
       <parent link="${prefix}_armlink4" />
       <child link="${prefix}_gripper" />
-      <origin rpy="0 ${pi/2} 0"
+      <origin rpy="0 0 0"
         xyz="${gripper_offset_x} ${gripper_offset_y} ${gripper_offset_z}" />
-      <axis xyz="0 0 ${-reflect*1}" />
+      <axis xyz="1 0 0" />
       <limit lower="${gripper_limit_lower}" upper="${gripper_limit_upper}" velocity="${gripper_velocity}" effort="${gripper_effort}" />
     </joint>
@@ -176,5 +176,5 @@
       <collision>
         <geometry>
-          <mesh filename="package://up1_description/meshes/mono_arm/armlink5.dae" scale="0.001 0.001 0.001" />
+          <mesh filename="package://up1_description/meshes/mono_arm/armlink5.stl" scale="0.001 0.001 0.001" />
         </geometry>
       </collision>

File: up1_description/urdf/manipulator_module/mono_arm_module/arm_root_link.xacro (robot description, xacro)
@@ -1,6 +1,6 @@
 <?xml version="1.0"?>
 <robot xmlns:xacro="http://www.ros.org/wiki/xacro" name="up1">
-  <xacro:property name="armroot_offset_z" value="0.03876" />
-  <xacro:property name="armroot_offset_x" value="-0.00869" />
+  <xacro:property name="armroot_offset_z" value="0.05058" />
+  <xacro:property name="armroot_offset_x" value="0.00556" />
   <xacro:property name="armroot_offset_y" value="0.0" />
   <xacro:macro name="arm_root_link">
@@ -16,5 +16,5 @@
       <collision>
         <geometry>
-          <mesh filename="package://up1_description/meshes/mono_arm/armroot.dae" scale="0.001 0.001 0.001" />
+          <mesh filename="package://up1_description/meshes/mono_arm/armroot.stl" scale="0.001 0.001 0.001" />
         </geometry>
       </collision>

File: up1_description/urdf/manipulator_module/mono_arm_module/gripper.xacro (robot description, xacro)
@@ -3,7 +3,7 @@
   <xacro:include filename="$(find up1_description)/urdf/manipulator_module/mono_arm_module/gripper.gazebo.xacro" />
   <xacro:include filename="$(find up1_description)/urdf/manipulator_module/mono_arm_module/gripper.transmission.xacro" />
-  <xacro:property name="finger_offset_x" value="0.01800" />
-  <xacro:property name="finger_offset_y" value="0.08121" />
-  <xacro:property name="finger_offset_z" value="0" />
+  <xacro:property name="finger_offset_x" value="0.0" />
+  <xacro:property name="finger_offset_y" value="0.0" />
+  <xacro:property name="finger_offset_z" value="0.07961" />
   <xacro:macro name="gripper" params="prefix reflect">
     <!-- ============================   Gripper   ============================ -->
@@ -12,7 +12,7 @@
       <parent link="${prefix}_gripper" />
       <child link="${prefix}_finger1" />
-      <origin rpy="0 ${pi/2} 0"
+      <origin rpy="0 0 0"
         xyz="${-finger_offset_x} ${finger_offset_y} ${finger_offset_z}" />
-      <axis xyz="0 0 1" />
+      <axis xyz="0 1 0" />
       <limit lower="0" upper="${finger_limit_upper}" velocity="${finger1_velocity}" effort="${finger1_effort}" />
     </joint>
@@ -27,5 +27,5 @@
       <collision>
         <geometry>
-          <mesh filename="package://up1_description/meshes/mono_arm/finger.dae" scale="0.001 0.001 0.001" />
+          <mesh filename="package://up1_description/meshes/mono_arm/finger_left.stl" scale="0.001 0.001 0.001" />
         </geometry>
       </collision>
@@ -40,7 +40,7 @@
       <parent link="${prefix}_gripper" />
       <child link="${prefix}_finger2" />
-      <origin rpy="0 ${-pi/2} 0"
+      <origin rpy="0 0 ${pi}"
         xyz="${finger_offset_x} ${finger_offset_y} ${finger_offset_z}" />
-      <axis xyz="0 0 1" />
+      <axis xyz="0 1 0" />
       <limit lower="0" upper="${finger_limit_upper}" velocity="${finger2_velocity}" effort="${finger2_effort}" />
       <mimic joint="${prefix}_finger_joint" multiplier="1" offset="0"/>
@@ -56,5 +56,5 @@
       <collision>
         <geometry>
-          <mesh filename="package://up1_description/meshes/mono_arm/finger.dae" scale="0.001 0.001 0.001" />
+          <mesh filename="package://up1_description/meshes/mono_arm/finger_left.stl" scale="0.001 0.001 0.001" />
         </geometry>
       </collision>

File: up1_description/urdf/up1_mono.urdf (robot description, URDF)
Before this commit: robot up1, 17 links, 16 joints
Links:
- link armroot_link: geometry collision mesh filename=package://up1_description/meshes/mono_arm/armroot.stl scale=0.001 0.001 0.001; visual mesh filename=package://up1_description/meshes/mono_arm/armroot_viz.dae scale=0.001 0.001 0.001
- link base_link: geometry collision mesh filename=package://up1_description/meshes/base/base.stl scale=0.001 0.001 0.001; visual mesh filename=package://up1_description/meshes/base/base_viz.dae scale=0.001 0.001 0.001
- link io_link: geometry collision mesh filename=package://up1_description/meshes/io/io.stl scale=0.001 0.001 0.001; visual mesh filename=package://up1_description/meshes/io/io_viz.dae scale=0.001 0.001 0.001
- link left_back_wheel: geometry collision mesh filename=package://up1_description/meshes/base/wheel_left.stl scale=0.001 0.001 0.001; visual mesh filename=package://up1_description/meshes/base/wheel_viz.dae scale=0.001 0.001 0.001
- link left_camera: geometry collision mesh filename=package://up1_description/meshes/io/camera.stl scale=0.001 0.001 0.001; visual mesh filename=package://up1_description/meshes/io/camera_viz.dae scale=0.001 0.001 0.001
- link left_front_wheel: geometry collision mesh filename=package://up1_description/meshes/base/wheel_left.stl scale=0.001 0.001 0.001; visual mesh filename=package://up1_description/meshes/base/wheel_viz.dae scale=0.001 0.001 0.001
- link right_armlink1: geometry collision mesh filename=package://up1_description/meshes/mono_arm/armlink1.stl scale=0.001 0.001 0.001; visual mesh filename=package://up1_description/meshes/mono_arm/armlink1_viz.dae scale=0.001 0.001 0.001
- link right_armlink2: geometry collision mesh filename=package://up1_description/meshes/mono_arm/armlink2.stl scale=0.001 0.001 0.001; visual mesh filename=package://up1_description/meshes/mono_arm/armlink2_viz.dae scale=0.001 0.001 0.001
- link right_armlink3: geometry collision mesh filename=package://up1_description/meshes/mono_arm/armlink3.stl scale=0.001 0.001 0.001; visual mesh filename=package://up1_description/meshes/mono_arm/armlink3_viz.dae scale=0.001 0.001 0.001
- link right_armlink4: geometry collision mesh filename=package://up1_description/meshes/mono_arm/armlink4.stl scale=0.001 0.001 0.001; visual mesh filename=package://up1_description/meshes/mono_arm/armlink4_viz.dae scale=0.001 0.001 0.001
- link right_back_wheel: geometry collision mesh filename=package://up1_description/meshes/base/wheel_left.stl scale=0.001 0.001 0.001; visual mesh filename=package://up1_description/meshes/base/wheel_viz.dae scale=0.001 0.001 0.001
- link right_camera: geometry collision mesh filename=package://up1_description/meshes/io/camera.stl scale=0.001 0.001 0.001; visual mesh filename=package://up1_description/meshes/io/camera_viz.dae scale=0.001 0.001 0.001
- link right_finger1: geometry collision mesh filename=package://up1_description/meshes/mono_arm/finger_left.stl scale=0.001 0.001 0.001; visual mesh filename=package://up1_description/meshes/mono_arm/finger_viz.dae scale=0.001 0.001 0.001
- link right_finger2: geometry collision mesh filename=package://up1_description/meshes/mono_arm/finger_left.stl scale=0.001 0.001 0.001; visual mesh filename=package://up1_description/meshes/mono_arm/finger_viz.dae scale=0.001 0.001 0.001
- link right_front_wheel: geometry collision mesh filename=package://up1_description/meshes/base/wheel_left.stl scale=0.001 0.001 0.001; visual mesh filename=package://up1_description/meshes/base/wheel_viz.dae scale=0.001 0.001 0.001
- link right_gripper: geometry collision mesh filename=package://up1_description/meshes/mono_arm/armlink5.stl scale=0.001 0.001 0.001; visual mesh filename=package://up1_description/meshes/mono_arm/armlink5_viz.dae scale=0.001 0.001 0.001
Joints:
- joint base_to_armroot: origin xyz=-0.00869 0.0 0.03876 -> xyz=0.00556 0.0 0.05058
- joint base_to_io: origin xyz=0.09136 0 0.03356 -> xyz=0.09184 0.0 0.03465
- joint base_to_left_back_wheel: axis 0 0 1.0 -> 0 1 0; origin xyz=-0.05883 0.12922 -0.0211 rpy=-1.570795 0 0 -> xyz=-0.05848 -0.12005 -0.02016 rpy=0 0 0
- joint base_to_left_front_wheel: axis 0 0 1.0 -> 0 1 0; origin xyz=0.05569 0.12922 -0.0211 rpy=-1.570795 0 0 -> xyz=0.05605 -0.12005 -0.02016 rpy=0 0 0
- joint base_to_right_back_wheel: axis 0 0 -1.0 -> 0 1 0; origin xyz=-0.05883 -0.12922 -0.0211 rpy=1.570795 0 0 -> xyz=-0.05848 0.12005 -0.02016 rpy=0 0 0
- joint base_to_right_front_wheel: axis 0 0 -1.0 -> 0 1 0; origin xyz=0.05569 -0.12922 -0.0211 rpy=1.570795 0 0 -> xyz=0.05605 0.12005 -0.02016 rpy=0 0 0
- joint io_to_left_camera: origin xyz=-0.00519 0.02127 0.00451 rpy=0 0.209439333333 0 -> xyz=-0.00751 -0.0215 0.00476 rpy=0 0.209439333333 0
- joint io_to_right_camera: origin xyz=-0.00519 -0.02127 0.00451 rpy=0 0.209439333333 0 -> xyz=-0.00751 0.0215 0.00476 rpy=0 0.209439333333 0
- joint right_armlink1_to_armlink2: axis 0 0 1.0 -> 0 1 0; origin xyz=0 0 -0.0553 rpy=1.570795 3.14159 0 -> xyz=0.0 0.0 0.05527 rpy=0 0 0
- joint right_armlink2_to_armlink3: axis 0 0 -1 -> 0 0 1; origin xyz=0 0.10602 0 rpy=-1.570795 3.14159 0 -> xyz=0.0 0.0 0.10602 rpy=0 0 0
- joint right_armlink3_to_armlink4: axis 0 0 1.0 -> 0 1 0; origin xyz=0 0 0.05588 rpy=1.570795 0 0 -> xyz=0.0 0.0 0.05588 rpy=0 0 0
- joint right_armlink4_to_gripper: axis 0 0 -1.0 -> 1 0 0; origin xyz=0 0.07641 0 rpy=0 1.570795 0 -> xyz=0.0 0.0 0.08471 rpy=0 0 0
- joint right_armroot_to_armlink1: origin xyz=0.01398 -0.0 0.0402 rpy=0 3.14159 0 -> xyz=0.0 0.0 0.03099 rpy=0 0 0
- joint right_finger_joint: axis 0 0 1 -> 0 1 0; origin xyz=-0.018 0.08121 0 rpy=0 1.570795 0 -> xyz=-0.0 0.0 0.07961 rpy=0 0 0
- joint right_finger_joint_fake: axis 0 0 1 -> 0 1 0; origin xyz=0.018 0.08121 0 rpy=0 -1.570795 0 -> xyz=0.0 0.0 0.07961 rpy=0 0 3.14159
