Commit message: description: progress save

File: up1_description/urdf/base_module/base_module.xacro (robot description, xacro)
@@ -23,5 +23,5 @@
     </link>
     <joint name="up1_footprint_joint" type="fixed">
-      <origin xyz="0 0 0.06016" rpy="0 0 0" />
+      <origin xyz="0 0 0" rpy="0 0 0" />
       <child link="base_link" />
       <parent link="up1_footprint"/>
@@ -46,6 +46,6 @@
     </link>
     <xacro:base_module_gazebo />
-    <xacro:wheel prefix="right" reflect="1" />
-    <xacro:wheel prefix="left" reflect="-1" />
+    <xacro:wheel prefix="right" />
+    <xacro:wheel prefix="left" />
   </xacro:macro>
 </robot>

File: up1_description/urdf/base_module/wheel.xacro (robot description, xacro)
@@ -1,12 +1,15 @@
 <?xml version="1.0"?>
 <robot xmlns:xacro="http://www.ros.org/wiki/xacro" name="up1">
-  <xacro:macro name="wheel" params="prefix reflect">
+  <xacro:property name="front_wheel_offset_x" value="0.05605" />
+  <xacro:property name="back_wheel_offset_x" value="0.05848" />
+  <xacro:property name="wheel_offset_y" value="0.12005" />
+  <xacro:property name="wheel_offset_z" value="0.02016" />
+  <xacro:macro name="wheel" params="prefix">
     <!-- ============================   Wheel   ============================ -->
-    <!-- Front Wheel Joint -->
+    <!-- Wheel Joint -->
     <joint name="base_to_${prefix}_front_wheel" type="continuous">
       <parent link="base_link" />
       <child link="${prefix}_front_wheel" />
-      <origin rpy="0 0 0"
-          xyz="${front_wheel_offset_x} ${reflect*front_wheel_offset_y} ${front_wheel_offset_z}" />
+      <origin rpy="0 0 0" xyz="${front_wheel_offset_x} ${wheel_offset_y} -${wheel_offset_z}" />
       <axis xyz="0 1 0" />
     </joint>
@@ -15,10 +18,10 @@
       <visual>
         <geometry>
-          <mesh filename="package://up1_description/meshes/base/wheel_viz.dae" scale="0.001 0.001 0.001" />
+          <mesh filename="package://up1_description/meshes/base/wheel_${prefix}_viz.dae" scale="0.001 0.001 0.001" />
         </geometry>
       </visual>
       <collision>
         <geometry>
-          <mesh filename="package://up1_description/meshes/base/wheel_left.stl" scale="0.001 0.001 0.001" />
+          <mesh filename="package://up1_description/meshes/base/wheel_${prefix}.stl" scale="0.001 0.001 0.001" />
         </geometry>
       </collision>
@@ -29,23 +32,20 @@
       </inertial>
     </link>
-    <!-- Back Wheel Joint -->
     <joint name="base_to_${prefix}_back_wheel" type="continuous">
       <parent link="base_link" />
       <child link="${prefix}_back_wheel" />
-      <origin rpy="0 0 0"
-          xyz="${back_wheel_offset_x} ${reflect*back_wheel_offset_y} ${back_wheel_offset_z}" />
+      <origin rpy="0 0 0" xyz="-${back_wheel_offset_x} ${wheel_offset_y} -${wheel_offset_z}" />
       <axis xyz="0 1 0" />
     </joint>
-    <!-- Back Wheel Link -->
+    <!-- Front Wheel Link -->
     <link name="${prefix}_back_wheel">
       <visual>
         <geometry>
-          <mesh filename="package://up1_description/meshes/base/wheel_viz.dae" scale="0.001 0.001 0.001" />
+          <mesh filename="package://up1_description/meshes/base/wheel_${prefix}_viz.dae" scale="0.001 0.001 0.001" />
         </geometry>
-        <material name="black" />
       </visual>
       <collision>
         <geometry>
-          <mesh filename="package://up1_description/meshes/base/wheel_left.stl" scale="0.001 0.001 0.001" />
+          <mesh filename="package://up1_description/meshes/base/wheel_${prefix}.stl" scale="0.001 0.001 0.001" />
         </geometry>
       </collision>

File: up1_description/urdf/common.xacro (robot description, xacro)
@@ -3,16 +3,4 @@
   <xacro:include filename="$(find up1_description)/urdf/common.gazebo.xacro" />
   <xacro:property name="pi" value="3.14159" />
-  <xacro:property name="front_wheel_offset_x" value="0.05605" />
-  <xacro:property name="front_wheel_offset_y" value="0.12005" />
-  <xacro:property name="front_wheel_offset_z" value="-0.02016" />
-  <xacro:property name="back_wheel_offset_x" value="-0.05848" />
-  <xacro:property name="back_wheel_offset_y" value="0.12005" />
-  <xacro:property name="back_wheel_offset_z" value="-0.02016" />
-  <xacro:property name="io_offset_x" value="0.09184" />
-  <xacro:property name="io_offset_y" value="0.0" />
-  <xacro:property name="io_offset_z" value="0.03465" />
-  <xacro:property name="camera_offset_y" value="0.02150" />
-  <xacro:property name="camera_offset_z" value="0.00476" />
-  <xacro:property name="camera_offset_x" value="-0.00751" />
   <material name="black">
     <color rgba="0 0 0 1" />

File: up1_description/urdf/io_module/camera.xacro (robot description, xacro)
@@ -1,4 +1,7 @@
 <?xml version="1.0"?>
 <robot xmlns:xacro="http://www.ros.org/wiki/xacro" name="up1">
+  <xacro:property name="camera_offset_y" value="0.02150" />
+  <xacro:property name="camera_offset_z" value="0.00476" />
+  <xacro:property name="camera_offset_x" value="-0.00751" />
   <xacro:macro name="camera" params="prefix reflect">
     <!-- ============================   Camera   ============================ -->

File: up1_description/urdf/io_module/io_module.xacro (robot description, xacro)
@@ -3,4 +3,7 @@
   <xacro:include filename="$(find up1_description)/urdf/io_module/camera.xacro" />
   <xacro:include filename="$(find up1_description)/urdf/io_module/io_module.gazebo.xacro" />
+  <xacro:property name="io_offset_x" value="0.09184" />
+  <xacro:property name="io_offset_y" value="0.0" />
+  <xacro:property name="io_offset_z" value="0.03465" />
   <xacro:macro name="io_module">
     <!-- ============================   IO Module   ============================ -->

File: up1_description/urdf/manipulator_module/mono_arm_module/gripper.xacro (robot description, xacro)
@@ -21,5 +21,5 @@
       <visual>
         <geometry>
-          <mesh filename="package://up1_description/meshes/mono_arm/finger_viz.dae" scale="0.001 0.001 0.001" />
+          <mesh filename="package://up1_description/meshes/mono_arm/finger_left_viz.dae" scale="0.001 0.001 0.001" />
         </geometry>
         <material name="grey" />
@@ -50,5 +50,5 @@
       <visual>
         <geometry>
-          <mesh filename="package://up1_description/meshes/mono_arm/finger_viz.dae" scale="0.001 0.001 0.001" />
+          <mesh filename="package://up1_description/meshes/mono_arm/finger_left_viz.dae" scale="0.001 0.001 0.001" />
         </geometry>
         <material name="grey" />

File: up1_description/urdf/up1_mono.urdf (robot description, URDF)
Before this commit: robot up1, 17 links, 16 joints
Links:
- link left_back_wheel: geometry collision mesh filename=package://up1_description/meshes/base/wheel_left.stl scale=0.001 0.001 0.001; visual mesh filename=package://up1_description/meshes/base/wheel_left_viz.dae scale=0.001 0.001 0.001
- link left_front_wheel: geometry collision mesh filename=package://up1_description/meshes/base/wheel_left.stl scale=0.001 0.001 0.001; visual mesh filename=package://up1_description/meshes/base/wheel_left_viz.dae scale=0.001 0.001 0.001
- link right_back_wheel: geometry collision mesh filename=package://up1_description/meshes/base/wheel_right.stl scale=0.001 0.001 0.001; visual mesh filename=package://up1_description/meshes/base/wheel_right_viz.dae scale=0.001 0.001 0.001
- link right_finger1: geometry collision mesh filename=package://up1_description/meshes/mono_arm/finger_left.stl scale=0.001 0.001 0.001; visual mesh filename=package://up1_description/meshes/mono_arm/finger_left_viz.d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 scale=0.001 0.001 0.001
- link right_finger2: geometry collision mesh filename=package://up1_description/meshes/mono_arm/finger_left.stl scale=0.001 0.001 0.001; visual mesh filename=package://up1_description/meshes/mono_arm/finger_left_viz.d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 scale=0.001 0.001 0.001
- link right_front_wheel: geometry collision mesh filename=package://up1_description/meshes/base/wheel_right.stl scale=0.001 0.001 0.001; visual mesh filename=package://up1_description/meshes/base/wheel_right_viz.dae scale=0.001 0.001 0.001
Joints:
- joint base_to_left_back_wheel: origin xyz=-0.05848 -0.12005 -0.02016 rpy=0 0 0 -> xyz=0.05848 0.12005 -0.02016 rpy=0 0 0
- joint base_to_left_front_wheel: origin xyz=0.05605 -0.12005 -0.02016 rpy=0 0 0 -> xyz=0.05605 0.12005 -0.02016 rpy=0 0 0
- joint base_to_right_back_wheel: origin xyz=-0.05848 0.12005 -0.02016 rpy=0 0 0 -> xyz=0.05848 0.12005 -0.02016 rpy=0 0 0
- joint up1_footprint_joint: origin xyz=0 0 0.06016 rpy=0 0 0 -> xyz=0 0 0 rpy=0 0 0

Commit message: description: fixed wheels

File: up1_description/urdf/base_module/base_module.xacro (robot description, xacro)
@@ -46,6 +46,8 @@
     </link>
     <xacro:base_module_gazebo />
-    <xacro:wheel prefix="right" />
-    <xacro:wheel prefix="left" />
+    <xacro:wheel prefix="right" end="front" reflect="1" wheel_offset_x="0.05605" />
+    <xacro:wheel prefix="right" end="back" reflect="1" wheel_offset_x="-0.05848" />
+    <xacro:wheel prefix="left" end="front" reflect="-1" wheel_offset_x="0.05605" />
+    <xacro:wheel prefix="left" end="back" reflect="-1" wheel_offset_x="-0.05848" />
   </xacro:macro>
 </robot>

File: up1_description/urdf/base_module/wheel.xacro (robot description, xacro)
@@ -1,43 +1,17 @@
 <?xml version="1.0"?>
 <robot xmlns:xacro="http://www.ros.org/wiki/xacro" name="up1">
-  <xacro:property name="front_wheel_offset_x" value="0.05605" />
-  <xacro:property name="back_wheel_offset_x" value="0.05848" />
   <xacro:property name="wheel_offset_y" value="0.12005" />
   <xacro:property name="wheel_offset_z" value="0.02016" />
-  <xacro:macro name="wheel" params="prefix">
+  <xacro:macro name="wheel" params="prefix end reflect wheel_offset_x">
     <!-- ============================   Wheel   ============================ -->
     <!-- Wheel Joint -->
-    <joint name="base_to_${prefix}_front_wheel" type="continuous">
+    <joint name="base_to_${prefix}_${end}_wheel" type="continuous">
       <parent link="base_link" />
-      <child link="${prefix}_front_wheel" />
-      <origin rpy="0 0 0" xyz="${front_wheel_offset_x} ${wheel_offset_y} -${wheel_offset_z}" />
+      <child link="${prefix}_${end}_wheel" />
+      <origin rpy="0 0 0" xyz="${wheel_offset_x} ${-1*reflect*wheel_offset_y} -${wheel_offset_z}" />
       <axis xyz="0 1 0" />
     </joint>
-    <!-- Front Wheel Link -->
-    <link name="${prefix}_front_wheel">
-      <visual>
-        <geometry>
-          <mesh filename="package://up1_description/meshes/base/wheel_${prefix}_viz.dae" scale="0.001 0.001 0.001" />
-        </geometry>
-      </visual>
-      <collision>
-        <geometry>
-          <mesh filename="package://up1_description/meshes/base/wheel_${prefix}.stl" scale="0.001 0.001 0.001" />
-        </geometry>
-      </collision>
-      <inertial>
-        <mass value="0.01791"/>
-        <inertia ixx="0.00000575118" ixy="-0.00000000224" ixz="0.0"
-                 iyy="0.00000575882" iyz="0.0" izz="0.0000094354"/>
-      </inertial>
-    </link>
-    <joint name="base_to_${prefix}_back_wheel" type="continuous">
-      <parent link="base_link" />
-      <child link="${prefix}_back_wheel" />
-      <origin rpy="0 0 0" xyz="-${back_wheel_offset_x} ${wheel_offset_y} -${wheel_offset_z}" />
-      <axis xyz="0 1 0" />
-    </joint>
-    <!-- Front Wheel Link -->
-    <link name="${prefix}_back_wheel">
+    <!-- Wheel Link -->
+    <link name="${prefix}_${end}_wheel">
       <visual>
         <geometry>

File: up1_description/urdf/up1_mono.urdf (robot description, URDF)
Before this commit: robot up1, 17 links, 16 joints
Joints:
- joint base_to_left_back_wheel: origin xyz=0.05848 0.12005 -0.02016 rpy=0 0 0 -> xyz=-0.05848 0.12005 -0.02016 rpy=0 0 0.0
- joint base_to_left_front_wheel: origin xyz=0.05605 0.12005 -0.02016 rpy=0 0 0 -> xyz=0.05605 0.12005 -0.02016 rpy=0 0 0.0
- joint base_to_right_back_wheel: origin xyz=0.05848 0.12005 -0.02016 rpy=0 0 0 -> xyz=-0.05848 -0.12005 -0.02016 rpy=0 0 0.0
- joint base_to_right_front_wheel: origin xyz=0.05605 0.12005 -0.02016 rpy=0 0 0 -> xyz=0.05605 -0.12005 -0.02016 rpy=0 0 0.0

Commit message: description: tweak colors in urdf

File: up1_description/urdf/base_module/base_module.xacro (robot description, xacro)
@@ -33,4 +33,5 @@
           <mesh filename="package://up1_description/meshes/base/base_viz.dae" scale="0.001 0.001 0.001" />
         </geometry>
+        <material name="dark grey" />
       </visual>
       <collision>

File: up1_description/urdf/base_module/wheel.xacro (robot description, xacro)
@@ -18,4 +18,5 @@
           <mesh filename="package://up1_description/meshes/base/wheel_${prefix}_viz.dae" scale="0.001 0.001 0.001" />
         </geometry>
+        <material name="black" />
       </visual>
       <collision>

File: up1_description/urdf/common.xacro (robot description, xacro)
@@ -12,6 +12,12 @@
     <color rgba="1 0 0 1" />
   </material>
+  <material name="dark grey">
+    <color rgba=".2 .2 .2 1" />
+  </material>
   <material name="grey">
-    <color rgba=".5 .5 .5 1" />
+    <color rgba=".4 .4 .4 1" />
+  </material>
+  <material name="light grey">
+    <color rgba=".7 .7 .7 1" />
   </material>
   <material name="green">

File: up1_description/urdf/io_module/camera.xacro (robot description, xacro)
@@ -18,4 +18,5 @@
           <mesh filename="package://up1_description/meshes/io/camera_viz.dae" scale="0.001 0.001 0.001" />
         </geometry>
+        <material name="black" />
       </visual>
       <collision>

File: up1_description/urdf/manipulator_module/mono_arm_module/arm.xacro (robot description, xacro)
@@ -60,5 +60,5 @@
           <mesh filename="package://up1_description/meshes/mono_arm/armlink1_viz.dae" scale="0.001 0.001 0.001" />
         </geometry>
-        <material name="white" />
+        <material name="light grey" />
       </visual>
       <collision>
@@ -88,5 +88,5 @@
           <mesh filename="package://up1_description/meshes/mono_arm/armlink2_viz.dae" scale="0.001 0.001 0.001" />
         </geometry>
-        <material name="white" />
+        <material name="light grey" />
       </visual>
       <collision>
@@ -116,5 +116,5 @@
           <mesh filename="package://up1_description/meshes/mono_arm/armlink3_viz.dae" scale="0.001 0.001 0.001" />
         </geometry>
-        <material name="white" />
+        <material name="light grey" />
       </visual>
       <collision>
@@ -144,5 +144,5 @@
           <mesh filename="package://up1_description/meshes/mono_arm/armlink4_viz.dae" scale="0.001 0.001 0.001" />
         </geometry>
-        <material name="white" />
+        <material name="light grey" />
       </visual>
       <collision>
@@ -172,5 +172,5 @@
           <mesh filename="package://up1_description/meshes/mono_arm/armlink5_viz.dae" scale="0.001 0.001 0.001" />
         </geometry>
-        <material name="white" />
+        <material name="light grey" />
       </visual>
       <collision>

File: up1_description/urdf/manipulator_module/mono_arm_module/arm_root_link.xacro (robot description, xacro)
@@ -12,5 +12,5 @@
           <mesh filename="package://up1_description/meshes/mono_arm/armroot_viz.dae" scale="0.001 0.001 0.001" />
         </geometry>
-        <material name="grey" />
+        <material name="light grey" />
       </visual>
       <collision>

File: up1_description/urdf/manipulator_module/mono_arm_module/gripper.xacro (robot description, xacro)
@@ -23,5 +23,5 @@
           <mesh filename="package://up1_description/meshes/mono_arm/finger_left_viz.dae" scale="0.001 0.001 0.001" />
         </geometry>
-        <material name="grey" />
+        <material name="light grey" />
       </visual>
       <collision>
@@ -52,5 +52,5 @@
           <mesh filename="package://up1_description/meshes/mono_arm/finger_left_viz.dae" scale="0.001 0.001 0.001" />
         </geometry>
-        <material name="grey" />
+        <material name="light grey" />
       </visual>
       <collision>

File: up1_description/urdf/up1_mono.urdf (robot description, URDF)
Before this commit: robot up1, 17 links, 16 joints
Joints:
- joint base_to_left_back_wheel: origin xyz=-0.05848 0.12005 -0.02016 rpy=0 0 0.0 -> xyz=-0.05848 0.12005 -0.02016 rpy=0 0 0
- joint base_to_left_front_wheel: origin xyz=0.05605 0.12005 -0.02016 rpy=0 0 0.0 -> xyz=0.05605 0.12005 -0.02016 rpy=0 0 0
- joint base_to_right_back_wheel: origin xyz=-0.05848 -0.12005 -0.02016 rpy=0 0 0.0 -> xyz=-0.05848 -0.12005 -0.02016 rpy=0 0 0
- joint base_to_right_front_wheel: origin xyz=0.05605 -0.12005 -0.02016 rpy=0 0 0.0 -> xyz=0.05605 -0.12005 -0.02016 rpy=0 0 0

Commit message: description: fixed some confusing reflection values

File: up1_description/urdf/base_module/base_module.xacro (robot description, xacro)
@@ -47,8 +47,8 @@
     </link>
     <xacro:base_module_gazebo />
-    <xacro:wheel prefix="right" end="front" reflect="1" wheel_offset_x="0.05605" />
-    <xacro:wheel prefix="right" end="back" reflect="1" wheel_offset_x="-0.05848" />
-    <xacro:wheel prefix="left" end="front" reflect="-1" wheel_offset_x="0.05605" />
-    <xacro:wheel prefix="left" end="back" reflect="-1" wheel_offset_x="-0.05848" />
+    <xacro:wheel prefix="right" end="front" reflect="-1" wheel_offset_x="0.05605" />
+    <xacro:wheel prefix="right" end="back" reflect="-1" wheel_offset_x="-0.05848" />
+    <xacro:wheel prefix="left" end="front" reflect="1" wheel_offset_x="0.05605" />
+    <xacro:wheel prefix="left" end="back" reflect="1" wheel_offset_x="-0.05848" />
   </xacro:macro>
 </robot>

File: up1_description/urdf/base_module/wheel.xacro (robot description, xacro)
@@ -9,5 +9,5 @@
       <parent link="base_link" />
       <child link="${prefix}_${end}_wheel" />
-      <origin rpy="0 0 0" xyz="${wheel_offset_x} ${-1*reflect*wheel_offset_y} -${wheel_offset_z}" />
+      <origin rpy="0 0 0" xyz="${wheel_offset_x} ${reflect*wheel_offset_y} -${wheel_offset_z}" />
       <axis xyz="0 1 0" />
     </joint>

File: up1_description/urdf/io_module/camera.xacro (robot description, xacro)
@@ -3,5 +3,5 @@
   <xacro:property name="camera_offset_y" value="0.02150" />
   <xacro:property name="camera_offset_z" value="0.00476" />
-  <xacro:property name="camera_offset_x" value="-0.00751" />
+  <xacro:property name="camera_offset_x" value="0.00751" />
   <xacro:macro name="camera" params="prefix reflect">
     <!-- ============================   Camera   ============================ -->
@@ -10,5 +10,5 @@
       <parent link="io_link" />
       <child link="${prefix}_camera" />
-      <origin xyz="${camera_offset_x} ${reflect*camera_offset_y} ${camera_offset_z}" rpy="0 ${pi/15} 0"/>
+      <origin xyz="-${camera_offset_x} ${reflect*camera_offset_y} ${camera_offset_z}" rpy="0 ${pi/15} 0"/>
     </joint>
     <!-- Camera Link -->

File: up1_description/urdf/manipulator_module/mono_arm_module/finger.xacro (robot description, xacro)
@@ -16,5 +16,5 @@
       <child link="${prefix}_finger${num}" />
       <origin rpy="0 0 0"
-        xyz="${-1*reflect*finger_offset_x} ${finger_offset_y} ${finger_offset_z}" />
+        xyz="${reflect*finger_offset_x} ${finger_offset_y} ${finger_offset_z}" />
       <axis xyz="0 1 0" />
       <limit lower="0" upper="${finger_limit_upper}" velocity="${finger_velocity}" effort="${finger_effort}" />

File: up1_description/urdf/manipulator_module/mono_arm_module/mono_arm_module.xacro (robot description, xacro)
@@ -9,6 +9,6 @@
     <xacro:arm_root />
     <xacro:arm prefix="right" reflect="1" />
-    <xacro:finger prefix="right" num="1" reflect="-1" flip="0" fake="" />
-    <xacro:finger prefix="right" num="2" reflect="1" flip="1" fake="_fake" />
+    <xacro:finger prefix="right" num="1" reflect="1" flip="0" fake="" />
+    <xacro:finger prefix="right" num="2" reflect="-1" flip="1" fake="_fake" />
   </xacro:macro>
 </robot>

Commit message: description: fixed ride height of base and moved up1_footprint

File: up1_description/urdf/base_module/base_module.xacro (robot description, xacro)
@@ -3,29 +3,13 @@
   <xacro:include filename="$(find up1_description)/urdf/base_module/wheel.xacro" />
   <xacro:include filename="$(find up1_description)/urdf/base_module/base_module.gazebo.xacro" />
+  <xacro:property name="wheel_radius" value="0.03999" />
   <xacro:macro name="base_module">
     <!-- ============================   Base Module   ============================ -->
-    <!-- base_footprint is a fictitious link(frame) that is on the ground right below base_link origin,
-         navigation stack dedpends on this frame -->
-    <link name="up1_footprint">
-      <visual>
-        <origin xyz="0 0 0" rpy="0 0 0" />
-        <geometry>
-          <box size="0.01 0.01 0.01" />
-        </geometry>
-        <material name="white" />
-      </visual>
-      <collision>
-        <origin xyz="0 0 0" rpy="0 0 0" />
-        <geometry>
-          <box size="0.001 0.001 0.001" />
-        </geometry>
-      </collision>
-    </link>
+    <!-- Base Link -->
     <joint name="up1_footprint_joint" type="fixed">
-      <origin xyz="0 0 0" rpy="0 0 0" />
+      <origin xyz="0 0 ${wheel_radius + wheel_offset_z}" rpy="0 0 0" />
       <child link="base_link" />
       <parent link="up1_footprint"/>
     </joint>
-    <!-- Base Link -->
     <link name="base_link">
       <visual>

File: up1_description/urdf/up1.xacro (robot description, xacro)
@@ -9,4 +9,21 @@
   <xacro:include filename="$(find up1_description)/urdf/io_module/$(arg io_module)_module.xacro" />
   <xacro:include filename="$(find up1_description)/urdf/manipulator_module/$(arg manipulator_module)_module/$(arg manipulator_module)_module.xacro" />
+  <!-- up1_footprint is a fictitious link(frame) that is on the ground right below base_link origin,
+       navigation stack dedpends on this frame -->
+  <link name="up1_footprint">
+    <visual>
+      <origin xyz="0 0 0" rpy="0 0 0" />
+      <geometry>
+        <box size="0.01 0.01 0.01" />
+      </geometry>
+      <material name="white" />
+    </visual>
+    <collision>
+      <origin xyz="0 0 0" rpy="0 0 0" />
+      <geometry>
+        <box size="0.001 0.001 0.001" />
+      </geometry>
+    </collision>
+  </link>
   <xacro:base_module />
   <xacro:io_module />

File: up1_description/urdf/up1_mono.urdf (robot description, URDF)
Before this commit: robot up1, 17 links, 16 joints
Joints:
- joint up1_footprint_joint: origin xyz=0 0 0 rpy=0 0 0 -> xyz=0 0 0.06015 rpy=0 0 0
