Commit message: description: removed virtual gripper joint and link and renamed others

File: up1_description/urdf/manipulator_module/dual_arm_module/arm.xacro (robot description, xacro)
@@ -118,7 +118,7 @@
     </link>
     <!-- Arm Joint 5 -->
-    <joint name="${prefix}_armlink4_to_armlink5" type="revolute">
+    <joint name="${prefix}_armlink4_to_gripper" type="revolute">
       <parent link="${prefix}_armlink4" />
-      <child link="${prefix}_armlink5" />
+      <child link="${prefix}_gripper" />
       <origin rpy="0 ${pi/2} 0"
         xyz="${armlink5_offset_x} ${armlink5_offset_y} ${armlink5_offset_z}" />
@@ -126,6 +126,6 @@
       <limit lower="${armlink5_limit_lower}" upper="${armlink5_limit_upper}" velocity="${armlink5_velocity}" effort="${armlink5_effort}" />
     </joint>
-    <!-- Arm Link 5 -->
-    <link name="${prefix}_armlink5">
+    <!-- Gripper Link -->
+    <link name="${prefix}_gripper">
       <visual>
         <geometry>
@@ -145,13 +145,4 @@
       </inertial>
     </link>
-    <!-- Gripper Joint -->
-    <joint name="${prefix}_gripper" type="fixed">
-      <parent link="${prefix}_armlink5" />
-      <child link="${prefix}_gripper" />
-      <origin rpy="0 0 0"
-        xyz="${gripper_offset_x} ${gripper_offset_y} ${gripper_offset_z}" />
-    </joint>
-    <!-- Gripper -->
-    <link name="${prefix}_gripper" />
     <xacro:arm_gazebo prefix="${prefix}" />
     <xacro:arm_transmission prefix="${prefix}" />

File: up1_description/urdf/manipulator_module/dual_arm_module/gripper.xacro (robot description, xacro)
@@ -6,6 +6,6 @@
     <!-- ============================   Gripper   ============================ -->
     <!-- Finger Joint 1 -->
-    <joint name="${prefix}_gripper_joint" type="prismatic">
-      <parent link="${prefix}_armlink5" />
+    <joint name="${prefix}_finger_joint" type="prismatic">
+      <parent link="${prefix}_gripper" />
       <child link="${prefix}_finger1" />
       <origin rpy="0 ${pi/2} 0"
@@ -34,6 +34,6 @@
     </link>
     <!-- Finger Joint 2 -->
-    <joint name="${prefix}_gripper_joint_fake" type="prismatic">
-      <parent link="${prefix}_armlink5" />
+    <joint name="${prefix}_finger_joint_fake" type="prismatic">
+      <parent link="${prefix}_gripper" />
       <child link="${prefix}_finger2" />
       <origin rpy="0 ${-pi/2} 0"
@@ -41,5 +41,5 @@
       <axis xyz="0 0 1" />
       <limit lower="0" upper="${finger_limit_upper}" velocity="${finger2_velocity}" effort="${finger2_effort}" />
-      <mimic joint="${prefix}_gripper_joint" multiplier="1" offset="0"/>
+      <mimic joint="${prefix}_finger_joint" multiplier="1" offset="0"/>
     </joint>
     <!-- Finger Link 2 -->
