Commit message: moveit: progress save

File: up1_description/urdf/manipulator_module/dual_arm_module/gripper.transmission.xacro (robot description, xacro)
@@ -5,16 +5,7 @@
     <transmission name="${prefix}_gripper_trans">
       <type>transmission_interface/SimpleTransmission</type>
-      <joint name="${prefix}_finger_joint">
-        <hardwareInterface>PositionJointInterface</hardwareInterface>
-      </joint>
-      <actuator name="${prefix}_gripper_motor">
-        <mechanicalReduction>1</mechanicalReduction>
-      </actuator>
-    </transmission>
-    <transmission name="${prefix}_gripper_trans">
-      <type>transmission_interface/SimpleTransmission</type>
-      <joint name="${prefix}_finger_joint_fake">
-        <hardwareInterface>PositionJointInterface</hardwareInterface>
-      </joint>
+      <joint name="${prefix}_finger_joint" />
+      <joint name="${prefix}_finger_joint_fake" />
+      <hardwareInterface>PositionJointInterface</hardwareInterface>
       <actuator name="${prefix}_gripper_motor">
         <mechanicalReduction>1</mechanicalReduction>
