Commit message: description: updated mono arm based on right arm from dual module

File: up1_description/urdf/manipulator_module/mono_arm_module/arm.gazebo.xacro (robot description, xacro)
@@ -1,6 +1,6 @@
 <?xml version="1.0"?>
 <robot xmlns:xacro="http://www.ros.org/wiki/xacro" name="up1">
-  <!-- ============================   Arm   ============================ -->
   <xacro:macro name="arm_gazebo" params="prefix">
+    <!-- ============================   Arm Gazebo  ============================ -->
     <gazebo reference="${prefix}_armlink1">
       <turnGravityOff>true</turnGravityOff>
@@ -15,5 +15,5 @@
       <turnGravityOff>true</turnGravityOff>
     </gazebo>
-    <gazebo reference="${prefix}_armlink5">
+    <gazebo reference="${prefix}_gripper">
       <turnGravityOff>true</turnGravityOff>
     </gazebo>

File: up1_description/urdf/manipulator_module/mono_arm_module/arm.xacro (robot description, xacro)
@@ -1,12 +1,54 @@
 <?xml version="1.0"?>
 <robot xmlns:xacro="http://www.ros.org/wiki/xacro" name="up1">
-  <xacro:include filename="$(find up1_description)/urdf/mono_arm_module/arm.gazebo.xacro" />
-  <!-- ============================   Arm   ============================ -->
+  <xacro:include filename="$(find up1_description)/urdf/manipulator_module/mono_arm_module/arm.gazebo.xacro" />
+  <xacro:include filename="$(find up1_description)/urdf/manipulator_module/mono_arm_module/arm.transmission.xacro" />
+  <xacro:property name="armlink1_offset_x" value="0.01777" />
+  <xacro:property name="armlink1_offset_y" value="0.07385" />
+  <xacro:property name="armlink1_offset_z" value="0.01853" />
+  <xacro:property name="armlink2_offset_x" value="0" />
+  <xacro:property name="armlink2_offset_y" value="0" />
+  <xacro:property name="armlink2_offset_z" value="-0.07038" />
+  <xacro:property name="armlink3_offset_x" value="0" />
+  <xacro:property name="armlink3_offset_y" value="0.09602" />
+  <xacro:property name="armlink3_offset_z" value="0" />
+  <xacro:property name="armlink4_offset_x" value="0" />
+  <xacro:property name="armlink4_offset_y" value="0" />
+  <xacro:property name="armlink4_offset_z" value="0.05588" />
+  <xacro:property name="gripper_offset_x" value="0" />
+  <xacro:property name="gripper_offset_y" value="0.07641" />
+  <xacro:property name="gripper_offset_z" value="0" />
+  <xacro:property name="armlink1_limit_lower" value="${-pi/2}" />
+  <xacro:property name="armlink1_limit_upper" value="${pi/2}" />
+  <xacro:property name="armlink2_limit_lower" value="${-pi/2}" />
+  <xacro:property name="armlink2_limit_upper" value="${pi/2}" />
+  <xacro:property name="armlink3_limit_lower" value="${-pi/2}" />
+  <xacro:property name="armlink3_limit_upper" value="${pi/2}" />
+  <xacro:property name="armlink4_limit_lower" value="${-pi/2}" />
+  <xacro:property name="armlink4_limit_upper" value="${pi/2}" />
+  <xacro:property name="gripper_limit_lower" value="${-pi/2}" />
+  <xacro:property name="gripper_limit_upper" value="${pi/2}" />
+  <xacro:property name="finger_limit_upper" value="0.018" />
+  <xacro:property name="armlink1_velocity" value="1" />
+  <xacro:property name="armlink2_velocity" value="1" />
+  <xacro:property name="armlink3_velocity" value="1" />
+  <xacro:property name="armlink4_velocity" value="1" />
+  <xacro:property name="gripper_velocity" value="1" />
+  <xacro:property name="finger1_velocity" value="1" />
+  <xacro:property name="finger2_velocity" value="1" />
+  <xacro:property name="armlink1_effort" value="6.0" />
+  <xacro:property name="armlink2_effort" value="6.0" />
+  <xacro:property name="armlink3_effort" value="6.0" />
+  <xacro:property name="armlink4_effort" value="6.0" />
+  <xacro:property name="gripper_effort" value="6.0" />
+  <xacro:property name="finger1_effort" value="6.0" />
+  <xacro:property name="finger2_effort" value="6.0" />
   <xacro:macro name="arm" params="prefix reflect">
+    <!-- ============================   Arm   ============================ -->
     <!-- Arm Joint 1 -->
     <joint name="${prefix}_armroot_to_armlink1" type="revolute">
       <parent link="armroot_link" />
       <child link="${prefix}_armlink1" />
-      <origin rpy="0 0 0" xyz="0 0 0" />
+      <origin rpy="${-reflect*pi/6} ${pi} 0"
+        xyz="${armlink1_offset_x} ${-reflect*armlink1_offset_y} ${armlink1_offset_z}" />
       <axis xyz="0 0 1" />
       <limit lower="${armlink1_limit_lower}" upper="${armlink1_limit_upper}" velocity="${armlink1_velocity}" effort="${armlink1_effort}" />
@@ -26,6 +68,5 @@
       </collision>
       <inertial>
-        <mass value="0.17905"/>
-        <!-- inertia is wrong, get update from Daniel -->
+        <mass value="0.06985"/>
         <inertia ixx="0.00023448766" ixy="0.0000000027" ixz="0.00000001913"
                  iyy="0.00024004726" iyz="-0.0000015393" izz="0.00007431363"/>
@@ -36,5 +77,6 @@
       <parent link="${prefix}_armlink1" />
       <child link="${prefix}_armlink2" />
-      <origin rpy="0 0 0" xyz="0 0 0" />
+      <origin rpy="${pi/2} ${pi} 0"
+        xyz="${armlink2_offset_x} ${armlink2_offset_y} ${armlink2_offset_z}" />
       <axis xyz="0 0 ${reflect*1}" />
       <limit lower="${armlink2_limit_lower}" upper="${armlink2_limit_upper}" velocity="${armlink2_velocity}" effort="${armlink2_effort}" />
@@ -54,6 +96,5 @@
       </collision>
       <inertial>
-        <mass value="0.49779"/>
-        <!-- inertia is wrong, get update from Daniel -->
+        <mass value="0.07067"/>
         <inertia ixx="0.00029708797" ixy="-0.00000000444" ixz="0.00000000068"
                  iyy="0.0000799845" iyz="-0.00000174097" izz="0.00026073683"/>
@@ -64,5 +105,6 @@
       <parent link="${prefix}_armlink2" />
       <child link="${prefix}_armlink3" />
-      <origin rpy="0 0 0" xyz="0 0 0" />
+      <origin rpy="${-pi/2} ${pi} 0"
+        xyz="${armlink3_offset_x} ${armlink3_offset_y} ${armlink3_offset_z}" />
       <axis xyz="0 0 -1" />
       <limit lower="${armlink3_limit_lower}" upper="${armlink3_limit_upper}" velocity="${armlink3_velocity}" effort="${armlink3_effort}" />
@@ -91,5 +133,6 @@
       <parent link="${prefix}_armlink3" />
       <child link="${prefix}_armlink4" />
-      <origin rpy="0 0 0" xyz="0 0 0" />
+      <origin rpy="${pi/2} 0 0"
+        xyz="${armlink4_offset_x} ${armlink4_offset_y} ${armlink4_offset_z}" />
       <axis xyz="0 0 ${reflect*1}" />
       <limit lower="${armlink4_limit_lower}" upper="${armlink4_limit_upper}" velocity="${armlink4_velocity}" effort="${armlink4_effort}" />
@@ -115,13 +158,14 @@
     </link>
     <!-- Arm Joint 5 -->
-    <joint name="${prefix}_armlink4_to_armlink5" type="revolute">
+    <joint name="${prefix}_armlink4_to_gripper" type="revolute">
       <parent link="${prefix}_armlink4" />
-      <child link="${prefix}_armlink5" />
-      <origin rpy="0 0 0" xyz="0 0 0" />
+      <child link="${prefix}_gripper" />
+      <origin rpy="0 ${pi/2} 0"
+        xyz="${gripper_offset_x} ${gripper_offset_y} ${gripper_offset_z}" />
       <axis xyz="0 0 ${-reflect*1}" />
-      <limit lower="${armlink5_limit_lower}" upper="${armlink5_limit_upper}" velocity="${armlink5_velocity}" effort="${armlink5_effort}" />
+      <limit lower="${gripper_limit_lower}" upper="${gripper_limit_upper}" velocity="${gripper_velocity}" effort="${gripper_effort}" />
     </joint>
-    <!-- Arm Link 5 -->
-    <link name="${prefix}_armlink5">
+    <!-- Gripper Link -->
+    <link name="${prefix}_gripper">
       <visual>
         <geometry>
@@ -141,13 +185,6 @@
       </inertial>
     </link>
-    <!-- Gripper Joint -->
-    <joint name="${prefix}_gripper" type="fixed">
-      <parent link="${prefix}_armlink5" />
-      <child link="${prefix}_gripper" />
-      <origin rpy="0 0 0" xyz="0 0 0" />
-    </joint>
-    <!-- Gripper -->
-    <link name="${prefix}_gripper" />
     <xacro:arm_gazebo prefix="${prefix}" />
+    <xacro:arm_transmission prefix="${prefix}" />
   </xacro:macro>
 </robot>

File: up1_description/urdf/manipulator_module/mono_arm_module/gripper.gazebo.xacro (robot description, xacro)
@@ -1,6 +1,6 @@
 <?xml version="1.0"?>
 <robot xmlns:xacro="http://www.ros.org/wiki/xacro" name="up1">
-  <!-- ============================   Gripper   ============================ -->
   <xacro:macro name="gripper_gazebo" params="prefix">
+    <!-- ============================   Gripper Gazebo   ============================ -->
     <gazebo reference="${prefix}_finger1">
       <turnGravityOff>true</turnGravityOff>

File: up1_description/urdf/manipulator_module/mono_arm_module/gripper.xacro (robot description, xacro)
@@ -1,10 +1,14 @@
 <?xml version="1.0"?>
 <robot xmlns:xacro="http://www.ros.org/wiki/xacro" name="up1">
-  <xacro:include filename="$(find up1_description)/urdf/mono_arm_module/gripper.gazebo.xacro" />
-  <!-- ============================   Gripper   ============================ -->
+  <xacro:include filename="$(find up1_description)/urdf/manipulator_module/mono_arm_module/gripper.gazebo.xacro" />
+  <xacro:include filename="$(find up1_description)/urdf/manipulator_module/mono_arm_module/gripper.transmission.xacro" />
+  <xacro:property name="finger_offset_x" value="0.01800" />
+  <xacro:property name="finger_offset_y" value="0.08121" />
+  <xacro:property name="finger_offset_z" value="0" />
   <xacro:macro name="gripper" params="prefix reflect">
+    <!-- ============================   Gripper   ============================ -->
     <!-- Finger Joint 1 -->
-    <joint name="${prefix}_gripper_joint" type="prismatic">
-      <parent link="${prefix}_armlink5" />
+    <joint name="${prefix}_finger_joint" type="prismatic">
+      <parent link="${prefix}_gripper" />
       <child link="${prefix}_finger1" />
       <origin rpy="0 ${pi/2} 0"
@@ -33,6 +37,6 @@
     </link>
     <!-- Finger Joint 2 -->
-    <joint name="${prefix}_gripper_joint_fake" type="prismatic">
-      <parent link="${prefix}_armlink5" />
+    <joint name="${prefix}_finger_joint_fake" type="prismatic">
+      <parent link="${prefix}_gripper" />
       <child link="${prefix}_finger2" />
       <origin rpy="0 ${-pi/2} 0"
@@ -40,5 +44,5 @@
       <axis xyz="0 0 1" />
       <limit lower="0" upper="${finger_limit_upper}" velocity="${finger2_velocity}" effort="${finger2_effort}" />
-      <mimic joint="${prefix}_gripper_joint" multiplier="1" offset="0"/>
+      <mimic joint="${prefix}_finger_joint" multiplier="1" offset="0"/>
     </joint>
     <!-- Finger Link 2 -->
@@ -62,4 +66,5 @@
     </link>
     <xacro:gripper_gazebo prefix="${prefix}" />
+    <xacro:gripper_transmission prefix="${prefix}" />
   </xacro:macro>
 </robot>

File: up1_description/urdf/manipulator_module/mono_arm_module/mono_arm_module.xacro (robot description, xacro)
@@ -1,38 +1,19 @@
 <?xml version="1.0"?>
 <robot xmlns:xacro="http://www.ros.org/wiki/xacro" name="up1">
-  <xacro:include filename="$(find up1_description)/urdf/mono_arm_module/arm.xacro" />
-  <xacro:include filename="$(find up1_description)/urdf/mono_arm_module/gripper.xacro" />
-  <xacro:include filename="$(find up1_description)/urdf/mono_arm_module/arm_module.gazebo.xacro" />
-  <!-- ============================   Arm Module   ============================ -->
+  <xacro:include filename="$(find up1_description)/urdf/manipulator_module/mono_arm_module/arm_root_link.xacro" />
+  <xacro:include filename="$(find up1_description)/urdf/manipulator_module/mono_arm_module/arm.xacro" />
+  <xacro:include filename="$(find up1_description)/urdf/manipulator_module/mono_arm_module/gripper.xacro" />
   <xacro:macro name="manipulator_module">
+    <!-- ============================   Dual Arm Module   ============================ -->
+    <!-- This xacro group is intended to be used in a full UP1 robot URDF -->
     <!-- Armroot Joint -->
     <joint name="base_to_armroot" type="fixed">
       <parent link="base_link" />
       <child link="armroot_link" />
-      <origin xyz="0.003804 -0.008022 0.001964" />
+      <origin xyz="${armroot_offset_x} ${armroot_offset_y} ${armroot_offset_z}" />
     </joint>
-    <!-- Armroot Link -->
-    <link name="armroot_link">
-      <visual>
-        <geometry>
-          <mesh filename="package://up1_description/meshes/mono_arm/armroot.stl" scale="0.001 0.001 0.001" />
-        </geometry>
-        <material name="grey" />
-      </visual>
-      <collision>
-        <geometry>
-          <mesh filename="package://up1_description/meshes/mono_arm/armroot.stl" scale="0.001 0.001 0.001" />
-        </geometry>
-      </collision>
-      <inertial>
-        <mass value="0.17621"/>
-        <!-- inertia is wrong, get update from Daniel -->
-        <inertia ixx="0.00096240277" ixy="-0.00000350376" ixz="0.00002354169"
-                 iyy="0.00057897825" iyz="0.00000127419" izz="0.00134814249"/>
-      </inertial>
-    </link>
-    <xacro:arm_module_gazebo />
-    <xacro:arm prefix="mono" reflect="1" />
-    <xacro:gripper prefix="mono" reflect="1" />
+    <xacro:arm_root_link />
+    <xacro:arm prefix="right" reflect="1" />
+    <xacro:gripper prefix="right" reflect="1" />
   </xacro:macro>
 </robot>
