Commit message: description: moved arm_root and renamed file

File: up1_description/urdf/manipulator_module/mono_arm_module/arm_root.xacro (robot description, xacro)
@@ -4,6 +4,12 @@
   <xacro:property name="armroot_offset_x" value="0.00556" />
   <xacro:property name="armroot_offset_y" value="0.0" />
-  <xacro:macro name="arm_root_link">
-    <!-- ============================   Arm Root Link   ============================ -->
+  <xacro:macro name="arm_root">
+    <!-- ============================   Arm Root  ============================ -->
+    <!-- Armroot Joint -->
+    <joint name="base_to_armroot" type="fixed">
+      <parent link="base_link" />
+      <child link="armroot_link" />
+      <origin xyz="${armroot_offset_x} ${armroot_offset_y} ${armroot_offset_z}" />
+    </joint>
     <!-- Armroot Link -->
     <link name="armroot_link">

File: up1_description/urdf/manipulator_module/mono_arm_module/mono_arm_module.xacro (robot description, xacro)
@@ -1,5 +1,5 @@
 <?xml version="1.0"?>
 <robot xmlns:xacro="http://www.ros.org/wiki/xacro" name="up1">
-  <xacro:include filename="$(find up1_description)/urdf/manipulator_module/mono_arm_module/arm_root_link.xacro" />
+  <xacro:include filename="$(find up1_description)/urdf/manipulator_module/mono_arm_module/arm_root.xacro" />
   <xacro:include filename="$(find up1_description)/urdf/manipulator_module/mono_arm_module/arm.xacro" />
   <xacro:include filename="$(find up1_description)/urdf/manipulator_module/mono_arm_module/gripper.xacro" />
@@ -7,11 +7,5 @@
     <!-- ============================   Mono Arm Module   ============================ -->
     <!-- This xacro group is intended to be used in a full UP1 robot URDF -->
-    <!-- Armroot Joint -->
-    <joint name="base_to_armroot" type="fixed">
-      <parent link="base_link" />
-      <child link="armroot_link" />
-      <origin xyz="${armroot_offset_x} ${armroot_offset_y} ${armroot_offset_z}" />
-    </joint>
-    <xacro:arm_root_link />
+    <xacro:arm_root />
     <xacro:arm prefix="right" reflect="1" />
     <xacro:gripper prefix="right" num="1" reflect="-1" flip="0" fake="" />
