Commit message: description: renamed instances of gripper to finger

File: up1_description/urdf/manipulator_module/mono_arm_module/finger.gazebo.xacro (robot description, xacro)
@@ -1,5 +1,5 @@
 <?xml version="1.0"?>
 <robot xmlns:xacro="http://www.ros.org/wiki/xacro" name="up1">
-  <xacro:macro name="gripper_gazebo" params="prefix">
+  <xacro:macro name="finger_gazebo" params="prefix">
     <!-- ============================   Gripper Gazebo   ============================ -->
     <gazebo reference="${prefix}_finger1">

File: up1_description/urdf/manipulator_module/mono_arm_module/finger.transmission.xacro (robot description, xacro)
@@ -1,21 +1,21 @@
 <?xml version="1.0"?>
 <robot xmlns:xacro="http://www.ros.org/wiki/xacro" name="up1">
-  <xacro:macro name="gripper_transmission" params="prefix">
-    <!-- ============================   Gripper Transmission   ============================ -->
-    <transmission name="${prefix}_gripper_trans">
+  <xacro:macro name="finger_transmission" params="prefix">
+    <!-- ============================   finger Transmission   ============================ -->
+    <transmission name="${prefix}_finger_trans">
       <type>transmission_interface/SimpleTransmission</type>
       <joint name="${prefix}_finger_joint">
         <hardwareInterface>PositionJointInterface</hardwareInterface>
       </joint>
-      <actuator name="${prefix}_gripper_motor">
+      <actuator name="${prefix}_finger_motor">
         <mechanicalReduction>1</mechanicalReduction>
       </actuator>
     </transmission>
-    <transmission name="${prefix}_gripper_trans">
+    <transmission name="${prefix}_finger_trans">
       <type>transmission_interface/SimpleTransmission</type>
       <joint name="${prefix}_finger_joint_fake">
         <hardwareInterface>PositionJointInterface</hardwareInterface>
       </joint>
-      <actuator name="${prefix}_gripper_motor">
+      <actuator name="${prefix}_finger_motor">
         <mechanicalReduction>1</mechanicalReduction>
       </actuator>

File: up1_description/urdf/manipulator_module/mono_arm_module/finger.xacro (robot description, xacro)
@@ -1,6 +1,6 @@
 <?xml version="1.0"?>
 <robot xmlns:xacro="http://www.ros.org/wiki/xacro" name="up1">
-  <xacro:include filename="$(find up1_description)/urdf/manipulator_module/mono_arm_module/gripper.gazebo.xacro" />
-  <xacro:include filename="$(find up1_description)/urdf/manipulator_module/mono_arm_module/gripper.transmission.xacro" />
+  <xacro:include filename="$(find up1_description)/urdf/manipulator_module/mono_arm_module/finger.gazebo.xacro" />
+  <xacro:include filename="$(find up1_description)/urdf/manipulator_module/mono_arm_module/finger.transmission.xacro" />
   <xacro:property name="finger_offset_x" value="0.0" />
   <xacro:property name="finger_offset_y" value="0.0" />
@@ -9,6 +9,6 @@
   <xacro:property name="finger_velocity" value="1" />
   <xacro:property name="finger_effort" value="6.0" />
-  <xacro:macro name="gripper" params="prefix num reflect flip fake">
-    <!-- ============================   Gripper   ============================ -->
+  <xacro:macro name="finger" params="prefix num reflect flip fake">
+    <!-- ============================   Finger   ============================ -->
     <!-- Finger Joint -->
     <joint name="${prefix}_finger_joint${fake}" type="prismatic">
@@ -39,6 +39,6 @@
       </inertial>
     </link>
-    <xacro:gripper_gazebo prefix="${prefix}" />
-    <xacro:gripper_transmission prefix="${prefix}" />
+    <xacro:finger_gazebo prefix="${prefix}" />
+    <xacro:finger_transmission prefix="${prefix}" />
   </xacro:macro>
 </robot>

File: up1_description/urdf/manipulator_module/mono_arm_module/mono_arm_module.xacro (robot description, xacro)
@@ -3,5 +3,5 @@
   <xacro:include filename="$(find up1_description)/urdf/manipulator_module/mono_arm_module/arm_root.xacro" />
   <xacro:include filename="$(find up1_description)/urdf/manipulator_module/mono_arm_module/arm.xacro" />
-  <xacro:include filename="$(find up1_description)/urdf/manipulator_module/mono_arm_module/gripper.xacro" />
+  <xacro:include filename="$(find up1_description)/urdf/manipulator_module/mono_arm_module/finger.xacro" />
   <xacro:macro name="manipulator_module">
     <!-- ============================   Mono Arm Module   ============================ -->
@@ -9,6 +9,6 @@
     <xacro:arm_root />
     <xacro:arm prefix="right" reflect="1" />
-    <xacro:gripper prefix="right" num="1" reflect="-1" flip="0" fake="" />
-    <xacro:gripper prefix="right" num="2" reflect="1" flip="1" fake="_fake" />
+    <xacro:finger prefix="right" num="1" reflect="-1" flip="0" fake="" />
+    <xacro:finger prefix="right" num="2" reflect="1" flip="1" fake="_fake" />
   </xacro:macro>
 </robot>
