Commit message: description: updated offsets for some links in new mono arm

File: up1_description/urdf/manipulator_module/mono_arm_module/arm.xacro (robot description, xacro)
@@ -3,10 +3,10 @@
   <xacro:include filename="$(find up1_description)/urdf/manipulator_module/mono_arm_module/arm.gazebo.xacro" />
   <xacro:include filename="$(find up1_description)/urdf/manipulator_module/mono_arm_module/arm.transmission.xacro" />
-  <xacro:property name="armlink1_offset_x" value="0.01777" />
-  <xacro:property name="armlink1_offset_y" value="0.07385" />
-  <xacro:property name="armlink1_offset_z" value="0.01853" />
+  <xacro:property name="armlink1_offset_x" value="0.01398" />
+  <xacro:property name="armlink1_offset_y" value="0" />
+  <xacro:property name="armlink1_offset_z" value="0.0402" />
   <xacro:property name="armlink2_offset_x" value="0" />
   <xacro:property name="armlink2_offset_y" value="0" />
-  <xacro:property name="armlink2_offset_z" value="-0.07038" />
+  <xacro:property name="armlink2_offset_z" value="-0.0553" />
   <xacro:property name="armlink3_offset_x" value="0" />
   <xacro:property name="armlink3_offset_y" value="0.09602" />
@@ -49,5 +49,5 @@
       <parent link="armroot_link" />
       <child link="${prefix}_armlink1" />
-      <origin rpy="${-reflect*pi/6} ${pi} 0"
+      <origin rpy="0 ${pi} 0"
         xyz="${armlink1_offset_x} ${-reflect*armlink1_offset_y} ${armlink1_offset_z}" />
       <axis xyz="0 0 1" />

File: up1_description/urdf/manipulator_module/mono_arm_module/arm_root_link.xacro (robot description, xacro)
@@ -1,7 +1,7 @@
 <?xml version="1.0"?>
 <robot xmlns:xacro="http://www.ros.org/wiki/xacro" name="up1">
-  <xacro:property name="armroot_offset_z" value="0.08022" />
-  <xacro:property name="armroot_offset_x" value="-0.03804" />
-  <xacro:property name="armroot_offset_y" value="0.01963" />
+  <xacro:property name="armroot_offset_z" value="0.03876" />
+  <xacro:property name="armroot_offset_x" value="-0.00869" />
+  <xacro:property name="armroot_offset_y" value="0.0" />
   <xacro:macro name="arm_root_link">
     <!-- ============================   Arm Root Link   ============================ -->

Commit message: description: fixed joint velocity limits

File: up1_description/urdf/manipulator_module/mono_arm_module/arm.xacro (robot description, xacro)
@@ -29,9 +29,9 @@
   <xacro:property name="gripper_limit_upper" value="${pi/2}" />
   <xacro:property name="finger_limit_upper" value="0.018" />
-  <xacro:property name="armlink1_velocity" value="1" />
-  <xacro:property name="armlink2_velocity" value="1" />
-  <xacro:property name="armlink3_velocity" value="1" />
-  <xacro:property name="armlink4_velocity" value="1" />
-  <xacro:property name="gripper_velocity" value="1" />
+  <xacro:property name="armlink1_velocity" value="5.236" />
+  <xacro:property name="armlink2_velocity" value="4.553" />
+  <xacro:property name="armlink3_velocity" value="5.236" />
+  <xacro:property name="armlink4_velocity" value="5.236" />
+  <xacro:property name="gripper_velocity" value="5.236" />
   <xacro:property name="finger1_velocity" value="1" />
   <xacro:property name="finger2_velocity" value="1" />

Commit message: description: updated fingers

File: up1_description/urdf/manipulator_module/mono_arm_module/arm.xacro (robot description, xacro)
@@ -28,5 +28,4 @@
   <xacro:property name="gripper_limit_lower" value="${-pi/2}" />
   <xacro:property name="gripper_limit_upper" value="${pi/2}" />
-  <xacro:property name="finger_limit_upper" value="0.018" />
   <xacro:property name="armlink1_velocity" value="5.236" />
   <xacro:property name="armlink2_velocity" value="4.553" />
@@ -34,6 +33,4 @@
   <xacro:property name="armlink4_velocity" value="5.236" />
   <xacro:property name="gripper_velocity" value="5.236" />
-  <xacro:property name="finger1_velocity" value="1" />
-  <xacro:property name="finger2_velocity" value="1" />
   <xacro:property name="armlink1_effort" value="6.0" />
   <xacro:property name="armlink2_effort" value="6.0" />
@@ -41,6 +38,4 @@
   <xacro:property name="armlink4_effort" value="6.0" />
   <xacro:property name="gripper_effort" value="6.0" />
-  <xacro:property name="finger1_effort" value="6.0" />
-  <xacro:property name="finger2_effort" value="6.0" />
   <xacro:macro name="arm" params="prefix reflect">
     <!-- ============================   Arm   ============================ -->

File: up1_description/urdf/manipulator_module/mono_arm_module/gripper.xacro (robot description, xacro)
@@ -6,20 +6,23 @@
   <xacro:property name="finger_offset_y" value="0.0" />
   <xacro:property name="finger_offset_z" value="0.07961" />
-  <xacro:macro name="gripper" params="prefix reflect">
+  <xacro:property name="finger_limit_upper" value="0.018" />
+  <xacro:property name="finger_velocity" value="1" />
+  <xacro:property name="finger_effort" value="6.0" />
+  <xacro:macro name="gripper" params="prefix num reflect flip fake">
     <!-- ============================   Gripper   ============================ -->
-    <!-- Finger Joint 1 -->
-    <joint name="${prefix}_finger_joint" type="prismatic">
+    <!-- Finger Joint -->
+    <joint name="${prefix}_finger_joint${fake}" type="prismatic">
       <parent link="${prefix}_gripper" />
-      <child link="${prefix}_finger1" />
+      <child link="${prefix}_finger${num}" />
       <origin rpy="0 0 0"
-        xyz="${-finger_offset_x} ${finger_offset_y} ${finger_offset_z}" />
+        xyz="${-1*reflect*finger_offset_x} ${finger_offset_y} ${finger_offset_z}" />
       <axis xyz="0 1 0" />
-      <limit lower="0" upper="${finger_limit_upper}" velocity="${finger1_velocity}" effort="${finger1_effort}" />
+      <limit lower="0" upper="${finger_limit_upper}" velocity="${finger_velocity}" effort="${finger_effort}" />
     </joint>
     <!-- Finger Link 1 -->
-    <link name="${prefix}_finger1">
+    <link name="${prefix}_finger${num}">
       <visual>
         <geometry>
-          <mesh filename="package://up1_description/meshes/mono_arm/finger_left_viz.dae" scale="0.001 0.001 0.001" />
+          <mesh filename="package://up1_description/meshes/mono_arm/finger_${num}_viz.dae" scale="0.001 0.001 0.001" />
         </geometry>
         <material name="light grey" />
@@ -27,34 +30,5 @@
       <collision>
         <geometry>
-          <mesh filename="package://up1_description/meshes/mono_arm/finger_left.stl" scale="0.001 0.001 0.001" />
-        </geometry>
-      </collision>
-      <inertial>
-        <mass value="0.01174"/>
-        <inertia ixx="0.00000285949" ixy="-0.00000001641" ixz="0.00000001803"
-                 iyy="0.00000203198" iyz="-0.00000077289" izz="0.00000299021"/>
-      </inertial>
-    </link>
-    <!-- Finger Joint 2 -->
-    <joint name="${prefix}_finger_joint_fake" type="prismatic">
-      <parent link="${prefix}_gripper" />
-      <child link="${prefix}_finger2" />
-      <origin rpy="0 0 ${pi}"
-        xyz="${finger_offset_x} ${finger_offset_y} ${finger_offset_z}" />
-      <axis xyz="0 1 0" />
-      <limit lower="0" upper="${finger_limit_upper}" velocity="${finger2_velocity}" effort="${finger2_effort}" />
-      <mimic joint="${prefix}_finger_joint" multiplier="1" offset="0"/>
-    </joint>
-    <!-- Finger Link 2 -->
-    <link name="${prefix}_finger2">
-      <visual>
-        <geometry>
-          <mesh filename="package://up1_description/meshes/mono_arm/finger_left_viz.dae" scale="0.001 0.001 0.001" />
-        </geometry>
-        <material name="light grey" />
-      </visual>
-      <collision>
-        <geometry>
-          <mesh filename="package://up1_description/meshes/mono_arm/finger_left.stl" scale="0.001 0.001 0.001" />
+          <mesh filename="package://up1_description/meshes/mono_arm/finger_${num}.stl" scale="0.001 0.001 0.001" />
         </geometry>
       </collision>

File: up1_description/urdf/manipulator_module/mono_arm_module/mono_arm_module.xacro (robot description, xacro)
@@ -5,5 +5,5 @@
   <xacro:include filename="$(find up1_description)/urdf/manipulator_module/mono_arm_module/gripper.xacro" />
   <xacro:macro name="manipulator_module">
-    <!-- ============================   Dual Arm Module   ============================ -->
+    <!-- ============================   Mono Arm Module   ============================ -->
     <!-- This xacro group is intended to be used in a full UP1 robot URDF -->
     <!-- Armroot Joint -->
@@ -15,5 +15,6 @@
     <xacro:arm_root_link />
     <xacro:arm prefix="right" reflect="1" />
-    <xacro:gripper prefix="right" reflect="1" />
+    <xacro:gripper prefix="right" num="1" reflect="-1" flip="0" fake="" />
+    <xacro:gripper prefix="right" num="2" reflect="1" flip="1" fake="_fake" />
   </xacro:macro>
 </robot>

File: up1_description/urdf/up1_mono.urdf (robot description, URDF)
Before this commit: robot up1, 17 links, 16 joints
Links:
- link right_finger1: geometry collision mesh filename=package://up1_description/meshes/mono_arm/finger_1.stl scale=0.001 0.001 0.001; visual mesh filename=package://up1_description/meshes/mono_arm/finger_1_viz.dae scale=0.001 0.001 0.001
- link right_finger2: geometry collision mesh filename=package://up1_description/meshes/mono_arm/finger_2.stl scale=0.001 0.001 0.001; visual mesh filename=package://up1_description/meshes/mono_arm/finger_2_viz.dae scale=0.001 0.001 0.001
Joints:
- joint right_finger_joint: origin xyz=-0.0 0.0 0.07961 rpy=0 0 0 -> xyz=0.0 0.0 0.07961 rpy=0 0 0
- joint right_finger_joint_fake: mimic joint=right_finger_joint multiplier=1 offset=0 -> (none); origin xyz=0.0 0.0 0.07961 rpy=0 0 3.14159 -> xyz=-0.0 0.0 0.07961 rpy=0 0 0

Commit message: description: fixed some urdf issues

File: up1_description/urdf/manipulator_module/mono_arm_module/arm.xacro (robot description, xacro)
@@ -44,7 +44,7 @@
       <parent link="armroot_link" />
       <child link="${prefix}_armlink1" />
-      <origin rpy="0 0 0"
+      <origin rpy="0 0 ${pi}"
         xyz="${armlink1_offset_x} ${armlink1_offset_y} ${armlink1_offset_z}" />
-      <axis xyz="0 0 1" />
+      <axis xyz="0 0 -1" />
       <limit lower="${armlink1_limit_lower}" upper="${armlink1_limit_upper}" velocity="${armlink1_velocity}" effort="${armlink1_effort}" />
     </joint>
@@ -102,5 +102,5 @@
       <origin rpy="0 0 0"
         xyz="${armlink3_offset_x} ${armlink3_offset_y} ${armlink3_offset_z}" />
-      <axis xyz="0 0 1" />
+      <axis xyz="0 0 -1" />
       <limit lower="${armlink3_limit_lower}" upper="${armlink3_limit_upper}" velocity="${armlink3_velocity}" effort="${armlink3_effort}" />
     </joint>
@@ -130,5 +130,5 @@
       <origin rpy="0 0 0"
         xyz="${armlink4_offset_x} ${armlink4_offset_y} ${armlink4_offset_z}" />
-      <axis xyz="0 1 0" />
+      <axis xyz="0 -1 0" />
       <limit lower="${armlink4_limit_lower}" upper="${armlink4_limit_upper}" velocity="${armlink4_velocity}" effort="${armlink4_effort}" />
     </joint>
@@ -156,7 +156,7 @@
       <parent link="${prefix}_armlink4" />
       <child link="${prefix}_gripper" />
-      <origin rpy="0 0 0"
+      <origin rpy="0 0 ${pi/2}"
         xyz="${gripper_offset_x} ${gripper_offset_y} ${gripper_offset_z}" />
-      <axis xyz="1 0 0" />
+      <axis xyz="0 1 0" />
       <limit lower="${gripper_limit_lower}" upper="${gripper_limit_upper}" velocity="${gripper_velocity}" effort="${gripper_effort}" />
     </joint>

File: up1_description/urdf/up1_mono.urdf (robot description, URDF)
Before this commit: robot up1, 17 links, 16 joints
Joints:
- joint right_armlink2_to_armlink3: axis 0 0 1 -> 0 0 -1
- joint right_armlink3_to_armlink4: axis 0 1 0 -> 0 -1 0
- joint right_armlink4_to_gripper: axis 1 0 0 -> 0 1 0; origin xyz=0.0 0.0 0.08471 rpy=0 0 0 -> xyz=0.0 0.0 0.08471 rpy=0 0 1.570795
- joint right_armroot_to_armlink1: axis 0 0 1 -> 0 0 -1; origin xyz=0.0 0.0 0.03099 rpy=0 0 0 -> xyz=0.0 0.0 0.03099 rpy=0 0 3.14159
