Commit message: description: added camera.dae

File: up1_description/urdf/io_module/camera.xacro (robot description, xacro)
@@ -13,5 +13,5 @@
       <visual>
         <geometry>
-          <mesh filename="package://up1_description/meshes/io/camera.stl" scale="0.001 0.001 0.001" />
+          <mesh filename="package://up1_description/meshes/io/camera.dae" scale="0.001 0.001 0.001" />
         </geometry>
         <material name="black" />
@@ -19,5 +19,5 @@
       <collision>
         <geometry>
-          <mesh filename="package://up1_description/meshes/io/camera.stl" scale="0.001 0.001 0.001" />
+          <mesh filename="package://up1_description/meshes/io/camera.dae" scale="0.001 0.001 0.001" />
         </geometry>
       </collision>
